File: PCB/Kicad/multiplexers.sch (KiCad schematic (older format))
At the start: 3 parts

Commit message: more sheets
pots
vumeters
switchers
Parts:
- U?: symbol 4xxx_IEEE:4067 -> 74xx:CD74HC4067M
Connections:
- net Vdd is gone; now on net VCC: U?.24 (VCC)
- net Vss is gone; now on net GND: U?.12 (GND)
- net A0: now also U?.15 (~E); no longer U?.1 (Z)
- net GND: now also U?.1 (COM); no longer U?.15 (~E)
Changed lines of the file:
@@
 $Descr A4 11693 8268
 encoding utf-8
-Sheet 3 4
+Sheet 3 6
 Title ""
 Date ""
@@
 $EndDescr
 $Comp
-L 4xxx_IEEE:4067 U?
+L 74xx:CD74HC4067M U?
 U 1 1 606035D2
 P 3200 2100
@@
 Text GLabel -1150 925  2    60   Input ~ 0
 BR1
-Text GLabel 2050 1250 1    40   Input ~ 0
+Text GLabel 3200 1100 1    40   Input ~ 0
 VCC
 $Comp
 L power:GND #PWR?
 U 1 1 606138F8
-P 2050 3350
-F 0 "#PWR?" H 2050 3100 50  0001 C CNN
-F 1 "GND" H 2055 3177 50  0000 C CNN
-F 2 "" H 2050 3350 50  0001 C CNN
-F 3 "" H 2050 3350 50  0001 C CNN
-	1    2050 3350
+P 3200 3200
+F 0 "#PWR?" H 3200 2950 50  0001 C CNN
+F 1 "GND" H 3205 3027 50  0000 C CNN
+F 2 "" H 3200 3200 50  0001 C CNN
+F 3 "" H 3200 3200 50  0001 C CNN
+	1    3200 3200
 	1    0    0    -1
 $EndComp
-Text GLabel 2600 2650 0    40   Input ~ 0
+Text GLabel 2700 2700 0    40   Input ~ 0
 A0
-Text GLabel 2600 1950 0    40   Input ~ 0
+Text GLabel 2700 2000 0    40   Input ~ 0
 D4
-Text GLabel 2600 2050 0    40   Input ~ 0
+Text GLabel 2700 2100 0    40   Input ~ 0
 D5
-Text GLabel 2600 2150 0    40   Input ~ 0
+Text GLabel 2700 2200 0    40   Input ~ 0
 D6
-Text GLabel 2600 2250 0    40   Input ~ 0
+Text GLabel 2700 2300 0    40   Input ~ 0
 D7
-Text GLabel 2600 1550 0    40   Input ~ 0
+Text GLabel 2700 1600 0    40   Input ~ 0
 GND
 $EndSCHEMATC

Commit message: multiplexers WIP
Parts:
- added U? (x2): CD74HC4067M, Package_SO:SOIC-24W_7.5x15.4mm_P1.27mm, symbol 74xx:CD74HC4067M
Connections:
- net A1: now also U?.15 (~E)
- net D4: now also U?.10 (S0), U?.10 (S0)
- net D5: now also U?.11 (S1), U?.11 (S1)
- net D6: now also U?.14 (S2), U?.14 (S2)
- net D7: now also U?.13 (S3), U?.13 (S3)
- net GND: now also U?.1 (COM), U?.1 (COM), U?.12 (GND), U?.12 (GND)
- net VCC: now also U?.24 (VCC), U?.24 (VCC)
- net FILTER-L2: now reaches U?.16 (I15)
- net BAS-L2: now reaches U?.17 (I14)
- net MID-L2: now reaches U?.18 (I13)
- net MID-L1: now reaches U?.19 (I12)
- net FADER-L1: now reaches U?.2 (I7)
- net BAS-L1: now reaches U?.20 (I11)
- net FILTER-L1: now reaches U?.21 (I10)
- net FADER-L2: now reaches U?.22 (I9)
- net SWPRECUE-L2: now reaches U?.23 (I8)
- net SWPRECUE-L1: now reaches U?.3 (I6)
- net PITCH-L: now reaches U?.4 (I5)
- net SWSHIFT-L: now reaches U?.5 (I4)
- net SWSYNC-L: now reaches U?.6 (I3)
- net SWRANGE-L: now reaches U?.7 (I2)
- net SWPLAY-L: now reaches U?.8 (I1)
- net SWCUE-L: now reaches U?.9 (I0)
- new net A2: U?.15 (~E)
- new net BAS-L3: U?.19 (I12)
- new net FADER-L3: U?.2 (I7)
- new net FILTER-L3: U?.18 (I13)
- new net MID-L3: U?.20 (I11)
- new net PFX-1R: U?.23 (I8)
- new net PFX-2R: U?.21 (I10)
- new net PFX-3R: U?.19 (I12)
- new net PITCH-R: U?.4 (I5)
- new net PMASTER: U?.21 (I10)
- new net PMIX-HP: U?.23 (I8)
- new net PVOL-HP: U?.22 (I9)
- new net SWBR-BACK-R: U?.16 (I15)
- new net SWBR-PREVIEW-R: U?.17 (I14)
- new net SWCUE-R: U?.9 (I0)
- new net SWFX1-R: U?.22 (I9)
- new net SWFX2-R: U?.20 (I11)
- new net SWFX3-R: U?.18 (I13)
- new net SWPAD-L1: U?.9 (I0)
- new net SWPAD-L2: U?.8 (I1)
- new net SWPAD-L3: U?.7 (I2)
- new net SWPAD-L4: U?.6 (I3)
- new net SWPAD-L5: U?.5 (I4)
- new net SWPAD-L6: U?.4 (I5)
- new net SWPAD-L7: U?.3 (I6)
- new net SWPAD-L8: U?.2 (I7)
- new net SWPLAY-R: U?.8 (I1)
- new net SWPRECUE-L3: U?.3 (I6)
- new net SWRANGE-R: U?.7 (I2)
- new net SWSHIFT-R: U?.5 (I4)
- new net SWSYNC-R: U?.6 (I3)
Changed lines of the file:
@@
 Text GLabel 2700 1600 0    40   Input ~ 0
 GND
+Text GLabel 3700 1400 2    40   Input ~ 0
+SWCUE-L
+Text GLabel 3700 1500 2    40   Input ~ 0
+SWPLAY-L
+Text GLabel 3700 1600 2    40   Input ~ 0
+SWRANGE-L
+Text GLabel 3700 1700 2    40   Input ~ 0
+SWSYNC-L
+Text GLabel 3700 1800 2    40   Input ~ 0
+SWSHIFT-L
+Text GLabel 3700 1900 2    40   Input ~ 0
+PITCH-L
+Text GLabel 3700 2000 2    40   Input ~ 0
+SWPRECUE-L1
+Text GLabel 3700 2100 2    40   Input ~ 0
+FADER-L1
+Text GLabel 3700 2200 2    40   Input ~ 0
+SWPRECUE-L2
+Text GLabel 3700 2300 2    40   Input ~ 0
+FADER-L2
+Text GLabel 3700 2400 2    40   Input ~ 0
+FILTER-L1
+Text GLabel 3700 2500 2    40   Input ~ 0
+BAS-L1
+Text GLabel 3700 2600 2    40   Input ~ 0
+MID-L1
+Text GLabel 3700 2700 2    40   Input ~ 0
+MID-L2
+Text GLabel 3700 2800 2    40   Input ~ 0
+BAS-L2
+Text GLabel 3700 2900 2    40   Input ~ 0
+FILTER-L2
+$Comp
+L 74xx:CD74HC4067M U?
+U 1 1 605FE2E2
+P 5450 2100
+F 0 "U?" H 5450 3300 50  0000 C CNN
+F 1 "CD74HC4067M" H 5450 3200 50  0000 C CNN
+F 2 "Package_SO:SOIC-24W_7.5x15.4mm_P1.27mm" H 6350 1100 50  0001 C CIN
+F 3 "http://www.ti.com/lit/ds/symlink/cd74hc4067.pdf" H 5100 2950 50  0001 C CNN
+	1    5450 2100
+	1    0    0    -1
+$EndComp
+Text GLabel 4950 2000 0    40   Input ~ 0
+D4
+Text GLabel 4950 2100 0    40   Input ~ 0
+D5
+Text GLabel 4950 2200 0    40   Input ~ 0
+D6
+Text GLabel 4950 2300 0    40   Input ~ 0
+D7
+Text GLabel 4950 1600 0    40   Input ~ 0
+GND
+Text GLabel 4950 2700 0    40   Input ~ 0
+A1
+Text GLabel 5950 1400 2    40   Input ~ 0
+SWCUE-R
+Text GLabel 5950 1500 2    40   Input ~ 0
+SWPLAY-R
+Text GLabel 5950 1600 2    40   Input ~ 0
+SWRANGE-R
+Text GLabel 5950 1700 2    40   Input ~ 0
+SWSYNC-R
+Text GLabel 5950 1800 2    40   Input ~ 0
+SWSHIFT-R
+Text GLabel 5950 1900 2    40   Input ~ 0
+PITCH-R
+Text GLabel 5950 2000 2    40   Input ~ 0
+SWPRECUE-L3
+Text GLabel 5950 2100 2    40   Input ~ 0
+FADER-L3
+Text GLabel 5950 2200 2    40   Input ~ 0
+PMIX-HP
+Text GLabel 5950 2300 2    40   Input ~ 0
+PVOL-HP
+Text GLabel 5950 2500 2    40   Input ~ 0
+MID-L3
+Text GLabel 5950 2600 2    40   Input ~ 0
+BAS-L3
+Text GLabel 5950 2700 2    40   Input ~ 0
+FILTER-L3
+Text GLabel 5950 2400 2    40   Input ~ 0
+PMASTER
+$Comp
+L 74xx:CD74HC4067M U?
+U 1 1 60601E62
+P 7750 2100
+F 0 "U?" H 7750 3300 50  0000 C CNN
+F 1 "CD74HC4067M" H 7750 3200 50  0000 C CNN
+F 2 "Package_SO:SOIC-24W_7.5x15.4mm_P1.27mm" H 8650 1100 50  0001 C CIN
+F 3 "http://www.ti.com/lit/ds/symlink/cd74hc4067.pdf" H 7400 2950 50  0001 C CNN
+	1    7750 2100
+	1    0    0    -1
+$EndComp
+Text GLabel 7250 2000 0    40   Input ~ 0
+D4
+Text GLabel 7250 2100 0    40   Input ~ 0
+D5
+Text GLabel 7250 2200 0    40   Input ~ 0
+D6
+Text GLabel 7250 2300 0    40   Input ~ 0
+D7
+Text GLabel 7250 1600 0    40   Input ~ 0
+GND
+Text GLabel 7250 2700 0    40   Input ~ 0
+A2
+Text GLabel 5450 1100 1    40   Input ~ 0
+VCC
+Text GLabel 7750 1100 1    40   Input ~ 0
+VCC
+$Comp
+L power:GND #PWR?
+U 1 1 606043CF
+P 5450 3200
+F 0 "#PWR?" H 5450 2950 50  0001 C CNN
+F 1 "GND" H 5455 3027 50  0000 C CNN
+F 2 "" H 5450 3200 50  0001 C CNN
+F 3 "" H 5450 3200 50  0001 C CNN
+	1    5450 3200
+	1    0    0    -1
+$EndComp
+$Comp
+L power:GND #PWR?
+U 1 1 606047E3
+P 7750 3200
+F 0 "#PWR?" H 7750 2950 50  0001 C CNN
+F 1 "GND" H 7755 3027 50  0000 C CNN
+F 2 "" H 7750 3200 50  0001 C CNN
+F 3 "" H 7750 3200 50  0001 C CNN
+	1    7750 3200
+	1    0    0    -1
+$EndComp
+Text GLabel 8250 1400 2    40   Input ~ 0
+SWPAD-L1
+Text GLabel 8250 1500 2    40   Input ~ 0
+SWPAD-L2
+Text GLabel 8250 1600 2    40   Input ~ 0
+SWPAD-L3
+Text GLabel 8250 1700 2    40   Input ~ 0
+SWPAD-L4
+Text GLabel 8250 1800 2    40   Input ~ 0
+SWPAD-L5
+Text GLabel 8250 1900 2    40   Input ~ 0
+SWPAD-L6
+Text GLabel 8250 2000 2    40   Input ~ 0
+SWPAD-L7
+Text GLabel 8250 2100 2    40   Input ~ 0
+SWPAD-L8
+Text GLabel 8250 2200 2    40   Input ~ 0
+PFX-1R
+Text GLabel 8250 2400 2    40   Input ~ 0
+PFX-2R
+Text GLabel 8250 2600 2    40   Input ~ 0
+PFX-3R
+Text GLabel 8250 2300 2    40   Input ~ 0
+SWFX1-R
+Text GLabel 8250 2500 2    40   Input ~ 0
+SWFX2-R
+Text GLabel 8250 2700 2    40   Input ~ 0
+SWFX3-R
+Text GLabel 8250 2800 2    40   Input ~ 0
+SWBR-PREVIEW-R
+Text GLabel 8250 2900 2    40   Input ~ 0
+SWBR-BACK-R
 $EndSCHEMATC
