File: PCB/Kicad/Traktorino.kicad_pcb (KiCad board)
At the start: 2 copper layers, 100.5 x 218.2 mm, 96 parts, among them J1 analog_pins, J2 mux_pins, J3 595_pins, J4 d13

Commit message: progress
Parts:
- removed BL1, BL2, BL3, BL4, BL5, BL6, BR1, BR2, BR3, BR4, BR5, BR6, Bshift1: SW_PUSH_SMALL, Gustavo:SW_tactile
- removed En1: Encoder_switch, Gustavo:SF-ROTARY-ENCODER_gus
- removed G***: LOGO, Gustavo:traktorino-silk-5
- removed J1: analog_pins, Pin_Headers:Pin_Header_Straight_1x07_Pitch2.54mm
- removed J2: mux_pins, Pin_Headers:Pin_Header_Straight_1x06_Pitch2.54mm
- removed J3: 595_pins, Pin_Headers:Pin_Header_Straight_1x05_Pitch2.54mm
- removed J4: d13, Pin_Headers:Pin_Header_Straight_1x03_Pitch2.54mm
- removed MUXbuttons1, MUXpots1: 4067D, Gustavo:cd4067
- removed REF** (x6): 1pin, Connect:1pin
- removed REF**: VIA-6mm, tactile:VIA-6mm
- removed RL1, RL2, RL3, RL4, RL5, ROnOff1, RR1, RR2, RR3, RR4, RR5, RVU0, RVU1, RVU10, RVU11, RVU12, RVU13, RVU2, RVU3, RVU4, RVU5, RVU6, RVU7, RVU8, RVU9: R_Small, Resistors_ThroughHole:Resistor_Horizontal_RM7mm
- removed SHIELD1: ARDUINO_SHIELD, arduino_shields:ARDUINO_SHIELD_2_040pins
- removed VU0, VU1, VU10, VU11, VU12, VU13, VU2, VU3, VU4, VU5, VU6, VU7, VU8, VU9, ledL1, ledL2, ledL3, ledL4, ledL5, ledOnOff1, ledR1, ledR2, ledR3, ledR4, ledR5: LED, LEDs:LED-3MM
- removed VUL1, VUR1, leds1: 74HC595, Gustavo:DIL16
- removed potCF1, potL1, potR1: POT, Gustavo:SLIDER-MEDIUM-2-fSilk
- removed potL2, potL3, potL4, potL5, potL6, potMain1, potR2, potR3, potR4, potR5, potR6: POT, Gustavo:Pot_vertical
- added A1: Arduino_UNO_R3, Module:Arduino_UNO_R3_WithMountingHoles, F.Cu at (-324.0, -37.0)
- added D1: VUL1-0, LED_THT:LED_Rectangular_W3.0mm_H2.0mm, F.Cu at (-318.0, 146.0)
- added D10: VUL2, LED_THT:LED_Rectangular_W3.0mm_H2.0mm, F.Cu at (-354.0, 92.0)
- added D11: VUL2, LED_THT:LED_Rectangular_W3.0mm_H2.0mm, F.Cu at (-275.0, -72.0)
- added D12: VUL2, LED_THT:LED_Rectangular_W3.0mm_H2.0mm, F.Cu at (-357.0, 52.0)
- added D13: VUL2, LED_THT:LED_Rectangular_W3.0mm_H2.0mm, F.Cu at (-257.0, -65.0)
- added D14: VUL2, LED_THT:LED_Rectangular_W3.0mm_H2.0mm, F.Cu at (-357.0, 47.0)
- added D15: VUL2, LED_THT:LED_Rectangular_W3.0mm_H2.0mm, F.Cu at (-353.0, 136.0)
- added D16: VUL2, LED_THT:LED_Rectangular_W3.0mm_H2.0mm, F.Cu at (-353.0, 141.0)
- added D17: VUL3, LED_THT:LED_Rectangular_W3.0mm_H2.0mm, F.Cu at (-263.0, -72.0)
- added D18: VUL3, LED_THT:LED_Rectangular_W3.0mm_H2.0mm, F.Cu at (-264.0, -67.0)
- added D19: VUL3, LED_THT:LED_Rectangular_W3.0mm_H2.0mm, F.Cu at (-299.0, 128.0)
- added D2: VUL1-1, LED_THT:LED_Rectangular_W3.0mm_H2.0mm, F.Cu at (-318.0, 141.0)
- added D20: VUL3, LED_THT:LED_Rectangular_W3.0mm_H2.0mm, F.Cu at (-275.0, -37.0)
- added D21: VUL3, LED_THT:LED_Rectangular_W3.0mm_H2.0mm, F.Cu at (-269.0, -72.0)
- added D22: VUL3, LED_THT:LED_Rectangular_W3.0mm_H2.0mm, F.Cu at (-350.0, 80.0)
- added D23: VUL3, LED_THT:LED_Rectangular_W3.0mm_H2.0mm, F.Cu at (-312.0, 135.0)
- added D24: VUL3, LED_THT:LED_Rectangular_W3.0mm_H2.0mm, F.Cu at (-294.0, 133.0)
- added D25: VUMAS-L, LED_THT:LED_Rectangular_W3.0mm_H2.0mm, F.Cu at (-334.0, 153.0)
- added D26: VUMAS-L, LED_THT:LED_Rectangular_W3.0mm_H2.0mm, F.Cu at (-257.0, -70.0)
- added D27: VUMAS-L, LED_THT:LED_Rectangular_W3.0mm_H2.0mm, F.Cu at (-264.0, -62.0)
- added D28: VUMAS-L, LED_THT:LED_Rectangular_W3.0mm_H2.0mm, F.Cu at (-346.0, 131.0)
- added D29: VUMAS-L, LED_THT:LED_Rectangular_W3.0mm_H2.0mm, F.Cu at (-257.0, -60.0)
- added D3: VUL1-, LED_THT:LED_Rectangular_W3.0mm_H2.0mm, F.Cu at (-328.0, 143.0)
- added D30: VUMAS-L, LED_THT:LED_Rectangular_W3.0mm_H2.0mm, F.Cu at (-334.0, 143.0)
- added D31: VUMAS-L, LED_THT:LED_Rectangular_W3.0mm_H2.0mm, F.Cu at (-341.0, 146.0)
- added D32: VUMAS-L, LED_THT:LED_Rectangular_W3.0mm_H2.0mm, F.Cu at (-332.0, 96.0)
- added D33: VUMAS-R, LED_THT:LED_Rectangular_W3.0mm_H2.0mm, F.Cu at (-328.0, 138.0)
- added D34: VUMAS-R, LED_THT:LED_Rectangular_W3.0mm_H2.0mm, F.Cu at (-356.0, 80.0)
- added D35: VUMAS-R, LED_THT:LED_Rectangular_W3.0mm_H2.0mm, F.Cu at (-353.0, 131.0)
- added D36: VUMAS-R, LED_THT:LED_Rectangular_W3.0mm_H2.0mm, F.Cu at (-342.0, 136.0)
- added D37: VUMAS-R, LED_THT:LED_Rectangular_W3.0mm_H2.0mm, F.Cu at (-354.0, 87.0)
- added D38: VUMAS-R, LED_THT:LED_Rectangular_W3.0mm_H2.0mm, F.Cu at (-335.0, 138.0)
- added D39: VUMAS-R, LED_THT:LED_Rectangular_W3.0mm_H2.0mm, F.Cu at (-340.0, 126.0)
- added D4: VUL1-, LED_THT:LED_Rectangular_W3.0mm_H2.0mm, F.Cu at (-318.0, 136.0)
- added D40: VUMAS-R, LED_THT:LED_Rectangular_W3.0mm_H2.0mm, F.Cu at (-342.0, 141.0)
- added D41: LED_ALT, LED_THT:LED_Rectangular_W3.0mm_H2.0mm, F.Cu at (-302.0, 138.0)
- added D42: LED_ALT, LED_THT:LED_Rectangular_W3.0mm_H2.0mm, F.Cu at (-293.0, 128.0)
- added D43: LED_ALT, LED_THT:LED_Rectangular_W3.0mm_H2.0mm, F.Cu at (-301.0, 133.0)
- added D44: LED_ALT, LED_THT:LED_Rectangular_W3.0mm_H2.0mm, F.Cu at (-236.0, 69.0)
- added D45: LED_ALT, LED_THT:LED_Rectangular_W3.0mm_H2.0mm, F.Cu at (-357.0, 42.0)
- added D46: LED_ALT, LED_THT:LED_Rectangular_W3.0mm_H2.0mm, F.Cu at (-312.0, 140.0)
- added D47: LED_ALT, LED_THT:LED_Rectangular_W3.0mm_H2.0mm, F.Cu at (-283.0, 115.0)
- added D5: VUL1-, LED_THT:LED_Rectangular_W3.0mm_H2.0mm, F.Cu at (-328.0, 148.0)
- added D6: VUL1-, LED_THT:LED_Rectangular_W3.0mm_H2.0mm, F.Cu at (-340.0, 131.0)
- added D7: VUL1-, LED_THT:LED_Rectangular_W3.0mm_H2.0mm, F.Cu at (-334.0, 148.0)
- added D8: VUL1-, LED_THT:LED_Rectangular_W3.0mm_H2.0mm, F.Cu at (-274.0, 100.0)
- added D9: VUL2, LED_THT:LED_Rectangular_W3.0mm_H2.0mm, F.Cu at (-281.0, -37.0)
- added ENCLEFT4001: RotaryEncoder_Switch, Rotary_Encoder:RotaryEncoder_Alps_EC11E_Vertical_H20mm_CircularMountingHoles, F.Cu at (-331.8, -52.6)
- added ENCRIGHT4001: RotaryEncoder_Switch, Rotary_Encoder:RotaryEncoder_Alps_EC11E_Vertical_H20mm_CircularMountingHoles, F.Cu at (-332.0, -69.0)
- added IC-POTS-1: 74HC4067D,653, Package_SO:SOIC-24W_7.5x15.4mm_P1.27mm, F.Cu at (-307.0, 23.0)
- added IC-POTS-2: 74HC4067D,653, Package_SO:SOIC-24W_7.5x15.4mm_P1.27mm, F.Cu at (-255.0, 21.0)
- added IC-SW-1: 74HC4067D,653, Package_SO:SOIC-24W_7.5x15.4mm_P1.27mm, F.Cu at (-281.0, 23.0)
- added IC-SW-2: 74HC4067D,653, Package_SO:SOIC-24W_7.5x15.4mm_P1.27mm, F.Cu at (-294.0, 23.0)
- added IC-SW-3: 74HC4067D,653, Package_SO:SOIC-24W_7.5x15.4mm_P1.27mm, F.Cu at (-268.0, 22.0)
- added R1: R_Small, Resistor_THT:R_Axial_DIN0207_L6.3mm_D2.5mm_P7.62mm_Horizontal, F.Cu at (-322.0, 113.0)
- added R10: R_Small, Resistor_THT:R_Axial_DIN0207_L6.3mm_D2.5mm_P7.62mm_Horizontal, F.Cu at (-355.0, 115.0)
- added R11: R_Small, Resistor_THT:R_Axial_DIN0207_L6.3mm_D2.5mm_P7.62mm_Horizontal, F.Cu at (-356.0, -63.0)
- added R12: R_Small, Resistor_THT:R_Axial_DIN0207_L6.3mm_D2.5mm_P7.62mm_Horizontal, F.Cu at (-355.0, -45.0)
- added R13: R_Small, Resistor_THT:R_Axial_DIN0207_L6.3mm_D2.5mm_P7.62mm_Horizontal, F.Cu at (-355.0, -51.0)
- added R14: R_Small, Resistor_THT:R_Axial_DIN0207_L6.3mm_D2.5mm_P7.62mm_Horizontal, F.Cu at (-352.0, 74.0)
- added R15: R_Small, Resistor_THT:R_Axial_DIN0207_L6.3mm_D2.5mm_P7.62mm_Horizontal, F.Cu at (-355.0, 109.0)
- added R16: R_Small, Resistor_THT:R_Axial_DIN0207_L6.3mm_D2.5mm_P7.62mm_Horizontal, F.Cu at (-355.0, 103.0)
- added R17: R_Small, Resistor_THT:R_Axial_DIN0207_L6.3mm_D2.5mm_P7.62mm_Horizontal, F.Cu at (-313.0, -71.0)
- added R18: R_Small, Resistor_THT:R_Axial_DIN0207_L6.3mm_D2.5mm_P7.62mm_Horizontal, F.Cu at (-356.0, -69.0)
- added R19: R_Small, Resistor_THT:R_Axial_DIN0207_L6.3mm_D2.5mm_P7.62mm_Horizontal, F.Cu at (-323.0, 131.0)
- added R2: R_Small, Resistor_THT:R_Axial_DIN0207_L6.3mm_D2.5mm_P7.62mm_Horizontal, F.Cu at (-322.0, 107.0)
- added R20: R_Small, Resistor_THT:R_Axial_DIN0207_L6.3mm_D2.5mm_P7.62mm_Horizontal, F.Cu at (-344.0, -51.0)
- added R21: R_Small, Resistor_THT:R_Axial_DIN0207_L6.3mm_D2.5mm_P7.62mm_Horizontal, F.Cu at (-345.0, -63.0)
- added R22: R_Small, Resistor_THT:R_Axial_DIN0207_L6.3mm_D2.5mm_P7.62mm_Horizontal, F.Cu at (-344.0, 97.0)
- added R23: R_Small, Resistor_THT:R_Axial_DIN0207_L6.3mm_D2.5mm_P7.62mm_Horizontal, F.Cu at (-323.0, 125.0)
- added R24: R_Small, Resistor_THT:R_Axial_DIN0207_L6.3mm_D2.5mm_P7.62mm_Horizontal, F.Cu at (-312.0, 130.0)
- added R25: R_Small, Resistor_THT:R_Axial_DIN0207_L6.3mm_D2.5mm_P7.62mm_Horizontal, F.Cu at (-337.0, 91.0)
- added R26: R_Small, Resistor_THT:R_Axial_DIN0207_L6.3mm_D2.5mm_P7.62mm_Horizontal, F.Cu at (-356.0, -57.0)
- added R27: R_Small, Resistor_THT:R_Axial_DIN0207_L6.3mm_D2.5mm_P7.62mm_Horizontal, F.Cu at (-345.0, -69.0)
- added R28: R_Small, Resistor_THT:R_Axial_DIN0207_L6.3mm_D2.5mm_P7.62mm_Horizontal, F.Cu at (-344.0, 103.0)
- added R29: R_Small, Resistor_THT:R_Axial_DIN0207_L6.3mm_D2.5mm_P7.62mm_Horizontal, F.Cu at (-345.0, -57.0)
- added R3: R_Small, Resistor_THT:R_Axial_DIN0207_L6.3mm_D2.5mm_P7.62mm_Horizontal, F.Cu at (-333.0, 119.0)
- added R30: R_Small, Resistor_THT:R_Axial_DIN0207_L6.3mm_D2.5mm_P7.62mm_Horizontal, F.Cu at (-333.0, 107.0)
- added R31: R_Small, Resistor_THT:R_Axial_DIN0207_L6.3mm_D2.5mm_P7.62mm_Horizontal, F.Cu at (-344.0, 121.0)
- added R32: R_Small, Resistor_THT:R_Axial_DIN0207_L6.3mm_D2.5mm_P7.62mm_Horizontal, F.Cu at (-344.0, 109.0)
- added R33: R_Small, Resistor_THT:R_Axial_DIN0207_L6.3mm_D2.5mm_P7.62mm_Horizontal, F.Cu at (-334.0, 133.0)
- added R34: R_Small, Resistor_THT:R_Axial_DIN0207_L6.3mm_D2.5mm_P7.62mm_Horizontal, F.Cu at (-341.0, 79.0)
- added R35: R_Small, Resistor_THT:R_Axial_DIN0207_L6.3mm_D2.5mm_P7.62mm_Horizontal, F.Cu at (-355.0, 97.0)
- added R36: R_Small, Resistor_THT:R_Axial_DIN0207_L6.3mm_D2.5mm_P7.62mm_Horizontal, F.Cu at (-337.0, 85.0)
- added R37: R_Small, Resistor_THT:R_Axial_DIN0207_L6.3mm_D2.5mm_P7.62mm_Horizontal, F.Cu at (-348.0, 85.0)
- added R38: R_Small, Resistor_THT:R_Axial_DIN0207_L6.3mm_D2.5mm_P7.62mm_Horizontal, F.Cu at (-348.0, 91.0)
- added R39: R_Small, Resistor_THT:R_Axial_DIN0207_L6.3mm_D2.5mm_P7.62mm_Horizontal, F.Cu at (-344.0, 115.0)
- added R4: R_Small, Resistor_THT:R_Axial_DIN0207_L6.3mm_D2.5mm_P7.62mm_Horizontal, F.Cu at (-326.0, 95.0)
- added R40: R_Small, Resistor_THT:R_Axial_DIN0207_L6.3mm_D2.5mm_P7.62mm_Horizontal, F.Cu at (-352.0, 68.0)
- added R41: R_Small, Resistor_THT:R_Axial_DIN0207_L6.3mm_D2.5mm_P7.62mm_Horizontal, F.Cu at (-311.0, 118.0)
- added R42: R_Small, Resistor_THT:R_Axial_DIN0207_L6.3mm_D2.5mm_P7.62mm_Horizontal, F.Cu at (-300.0, 123.0)
- added R43: R_Small, Resistor_THT:R_Axial_DIN0207_L6.3mm_D2.5mm_P7.62mm_Horizontal, F.Cu at (-311.0, 124.0)
- added R44: R_Small, Resistor_THT:R_Axial_DIN0207_L6.3mm_D2.5mm_P7.62mm_Horizontal, F.Cu at (-239.0, 62.0)
- added R45: R_Small, Resistor_THT:R_Axial_DIN0207_L6.3mm_D2.5mm_P7.62mm_Horizontal, F.Cu at (-311.0, 36.0)
- added R46: R_Small, Resistor_THT:R_Axial_DIN0207_L6.3mm_D2.5mm_P7.62mm_Horizontal, F.Cu at (-322.0, 119.0)
- added R47: R_Small, Resistor_THT:R_Axial_DIN0207_L6.3mm_D2.5mm_P7.62mm_Horizontal, F.Cu at (-311.0, 112.0)
- added R5: R_Small, Resistor_THT:R_Axial_DIN0207_L6.3mm_D2.5mm_P7.62mm_Horizontal, F.Cu at (-333.0, 113.0)
- added R6: R_Small, Resistor_THT:R_Axial_DIN0207_L6.3mm_D2.5mm_P7.62mm_Horizontal, F.Cu at (-334.0, 127.0)
- added R7: R_Small, Resistor_THT:R_Axial_DIN0207_L6.3mm_D2.5mm_P7.62mm_Horizontal, F.Cu at (-333.0, 101.0)
- added R8: R_Small, Resistor_THT:R_Axial_DIN0207_L6.3mm_D2.5mm_P7.62mm_Horizontal, F.Cu at (-322.0, 101.0)
- added R9: R_Small, Resistor_THT:R_Axial_DIN0207_L6.3mm_D2.5mm_P7.62mm_Horizontal, F.Cu at (-344.0, -45.0)
- added RV1: R_POT, Potentiometer_THT:Potentiometer_Bourns_PTV09A-1_Single_Vertical, F.Cu at (-351.0, 48.0)
- added RV10: R_POT, Potentiometer_THT:Potentiometer_Bourns_PTV09A-1_Single_Vertical, F.Cu at (-285.0, 58.0)
- added RV11: R_POT, Potentiometer_THT:Potentiometer_Bourns_PTV09A-1_Single_Vertical, F.Cu at (-270.0, 57.0)
- added RV12: R_POT, Potentiometer_THT:Potentiometer_Bourns_PTV09A-1_Single_Vertical, F.Cu at (-255.0, 45.0)
- added RV13: R_POT, Potentiometer_THT:Potentiometer_Bourns_PTV09A-1_Single_Vertical, F.Cu at (-315.0, 73.0)
- added RV14: R_POT, Potentiometer_THT:Potentiometer_Bourns_PTV09A-1_Single_Vertical, F.Cu at (-281.0, -24.0)
- added RV15: R_POT, Potentiometer_THT:Potentiometer_Bourns_PTV09A-1_Single_Vertical, F.Cu at (-300.0, 92.0)
- added RV16: R_POT, Potentiometer_THT:Potentiometer_Bourns_PTV09A-1_Single_Vertical, F.Cu at (-270.0, 41.0)
- added RV17: R_POT, Potentiometer_THT:Potentiometer_Bourns_PTV09A-1_Single_Vertical, F.Cu at (-247.0, 29.0)
- added RV18: R_POT, Potentiometer_THT:Potentiometer_Bourns_PTV09A-1_Single_Vertical, F.Cu at (-247.0, 13.0)
- added RV19: R_POT, Potentiometer_THT:Potentiometer_Bourns_PTV09A-1_Single_Vertical, F.Cu at (-300.0, 76.0)
- added RV2: R_POT, Potentiometer_THT:Potentiometer_Bourns_PTV09A-1_Single_Vertical, F.Cu at (-330.0, 73.0)
- added RV20: R_POT, Potentiometer_THT:Potentiometer_Bourns_PTV09A-1_Single_Vertical, F.Cu at (-217.0, 16.0)
- added RV21: R_POT, Potentiometer_THT:Potentiometer_Bourns_PTV09A-1_Single_Vertical, F.Cu at (-266.0, -25.0)
- added RV22: R_POT, Potentiometer_THT:Potentiometer_Bourns_PTV09A-1_Single_Vertical, F.Cu at (-262.0, -9.00)
- added RV23: R_POT, Potentiometer_THT:Potentiometer_Bourns_PTV09A-1_Single_Vertical, F.Cu at (-278.0, 8.00)
- added RV24: R_POT, Potentiometer_THT:Potentiometer_Bourns_PTV09A-1_Single_Vertical, F.Cu at (-232.0, 31.0)
- added RV25: R_POT, Potentiometer_THT:Potentiometer_Bourns_PTV09A-1_Single_Vertical, F.Cu at (-232.0, 15.0)
- added RV26: R_POT, Potentiometer_THT:Potentiometer_Bourns_PTV09A-1_Single_Vertical, F.Cu at (-263.0, 7.00)
- added RV27: R_POT, Potentiometer_THT:Potentiometer_Bourns_PTV09A-1_Single_Vertical, F.Cu at (-315.0, 90.0)
- added RV28: R_POT, Potentiometer_THT:Potentiometer_Bourns_PTV09A-1_Single_Vertical, F.Cu at (-313.0, -47.0)
- added RV29: R_POT, Potentiometer_THT:Potentiometer_Bourns_PTV09A-1_Single_Vertical, F.Cu at (-247.0, -3.00)
- added RV3: R_POT, Potentiometer_THT:Potentiometer_Bourns_PTV09A-1_Single_Vertical, F.Cu at (-285.0, 74.0)
- added RV4: R_POT, Potentiometer_THT:Potentiometer_Bourns_PTV09A-1_Single_Vertical, F.Cu at (-281.0, -8.00)
- added RV5: R_POT, Potentiometer_THT:Potentiometer_Bourns_PTV09A-1_Single_Vertical, F.Cu at (-254.0, 61.0)
- added RV6: R_POT, Potentiometer_THT:Potentiometer_Bourns_PTV09A-1_Single_Vertical, F.Cu at (-217.0, 32.0)
- added RV7: R_POT, Potentiometer_THT:Potentiometer_Bourns_PTV09A-1_Single_Vertical, F.Cu at (-300.0, 42.0)
- added RV8: R_POT, Potentiometer_THT:Potentiometer_Bourns_PTV09A-1_Single_Vertical, F.Cu at (-300.0, 58.0)
- added RV9: R_POT, Potentiometer_THT:Potentiometer_Bourns_PTV09A-1_Single_Vertical, F.Cu at (-285.0, 42.0)
- added SWBRBACKL4001: SW_Push, Button_Switch_THT:SW_PUSH_6mm_H5mm, F.Cu at (-295.0, 112.0)
- added SWBRBACKR4001: SW_Push, Button_Switch_THT:SW_PUSH_6mm_H5mm, F.Cu at (-295.0, 101.0)
- added SWBRPREVL4001: SW_Push, Button_Switch_THT:SW_PUSH_6mm_H5mm, F.Cu at (-350.0, 57.0)
- added SWBRPREVR4001: SW_Push, Button_Switch_THT:SW_PUSH_6mm_H5mm, F.Cu at (-357.0, 20.0)
- added SWCUEL4001: SW_Push, Button_Switch_THT:SW_PUSH_6mm_H5mm, F.Cu at (-220.0, -13.0)
- added SWCUER4001: SW_Push, Button_Switch_THT:SW_PUSH_6mm_H5mm, F.Cu at (-231.0, -3.00)
- added SWFX1L4001: SW_Push, Button_Switch_THT:SW_PUSH_6mm_H5mm, F.Cu at (-297.0, -71.0)
- added SWFX1R4001: SW_Push, Button_Switch_THT:SW_PUSH_6mm_H5mm, F.Cu at (-246.0, -21.0)
- added SWFX2L4001: SW_Push, Button_Switch_THT:SW_PUSH_6mm_H5mm, F.Cu at (-286.0, -59.0)
- added SWFX2R4001: SW_Push, Button_Switch_THT:SW_PUSH_6mm_H5mm, F.Cu at (-253.0, -43.0)
- added SWFX3L4001: SW_Push, Button_Switch_THT:SW_PUSH_6mm_H5mm, F.Cu at (-231.0, -13.0)
- added SWFX3R4001: SW_Push, Button_Switch_THT:SW_PUSH_6mm_H5mm, F.Cu at (-257.0, 70.0)
- added SWPAD-L1: SW_Push, Button_Switch_THT:SW_PUSH_6mm_H5mm, F.Cu at (-307.0, 101.0)
- added SWPAD-L2: SW_Push, Button_Switch_THT:SW_PUSH_6mm_H5mm, F.Cu at (-286.0, -49.0)
- added SWPAD-L3: SW_Push, Button_Switch_THT:SW_PUSH_6mm_H5mm, F.Cu at (-357.0, 30.0)
- added SWPAD-L4: SW_Push, Button_Switch_THT:SW_PUSH_6mm_H5mm, F.Cu at (-308.0, -65.0)
- added SWPAD-L5: SW_Push, Button_Switch_THT:SW_PUSH_6mm_H5mm, F.Cu at (-297.0, -61.0)
- added SWPAD-L6: SW_Push, Button_Switch_THT:SW_PUSH_6mm_H5mm, F.Cu at (-297.0, -51.0)
- added SWPAD-L7: SW_Push, Button_Switch_THT:SW_PUSH_6mm_H5mm, F.Cu at (-325.0, 84.0)
- added SWPAD-L8: SW_Push, Button_Switch_THT:SW_PUSH_6mm_H5mm, F.Cu at (-340.0, 68.0)
- added SWPAD-R1: SW_Push, Button_Switch_THT:SW_PUSH_6mm_H5mm, F.Cu at (-269.0, 77.0)
- added SWPAD-R2: SW_Push, Button_Switch_THT:SW_PUSH_6mm_H5mm, F.Cu at (-238.0, 40.0)
- added SWPAD-R3: SW_Push, Button_Switch_THT:SW_PUSH_6mm_H5mm, F.Cu at (-246.0, 70.0)
- added SWPAD-R4: SW_Push, Button_Switch_THT:SW_PUSH_6mm_H5mm, F.Cu at (-268.0, 66.0)
- added SWPAD-R5: SW_Push, Button_Switch_THT:SW_PUSH_6mm_H5mm, F.Cu at (-208.0, -2.00)
- added SWPAD-R6: SW_Push, Button_Switch_THT:SW_PUSH_6mm_H5mm, F.Cu at (-250.0, -31.0)
- added SWPAD-R7: SW_Push, Button_Switch_THT:SW_PUSH_6mm_H5mm, F.Cu at (-264.0, -45.0)
- added SWPAD-R8: SW_Push, Button_Switch_THT:SW_PUSH_6mm_H5mm, F.Cu at (-275.0, -47.0)
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Routing:
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- removed copper zone on B.Cu, net +5V
- removed copper zone on F.Cu, net GND
Other:
- board size 100.5 x 218.2 mm -> 360 x 300 mm
- net class Default removed
- board text removed: "10"
- board text removed: "11"
- board text removed: "13"
- board text removed: "14"
- board text removed: "595 pins"
- board text removed: "5v"
- board text removed: "8"
- board text removed: "9"
- board text removed: "A2"
- board text removed: "A3"
- board text removed: "A4"
- board text removed: "A5"
- board text removed: "D13"
- board text removed: "Traktorino - Rev. 4 by Gustavo Silveira gustavosilveira@musiconerd.com www.musiconerd.com"
- board text removed: "analog pins"
- board text removed: "digital pins"
- board text removed: "gnd"
- board text removed: "mux pins"
- board text removed: "vin"

Commit message: mod layout
Parts:
- removed A1: Arduino_UNO_R3, Module:Arduino_UNO_R3_WithMountingHoles
- removed ENCLEFT4001, ENCRIGHT4001: RotaryEncoder_Switch, Rotary_Encoder:RotaryEncoder_Alps_EC11E_Vertical_H20mm_CircularMountingHoles
- removed SWBRBACKL4001, SWBRBACKR4001, SWBRPREVL4001, SWBRPREVR4001, SWCUEL4001, SWCUER4001, SWFX1L4001, SWFX1R4001, SWFX2L4001, SWFX2R4001, SWFX3L4001, SWFX3R4001, SWPAD-L1, SWPAD-L2, SWPAD-L3, SWPAD-L4, SWPAD-L5, SWPAD-L6, SWPAD-L7, SWPAD-L8, SWPAD-R1, SWPAD-R2, SWPAD-R3, SWPAD-R4, SWPAD-R5, SWPAD-R6, SWPAD-R7, SWPAD-R8, SWPLAYL4001, SWPLAYR4001, SWPRECUEL1, SWPRECUEL2, SWPRECUEL3, SWRANGEL4001, SWRANGER4001, SWSEL1, SWSEL2, SWSEL3, SWSHIFTL4001, SWSHIFTR4001, SWSYNCL4001, SWSYNCR4001: SW_Push, Button_Switch_THT:SW_PUSH_6mm_H5mm
- added J1: Power, Connector_PinHeader_2.54mm:PinHeader_1x08_P2.54mm_Vertical, F.Cu at (-400.9, 49.2)
- added J2: Analog IN, Connector_PinHeader_2.54mm:PinHeader_1x06_P2.54mm_Vertical, F.Cu at (-391.6, 49.2)
- added J3: Digital 8-end, Connector_PinHeader_2.54mm:PinHeader_1x10_P2.54mm_Vertical, F.Cu at (-405.5, 49.2)
- added J4: Digital 0-7, Connector_PinHeader_2.54mm:PinHeader_1x08_P2.54mm_Vertical, F.Cu at (-396.2, 49.2)
- added SW1: SWPADL1, Library:sw-pad, F.Cu at (-570.0, 139.1)
- added SW10: SWPADR2, Library:sw-pad, F.Cu at (-575.0, 190.0)
- added SW11: SWPADR3, Library:sw-pad, F.Cu at (-555.1, 211.5)
- added SW12: SWPADR4, Library:sw-pad, F.Cu at (-603.3, 196.4)
- added SW13: SWPADR5, Library:sw-pad, F.Cu at (-587.8, 156.2)
- added SW14: SWPADR6, Library:sw-pad, F.Cu at (-559.5, 139.1)
- added SW15: SWPADR7, Library:sw-pad, F.Cu at (-555.1, 203.0)
- added SW16: SWPADR8, Library:sw-pad, F.Cu at (-565.7, 211.5)
- added SW17: SWPLAYL, Button_Switch_THT:SW_PUSH_6mm_H5mm, F.Cu at (-640.6, 171.0)
- added SW18: SWCUEL, Button_Switch_THT:SW_PUSH_6mm_H5mm, F.Cu at (-612.2, 139.1)
- added SW19: SWSHIFTL, Button_Switch_THT:SW_PUSH_6mm_H5mm, F.Cu at (-622.8, 147.7)
- added SW2: SWPADL2, Library:sw-pad, F.Cu at (-548.9, 130.6)
- added SW20: SWSYNCL, Button_Switch_THT:SW_PUSH_6mm_H5mm, F.Cu at (-640.6, 179.6)
- added SW21: SWRANGEL, Button_Switch_THT:SW_PUSH_6mm_H5mm, F.Cu at (-601.7, 139.1)
- added SW22: SWFX1L, Button_Switch_THT:SW_PUSH_6mm_H5mm, F.Cu at (-601.7, 130.6)
- added SW23: SWFX2L, Button_Switch_THT:SW_PUSH_6mm_H5mm, F.Cu at (-630.0, 162.5)
- added SW24: SWFX3L, Button_Switch_THT:SW_PUSH_6mm_H5mm, F.Cu at (-622.8, 130.6)
- added SW25: SWBR-PREVL, Button_Switch_THT:SW_PUSH_6mm_H5mm, F.Cu at (-622.8, 139.1)
- added SW26: SWBR-BACKL, Button_Switch_THT:SW_PUSH_6mm_H5mm, F.Cu at (-619.5, 164.8)
- added SW27: SWPLAYR, Button_Switch_THT:SW_PUSH_6mm_H5mm, F.Cu at (-612.2, 147.7)
- added SW28: SWCUER, Button_Switch_THT:SW_PUSH_6mm_H5mm, F.Cu at (-630.0, 171.0)
- added SW29: SWSHIFTR, Button_Switch_THT:SW_PUSH_6mm_H5mm, F.Cu at (-591.1, 130.6)
- added SW3: SWPADL3, Library:sw-pad, F.Cu at (-559.5, 130.6)
- added SW30: SWSYNCR, Button_Switch_THT:SW_PUSH_6mm_H5mm, F.Cu at (-619.5, 156.2)
- added SW31: SWRANGER, Button_Switch_THT:SW_PUSH_6mm_H5mm, F.Cu at (-608.9, 156.2)
- added SW32: SWFX1R, Button_Switch_THT:SW_PUSH_6mm_H5mm, F.Cu at (-630.0, 179.6)
- added SW33: SWFX2R, Button_Switch_THT:SW_PUSH_6mm_H5mm, F.Cu at (-591.1, 139.1)
- added SW34: SWFX3R, Button_Switch_THT:SW_PUSH_6mm_H5mm, F.Cu at (-601.7, 147.7)
- added SW35: SWBR-PREVR, Button_Switch_THT:SW_PUSH_6mm_H5mm, F.Cu at (-570.0, 147.7)
- added SW36: SWBR-BACKR, Button_Switch_THT:SW_PUSH_6mm_H5mm, F.Cu at (-566.7, 156.2)
- added SW37: SWPCUEL1, Button_Switch_THT:SW_PUSH_6mm_H5mm, F.Cu at (-580.6, 130.6)
- added SW38: SWPCUEL2, Button_Switch_THT:SW_PUSH_6mm_H5mm, F.Cu at (-608.9, 164.8)
- added SW39: SWPCUEL3, Button_Switch_THT:SW_PUSH_6mm_H5mm, F.Cu at (-619.5, 173.3)
- added SW4: SWPADL4, Library:sw-pad, F.Cu at (-600.0, 205.0)
- added SW40: SWSEL1, Button_Switch_THT:SW_PUSH_6mm_H5mm, F.Cu at (-598.4, 156.2)
- added SW41: SWSEL2, Button_Switch_THT:SW_PUSH_6mm_H5mm, F.Cu at (-591.1, 147.7)
- added SW42: SWSEL3, Button_Switch_THT:SW_PUSH_6mm_H5mm, F.Cu at (-580.6, 139.1)
- added SW43: BROWSER-L, Rotary_Encoder:RotaryEncoder_Alps_EC11E-Switch_Vertical_H20mm_CircularMountingHoles, F.Cu at (-640.8, 150.0)
- added SW44: BROWSER-R, Rotary_Encoder:RotaryEncoder_Alps_EC11E-Switch_Vertical_H20mm_CircularMountingHoles, F.Cu at (-105.0, -70.0)
- added SW5: SWPADL5, Library:sw-pad, F.Cu at (-535.0, 185.0)
- added SW6: SWPADL6, Library:sw-pad, F.Cu at (-505.0, 205.0)
- added SW7: SWPADL7, Library:sw-pad, F.Cu at (-576.2, 211.5)
- added SW8: SWPADL8, Library:sw-pad, F.Cu at (-570.0, 130.6)
- added SW9: SWPADR1, Library:sw-pad, F.Cu at (-550.0, 180.0)
- D10, D11, D12, D9: value VUL2 -> LED_ALT
- D17, D18, D19, D20: value VUL3 -> VUL2
- D21, D22, D23: value VUL3 -> LED_ALT
- D25, D26, D27, D28, D29, D30, D31: value VUMAS-L -> VUL3
- D33, D34, D35, D36, D37, D38, D39: value VUMAS-R -> VUMAS-L
- D41, D42, D43, D44, D45, D46, D47: value LED_ALT -> VUMAS-R
- RV1: value R_POT -> FADERL1; footprint Potentiometer_THT:Potentiometer_Bourns_PTV09A-1_Single_Vertical -> Library:fader-L60
- RV10: value R_POT -> PFX1L
- RV11: value R_POT -> PFX1R
- RV12: value R_POT -> PVOL-HP
- RV13: value R_POT -> BASL1
- RV14: value R_POT -> BASL2
- RV15: value R_POT -> BASL3
- RV16: value R_POT -> PFX2L
- RV17: value R_POT -> PFX2R
- RV18: value R_POT -> PMASTER
- RV19: value R_POT -> MIDL1
- RV2: value R_POT -> FADERL2; footprint Potentiometer_THT:Potentiometer_Bourns_PTV09A-1_Single_Vertical -> Library:fader-L60
- RV20: value R_POT -> MIDL2
- RV21: value R_POT -> MIDL3
- RV22: value R_POT -> PFX3L
- RV23: value R_POT -> PFX3R
- RV24: value R_POT -> TREL1
- RV25: value R_POT -> TREL2
- RV26: value R_POT -> TREL3
- RV27: value R_POT -> GAINL1
- RV28: value R_POT -> GAINL2
- RV29: value R_POT -> GAINL3
- RV3: value R_POT -> FADERL3; footprint Potentiometer_THT:Potentiometer_Bourns_PTV09A-1_Single_Vertical -> Library:fader-L60
- RV4: value R_POT -> PITCH-L; footprint Potentiometer_THT:Potentiometer_Bourns_PTV09A-1_Single_Vertical -> Library:fader-L60
- RV5: value R_POT -> PITH-R; footprint Potentiometer_THT:Potentiometer_Bourns_PTV09A-1_Single_Vertical -> Library:fader-L60
- RV6: value R_POT -> PMIX-HP
- RV7: value R_POT -> FILTERL1
- RV8: value R_POT -> FILTERL2
- RV9: value R_POT -> FILTERL3
- moved RV20 433.3 mm to (-640.9, 105.7)
- moved RV24 413.3 mm to (-640.9, 91.4)
- moved RV25 403.8 mm to (-625.5, 105.7)
- moved RV28 368.0 mm to (-640.9, 120.1)
- moved RV21 368.0 mm to (-610.0, 105.7)
- moved RV14 348.7 mm to (-610.0, 91.4)
- moved RV7 346.1 mm to (-646.0, 50.1)
- moved RV11 345.8 mm to (-610.0, 120.1)
- moved RV17 341.8 mm to (-579.1, 109.9)
- moved RV26 339.8 mm to (-594.6, 81.2)
- moved RV6 335.5 mm to (-548.2, 85.3)
- moved RV22 333.9 mm to (-579.1, 95.5)
- moved RV19 331.6 mm to (-630.6, 50.1)
- moved RV15 326.7 mm to (-625.5, 120.1)
- moved RV29 324.9 mm to (-564.3, 66.8)
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Connections:
- IC-POTS-2 pad 16: (no net) -> unconnected-(IC-POTS-2-Pad16)
- IC-POTS-2 pad 17: (no net) -> unconnected-(IC-POTS-2-Pad17)
- IC-POTS-2 pad 18: (no net) -> unconnected-(IC-POTS-2-Pad18)
- IC-SW-1 pad 16: (no net) -> unconnected-(IC-SW-1-Pad16)
- IC-SW-1 pad 17: (no net) -> unconnected-(IC-SW-1-Pad17)
- IC-SW-1 pad 18: (no net) -> unconnected-(IC-SW-1-Pad18)
- IC-SW-3 pad 16: (no net) -> unconnected-(IC-SW-3-Pad16)
- IC-SW-3 pad 17: (no net) -> unconnected-(IC-SW-3-Pad17)
- IC-SW-3 pad 18: (no net) -> unconnected-(IC-SW-3-Pad18)
- IC-SW-3 pad 19: (no net) -> SW_BROWSER_R
- IC-SW-3 pad 20: (no net) -> SW_BROWSER_L
- R10 pad 1: VUL2-1 -> LEDCUER
- R11 pad 1: VUL2-2 -> LEDPLAYL
- R12 pad 1: VUL2-3 -> LEDCUEL
- R13 pad 1: VUL2-4 -> VUL2-0
- R14 pad 1: VUL2-5 -> VUL2-1
- R15 pad 1: VUL2-6 -> VUL2-2
- R16 pad 1: VUL2-7 -> VUL2-3
- R17 pad 1: VUL3-0 -> VUL2-4
- R18 pad 1: VUL3-1 -> VUL2-5
- R19 pad 1: VUL3-2 -> VUL2-6
- R20 pad 1: VUL3-3 -> VUL2-7
- R21 pad 1: VUL3-4 -> LEDHPL3
- R22 pad 1: VUL3-5 -> LEDHPL2
- R23 pad 1: VUL3-6 -> LEDHPL1
- R24 pad 1: VUL3-7 -> VUL3-0
- R25 pad 1: VUMASL-0 -> VUL3-1
- R26 pad 1: VUMASL-1 -> VUL3-2
- R27 pad 1: VUMASL-2 -> VUL3-3
- R28 pad 1: VUMASL-3 -> VUL3-4
- R29 pad 1: VUMASL-4 -> VUL3-5
- R30 pad 1: VUMASL-5 -> VUL3-6
- R31 pad 1: VUMASL-6 -> VUL3-7
- R32 pad 1: VUMASL-7 -> VUMASL-0
- R33 pad 1: VUMASR-0 -> VUMASL-1
- R34 pad 1: VUMASR-1 -> VUMASL-2
- R35 pad 1: VUMASR-2 -> VUMASL-3
- R36 pad 1: VUMASR-3 -> VUMASL-4
- R37 pad 1: VUMASR-4 -> VUMASL-5
- R38 pad 1: VUMASR-5 -> VUMASL-6
- R39 pad 1: VUMASR-6 -> VUMASL-7
- R40 pad 1: VUMASR-7 -> VUMASR-0
- R41 pad 1: LEDPLAYR -> VUMASR-1
- R42 pad 1: LEDCUER -> VUMASR-2
- R43 pad 1: LEDPLAYL -> VUMASR-3
- R44 pad 1: LEDCUEL -> VUMASR-4
- R45 pad 1: LEDHPL3 -> VUMASR-5
- R46 pad 1: LEDHPL2 -> VUMASR-6
- R47 pad 1: LEDHPL1 -> VUMASR-7
- R9 pad 1: VUL2-0 -> LEDPLAYR
- RV10 pad 2: MID-L2 -> PFX-1L
- RV11 pad 2: TRE-L2 -> PFX-1R
- RV12 pad 2: GAIN-L2 -> PVOL-HP
- RV13 pad 2: FADER-L3 -> BAS-L1
- RV14 pad 2: FILTER-L3 -> BAS-L2
- RV16 pad 2: MID-L3 -> PFX-2L
- RV17 pad 2: TRE-L3 -> PFX-2R
- RV18 pad 2: GAIN-L3 -> PMASTER
- RV19 pad 2: PITCH-L -> MID-L1
- RV2 pad 2: FILTER-L1 -> FADER-L2
- RV20 pad 2: PFX-1L -> MID-L2
- RV21 pad 2: PFX-2L -> MID-L3
- RV23 pad 2: PITCH-R -> PFX-3R
- RV24 pad 2: PFX-1R -> TRE-L1
- RV25 pad 2: PFX-2R -> TRE-L2
- RV26 pad 2: PFX-3R -> TRE-L3
- RV27 pad 2: PMIX-HP -> GAIN-L1
- RV28 pad 2: PVOL-HP -> GAIN-L2
- RV29 pad 2: PMASTER -> GAIN-L3
- RV3 pad 2: BAS-L1 -> FADER-L3
- RV4 pad 2: MID-L1 -> PITCH-L
- RV5 pad 2: TRE-L1 -> PITCH-R
- RV6 pad 2: GAIN-L1 -> PMIX-HP
- RV7 pad 2: FADER-L2 -> FILTER-L1
- RV9 pad 2: BAS-L2 -> FILTER-L3
- U-LEDS1 pad 15: (no net) -> unconnected-(U-LEDS1-Pad15)
- U-LEDS1 pad 9: (no net) -> unconnected-(U-LEDS1-Pad9)
Other:
- board size 360 x 300 mm -> 340 x 300 mm

Commit message: WIP
Parts:
- moved SW30 561.9 mm to (-57.8, 140.2)
- moved SW27 554.9 mm to (-57.5, 163.0)
- moved SW31 551.9 mm to (-57.8, 128.2)
- moved SW28 518.5 mm to (-111.5, 166.0)
- moved SW35 501.8 mm to (-110.2, -53.2)
- moved R16 498.3 mm to (-24.0, 206.0)
- moved R7 494.1 mm to (-24.0, 212.0)
- moved R29 491.9 mm to (-24.0, 188.0)
- moved R1 481.6 mm to (-24.0, -35.0)
- moved R5 480.0 mm to (-24.0, 182.0)
- moved R38 476.9 mm to (-24.0, 140.0)
- moved R17 476.8 mm to (-26.8, -46.0)
- moved R25 476.4 mm to (-24.0, 19.0)
- moved R8 475.9 mm to (-24.0, 37.0)
- moved R21 475.7 mm to (-24.0, 31.0)
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Connections:
- IC-POTS-2 pad 16: unconnected-(IC-POTS-2-Pad16) -> (no net)
- IC-POTS-2 pad 17: unconnected-(IC-POTS-2-Pad17) -> (no net)
- IC-POTS-2 pad 18: unconnected-(IC-POTS-2-Pad18) -> (no net)
- IC-SW-1 pad 16: unconnected-(IC-SW-1-Pad16) -> (no net)
- IC-SW-1 pad 17: unconnected-(IC-SW-1-Pad17) -> (no net)
- IC-SW-1 pad 18: unconnected-(IC-SW-1-Pad18) -> (no net)
- IC-SW-3 pad 16: unconnected-(IC-SW-3-Pad16) -> (no net)
- IC-SW-3 pad 17: unconnected-(IC-SW-3-Pad17) -> (no net)
- IC-SW-3 pad 18: unconnected-(IC-SW-3-Pad18) -> (no net)
- J1 pad 1: unconnected-(J1-Pad1) -> (no net)
- J1 pad 2: unconnected-(J1-Pad2) -> (no net)
- J1 pad 3: unconnected-(J1-Pad3) -> (no net)
- J1 pad 4: unconnected-(J1-Pad4) -> (no net)
- J1 pad 8: unconnected-(J1-Pad8) -> (no net)
- J2 pad 6: unconnected-(J2-Pad6) -> (no net)
- J3 pad 10: unconnected-(J3-Pad10) -> (no net)
- J3 pad 2: unconnected-(J3-Pad2) -> (no net)
- J3 pad 3: unconnected-(J3-Pad3) -> (no net)
- J3 pad 6: unconnected-(J3-Pad6) -> (no net)
- J3 pad 8: unconnected-(J3-Pad8) -> (no net)
- J3 pad 9: unconnected-(J3-Pad9) -> (no net)
- J4 pad 1: unconnected-(J4-Pad1) -> (no net)
- J4 pad 2: unconnected-(J4-Pad2) -> (no net)
- U-LEDS1 pad 15: unconnected-(U-LEDS1-Pad15) -> (no net)
- U-LEDS1 pad 9: unconnected-(U-LEDS1-Pad9) -> (no net)

Commit message: Arduino mega retrofit WIP
Parts:
- removed D1: VUL1-0, LED_THT:LED_Rectangular_W3.0mm_H2.0mm
- removed D10, D11, D12, D21, D22, D9: LED_ALT, LED_THT:LED_Rectangular_W3.0mm_H2.0mm
- removed D13, D14, D15, D16, D17, D18, D19, D20: VUL2, LED_THT:LED_Rectangular_W3.0mm_H2.0mm
- removed D2: VUL1-1, LED_THT:LED_Rectangular_W3.0mm_H2.0mm
- removed D24, D25, D26, D27, D28, D29, D30, D31: VUL3, LED_THT:LED_Rectangular_W3.0mm_H2.0mm
- removed D3, D4, D5, D6, D7, D8: VUL1-, LED_THT:LED_Rectangular_W3.0mm_H2.0mm
- removed D32, D33, D34, D35, D36, D37, D38, D39: VUMAS-L, LED_THT:LED_Rectangular_W3.0mm_H2.0mm
- removed D40, D41, D42, D43, D44, D45, D46, D47: VUMAS-R, LED_THT:LED_Rectangular_W3.0mm_H2.0mm
- removed J1: Power, Connector_PinHeader_2.54mm:PinHeader_1x08_P2.54mm_Vertical
- removed J2: Analog IN, Connector_PinHeader_2.54mm:PinHeader_1x06_P2.54mm_Vertical
- removed J3: Digital 8-end, Connector_PinHeader_2.54mm:PinHeader_1x10_P2.54mm_Vertical
- removed J4: Digital 0-7, Connector_PinHeader_2.54mm:PinHeader_1x08_P2.54mm_Vertical
- removed R1, R10, R11, R12, R13, R14, R15, R16, R17, R18, R19, R2, R20, R21, R22, R24, R25, R26, R27, R28, R29, R3, R30, R31, R32, R33, R34, R35, R36, R37, R38, R39, R4, R40, R41, R42, R43, R44, R45, R46, R47, R5, R6, R7, R8, R9: R_Small, Resistor_THT:R_Axial_DIN0207_L6.3mm_D2.5mm_P7.62mm_Horizontal
- added BCUELD1: LED_ALT, LED_THT:LED_Rectangular_W3.0mm_H2.0mm, F.Cu at (-339.5, 147.2)
- added BCUELR1: R_Small, Resistor_SMD:R_1206_3216Metric_Pad1.30x1.75mm_HandSolder, F.Cu at (36.5, -35.5)
- added BCUERD1: LED_ALT, LED_THT:LED_Rectangular_W3.0mm_H2.0mm, F.Cu at (-109.3, 162.9)
- added BCUERR1: R_Small, Resistor_SMD:R_1206_3216Metric_Pad1.30x1.75mm_HandSolder, F.Cu at (130.2, -22.6)
- added BHPL1D1: LED_ALT, LED_THT:LED_Rectangular_W3.0mm_H2.0mm, F.Cu at (-248.4, 113.5)
- added BHPL1R1: R_Small, Resistor_SMD:R_1206_3216Metric_Pad1.30x1.75mm_HandSolder, F.Cu at (58.1, -59.8)
- added BHPL2D1: LED_ALT, LED_THT:LED_Rectangular_W3.0mm_H2.0mm, F.Cu at (-213.2, 113.5)
- added BHPL2R1: R_Small, Resistor_SMD:R_1206_3216Metric_Pad1.30x1.75mm_HandSolder, F.Cu at (36.5, -51.7)
- added BPLAYLD1: LED_ALT, LED_THT:LED_Rectangular_W3.0mm_H2.0mm, F.Cu at (-339.6, 164.5)
- added BPLAYLR1: R_Small, Resistor_SMD:R_1206_3216Metric_Pad1.30x1.75mm_HandSolder, F.Cu at (25.8, -39.5)
- added BPLAYRD1: LED_ALT, LED_THT:LED_Rectangular_W3.0mm_H2.0mm, F.Cu at (-109.5, 148.1)
- added BPLAYRR1: R_Small, Resistor_SMD:R_1206_3216Metric_Pad1.30x1.75mm_HandSolder, F.Cu at (47.3, -55.7)
- added VUL1D1: LED_Filled, LED_THT:LED_Rectangular_W3.0mm_H2.0mm, F.Cu at (-232.9, 62.1)
- added VUL1D2: LED_Filled, LED_THT:LED_Rectangular_W3.0mm_H2.0mm, F.Cu at (-232.9, 56.1)
- added VUL1D3: LED_Filled, LED_THT:LED_Rectangular_W3.0mm_H2.0mm, F.Cu at (-232.9, 50.1)
- added VUL1D4: LED_Filled, LED_THT:LED_Rectangular_W3.0mm_H2.0mm, F.Cu at (-232.9, 44.1)
- added VUL1D5: LED_Filled, LED_THT:LED_Rectangular_W3.0mm_H2.0mm, F.Cu at (-232.9, 38.1)
- added VUL1D6: LED_Filled, LED_THT:LED_Rectangular_W3.0mm_H2.0mm, F.Cu at (-232.9, 32.1)
- added VUL1D7: LED_Filled, LED_THT:LED_Rectangular_W3.0mm_H2.0mm, F.Cu at (-232.9, 26.1)
- added VUL1D8: LED_Filled, LED_THT:LED_Rectangular_W3.0mm_H2.0mm, F.Cu at (-232.9, 20.1)
- added VUL1R1: R_Small, Resistor_SMD:R_1206_3216Metric_Pad1.30x1.75mm_HandSolder, B.Cu at (-294.2, 52.3)
- added VUL1R2: R_Small, Resistor_SMD:R_1206_3216Metric_Pad1.30x1.75mm_HandSolder, B.Cu at (-294.2, 47.2)
- added VUL1R3: R_Small, Resistor_SMD:R_1206_3216Metric_Pad1.30x1.75mm_HandSolder, B.Cu at (-294.2, 44.7)
- added VUL1R4: R_Small, Resistor_SMD:R_1206_3216Metric_Pad1.30x1.75mm_HandSolder, B.Cu at (-294.2, 42.1)
- added VUL1R5: R_Small, Resistor_SMD:R_1206_3216Metric_Pad1.30x1.75mm_HandSolder, B.Cu at (-294.2, 39.6)
- added VUL1R6: R_Small, Resistor_SMD:R_1206_3216Metric_Pad1.30x1.75mm_HandSolder, B.Cu at (-294.2, 37.0)
- added VUL1R7: R_Small, Resistor_SMD:R_1206_3216Metric_Pad1.30x1.75mm_HandSolder, B.Cu at (-294.2, 34.5)
- added VUL1R8: R_Small, Resistor_SMD:R_1206_3216Metric_Pad1.30x1.75mm_HandSolder, B.Cu at (-294.2, 30.5)
- added VUL2D1: LED_Filled, LED_THT:LED_Rectangular_W3.0mm_H2.0mm, F.Cu at (-197.9, 61.8)
- added VUL2D2: LED_Filled, LED_THT:LED_Rectangular_W3.0mm_H2.0mm, F.Cu at (-197.9, 55.8)
- added VUL2D3: LED_Filled, LED_THT:LED_Rectangular_W3.0mm_H2.0mm, F.Cu at (-197.9, 49.8)
- added VUL2D4: LED_Filled, LED_THT:LED_Rectangular_W3.0mm_H2.0mm, F.Cu at (-197.9, 43.8)
- added VUL2D5: LED_Filled, LED_THT:LED_Rectangular_W3.0mm_H2.0mm, F.Cu at (-197.9, 37.8)
- added VUL2D6: LED_Filled, LED_THT:LED_Rectangular_W3.0mm_H2.0mm, F.Cu at (-197.9, 31.8)
- added VUL2D7: LED_Filled, LED_THT:LED_Rectangular_W3.0mm_H2.0mm, F.Cu at (-197.9, 25.8)
- added VUL2D8: LED_Filled, LED_THT:LED_Rectangular_W3.0mm_H2.0mm, F.Cu at (-197.9, 19.8)
- added VUL2R1: R_Small, Resistor_SMD:R_1206_3216Metric_Pad1.30x1.75mm_HandSolder, F.Cu at (130.2, -10.5)
- added VUL2R2: R_Small, Resistor_SMD:R_1206_3216Metric_Pad1.30x1.75mm_HandSolder, F.Cu at (25.8, -47.6)
- added VUL2R3: R_Small, Resistor_SMD:R_1206_3216Metric_Pad1.30x1.75mm_HandSolder, F.Cu at (58.1, -51.7)
- added VUL2R4: R_Small, Resistor_SMD:R_1206_3216Metric_Pad1.30x1.75mm_HandSolder, F.Cu at (36.5, -47.6)
- added VUL2R5: R_Small, Resistor_SMD:R_1206_3216Metric_Pad1.30x1.75mm_HandSolder, F.Cu at (47.3, -31.4)
- added VUL2R6: R_Small, Resistor_SMD:R_1206_3216Metric_Pad1.30x1.75mm_HandSolder, F.Cu at (68.9, -59.8)
- added VUL2R7: R_Small, Resistor_SMD:R_1206_3216Metric_Pad1.30x1.75mm_HandSolder, F.Cu at (36.5, -55.7)
- added VUL2R8: R_Small, Resistor_SMD:R_1206_3216Metric_Pad1.30x1.75mm_HandSolder, F.Cu at (130.2, -26.7)
- added VUL3D1: LED_Filled, LED_THT:LED_Rectangular_W3.0mm_H2.0mm, F.Cu at (-163.9, 61.8)
- added VUL3D2: LED_Filled, LED_THT:LED_Rectangular_W3.0mm_H2.0mm, F.Cu at (-163.9, 55.8)
- added VUL3D3: LED_Filled, LED_THT:LED_Rectangular_W3.0mm_H2.0mm, F.Cu at (-163.9, 49.8)
- added VUL3D4: LED_Filled, LED_THT:LED_Rectangular_W3.0mm_H2.0mm, F.Cu at (-163.9, 43.8)
- added VUL3D5: LED_Filled, LED_THT:LED_Rectangular_W3.0mm_H2.0mm, F.Cu at (-163.9, 37.8)
- added VUL3D6: LED_Filled, LED_THT:LED_Rectangular_W3.0mm_H2.0mm, F.Cu at (-163.9, 31.8)
- added VUL3D7: LED_Filled, LED_THT:LED_Rectangular_W3.0mm_H2.0mm, F.Cu at (-163.9, 25.8)
- added VUL3D8: LED_Filled, LED_THT:LED_Rectangular_W3.0mm_H2.0mm, F.Cu at (-163.9, 19.8)
- added VUL3R1: R_Small, Resistor_SMD:R_1206_3216Metric_Pad1.30x1.75mm_HandSolder, F.Cu at (47.3, -47.6)
- added VUL3R2: R_Small, Resistor_SMD:R_1206_3216Metric_Pad1.30x1.75mm_HandSolder, F.Cu at (68.9, -55.7)
- added VUL3R3: R_Small, Resistor_SMD:R_1206_3216Metric_Pad1.30x1.75mm_HandSolder, F.Cu at (130.2, -38.8)
- added VUL3R4: R_Small, Resistor_SMD:R_1206_3216Metric_Pad1.30x1.75mm_HandSolder, F.Cu at (25.8, -35.5)
- added VUL3R5: R_Small, Resistor_SMD:R_1206_3216Metric_Pad1.30x1.75mm_HandSolder, F.Cu at (47.3, -59.8)
- added VUL3R6: R_Small, Resistor_SMD:R_1206_3216Metric_Pad1.30x1.75mm_HandSolder, F.Cu at (47.3, -51.7)
- added VUL3R7: R_Small, Resistor_SMD:R_1206_3216Metric_Pad1.30x1.75mm_HandSolder, F.Cu at (58.1, -43.6)
- added VUL3R8: R_Small, Resistor_SMD:R_1206_3216Metric_Pad1.30x1.75mm_HandSolder, F.Cu at (36.5, -39.5)
- added VUMASLD1: LED_Filled, LED_THT:LED_Rectangular_W3.0mm_H2.0mm, F.Cu at (-150.1, -7.80)
- added VUMASLD2: LED_Filled, LED_THT:LED_Rectangular_W3.0mm_H2.0mm, F.Cu at (-150.1, -13.8)
- added VUMASLD3: LED_Filled, LED_THT:LED_Rectangular_W3.0mm_H2.0mm, F.Cu at (-150.1, -19.8)
- added VUMASLD4: LED_Filled, LED_THT:LED_Rectangular_W3.0mm_H2.0mm, F.Cu at (-150.1, -25.8)
- added VUMASLD5: LED_Filled, LED_THT:LED_Rectangular_W3.0mm_H2.0mm, F.Cu at (-150.1, -31.8)
- added VUMASLD6: LED_Filled, LED_THT:LED_Rectangular_W3.0mm_H2.0mm, F.Cu at (-150.1, -37.8)
- added VUMASLD7: LED_Filled, LED_THT:LED_Rectangular_W3.0mm_H2.0mm, F.Cu at (-150.1, -43.8)
- added VUMASLD8: LED_Filled, LED_THT:LED_Rectangular_W3.0mm_H2.0mm, F.Cu at (-150.1, -49.8)
- added VUMASLR1: R_Small, Resistor_SMD:R_1206_3216Metric_Pad1.30x1.75mm_HandSolder, F.Cu at (36.5, -59.8)
- added VUMASLR2: R_Small, Resistor_SMD:R_1206_3216Metric_Pad1.30x1.75mm_HandSolder, F.Cu at (130.2, -14.5)
- added VUMASLR3: R_Small, Resistor_SMD:R_1206_3216Metric_Pad1.30x1.75mm_HandSolder, F.Cu at (58.1, -39.5)
- added VUMASLR4: R_Small, Resistor_SMD:R_1206_3216Metric_Pad1.30x1.75mm_HandSolder, F.Cu at (25.8, -31.4)
- added VUMASLR5: R_Small, Resistor_SMD:R_1206_3216Metric_Pad1.30x1.75mm_HandSolder, F.Cu at (130.2, -30.7)
- added VUMASLR6: R_Small, Resistor_SMD:R_1206_3216Metric_Pad1.30x1.75mm_HandSolder, F.Cu at (36.5, -27.4)
- added VUMASLR7: R_Small, Resistor_SMD:R_1206_3216Metric_Pad1.30x1.75mm_HandSolder, F.Cu at (51.0, -80.0)
- added VUMASLR8: R_Small, Resistor_SMD:R_1206_3216Metric_Pad1.30x1.75mm_HandSolder, F.Cu at (36.5, -43.6)
- added VUMASRD1: LED_Filled, LED_THT:LED_Rectangular_W3.0mm_H2.0mm, F.Cu at (-138.1, -7.80)
- added VUMASRD2: LED_Filled, LED_THT:LED_Rectangular_W3.0mm_H2.0mm, F.Cu at (-138.1, -13.8)
- added VUMASRD3: LED_Filled, LED_THT:LED_Rectangular_W3.0mm_H2.0mm, F.Cu at (-138.1, -19.8)
- added VUMASRD4: LED_Filled, LED_THT:LED_Rectangular_W3.0mm_H2.0mm, F.Cu at (-138.1, -25.8)
- added VUMASRD5: LED_Filled, LED_THT:LED_Rectangular_W3.0mm_H2.0mm, F.Cu at (-138.1, -31.8)
- added VUMASRD6: LED_Filled, LED_THT:LED_Rectangular_W3.0mm_H2.0mm, F.Cu at (-138.1, -37.8)
- added VUMASRD7: LED_Filled, LED_THT:LED_Rectangular_W3.0mm_H2.0mm, F.Cu at (-138.1, -43.8)
- added VUMASRD8: LED_Filled, LED_THT:LED_Rectangular_W3.0mm_H2.0mm, F.Cu at (-138.1, -49.8)
- added VUMASRR1: R_Small, Resistor_SMD:R_1206_3216Metric_Pad1.30x1.75mm_HandSolder, F.Cu at (130.2, -42.9)
- added VUMASRR2: R_Small, Resistor_SMD:R_1206_3216Metric_Pad1.30x1.75mm_HandSolder, F.Cu at (130.2, -18.6)
- added VUMASRR3: R_Small, Resistor_SMD:R_1206_3216Metric_Pad1.30x1.75mm_HandSolder, F.Cu at (47.3, -35.5)
- added VUMASRR4: R_Small, Resistor_SMD:R_1206_3216Metric_Pad1.30x1.75mm_HandSolder, F.Cu at (36.5, -31.4)
- added VUMASRR5: R_Small, Resistor_SMD:R_1206_3216Metric_Pad1.30x1.75mm_HandSolder, F.Cu at (47.3, -43.6)
- added VUMASRR6: R_Small, Resistor_SMD:R_1206_3216Metric_Pad1.30x1.75mm_HandSolder, F.Cu at (47.3, -39.5)
- added VUMASRR7: R_Small, Resistor_SMD:R_1206_3216Metric_Pad1.30x1.75mm_HandSolder, F.Cu at (130.2, -6.43)
- added VUMASRR8: R_Small, Resistor_SMD:R_1206_3216Metric_Pad1.30x1.75mm_HandSolder, F.Cu at (25.8, -23.3)
- added XA1: Arduino_Mega2560_Shield, Arduino:Arduino_Mega2560_Shield, F.Cu at (-124.9, -85.0)
- U-LEDS1, UVU-LINE1, UVU-LINE2, UVU-LINE3, UVU-MASTER-L1, UVU-MASTER-R1: footprint Package_DIP:DIP-16_W7.62mm_LongPads -> Package_SO:SO-16_3.9x9.9mm_P1.27mm
- moved SW12 588.5 mm to (-28.7, 69.4)
- moved SW36 567.5 mm to (-38.8, -51.9)
- moved SW16 562.6 mm to (-28.5, 44.2)
- moved SW13 552.2 mm to (-103.6, 44.3)
- moved RV23 548.0 mm to (-23.6, -7.92), turned to 90 degrees
- moved RV17 536.8 mm to (-55.4, -7.92), turned to 90 degrees
- moved SW29 535.1 mm to (-57.8, 174.1)
- moved SW15 526.1 mm to (-53.6, 44.2)
- moved SW11 521.4 mm to (-53.5, 69.1)
- moved SW10 511.0 mm to (-78.5, 69.4)
- moved RV11 509.5 mm to (-87.2, -7.90), turned to 90 degrees
- moved SW14 486.2 mm to (-78.6, 44.5)
- moved SW9 460.0 mm to (-103.6, 69.2)
- moved SW24 396.9 mm to (-284.2, 1.53)
- moved UVU-MASTER-R1 388.0 mm to (-149.0, -62.4), turned to 180 degrees
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Connections:
- D23 pad 1: GND -> Net-(D23-Pad1)
- D23 pad 2: Net-(D23-Pad2) -> LEDHPL3
- R23 pad 1: LEDHPL1 -> Net-(D23-Pad1)
- R23 pad 2: Net-(D23-Pad2) -> GND
