File: PCB/Kicad/Traktorino.kicad_pcb (KiCad board)
At the start: 2 copper layers, 340 x 300 mm, 179 parts, among them SW1 SWPADL1, SW10 SWPADR2, SW11 SWPADR3, SW12 SWPADR4, SW13 SWPADR5, SW14 SWPADR6, SW15 SWPADR7, SW16 SWPADR8, SW17 SWPLAYL, SW18 SWCUEL, SW19 SWSHIFTL, SW2 SWPADL2, SW20 SWSYNCL, SW21 SWRANGEL, SW22 SWFX1L, SW23 SWFX2L, SW24 SWFX3L, SW25 SWBR-PREVL, SW26 SWBR-BACKL, SW27 SWPLAYR, SW28 SWCUER, SW29 SWSHIFTR, SW3 SWPADL3, SW30 SWSYNCR, SW31 SWRANGER, SW32 SWFX1R, SW33 SWFX2R, SW34 SWFX3R, SW35 SWBR-PREVR, SW36 SWBR-BACKR, SW37 SWPCUEL1, SW38 SWPCUEL2, SW39 SWPCUEL3, SW4 SWPADL4, SW40 SWSEL1, SW41 SWSEL2, SW42 SWSEL3, SW43 BROWSER-L, SW44 BROWSER-R, SW5 SWPADL5, SW6 SWPADL6, SW7 SWPADL7, SW8 SWPADL8, SW9 SWPADR1

Commit message: pad footprint updated
Parts:
- BHPL1R1, BHPL2R1, VUL2R1, VUL2R2, VUL2R3, VUL2R4, VUL2R5, VUL2R6, VUL2R7, VUL2R8, VUL3R1, VUL3R2, VUL3R3, VUL3R4, VUL3R5, VUL3R6, VUL3R7, VUL3R8, VUMASLR1, VUMASLR2, VUMASLR3, VUMASLR4, VUMASLR5, VUMASLR6, VUMASLR7, VUMASLR8, VUMASRR1, VUMASRR2, VUMASRR3, VUMASRR4, VUMASRR5, VUMASRR6, VUMASRR7, VUMASRR8: moved to B.Cu
- R23: footprint Resistor_THT:R_Axial_DIN0207_L6.3mm_D2.5mm_P7.62mm_Horizontal -> Resistor_SMD:R_1206_3216Metric_Pad1.30x1.75mm_HandSolder
- moved BCUELR1 412.8 mm to (-325.4, 163.1)
- moved BPLAYLR1 401.0 mm to (-325.2, 154.5)
- moved BHPL1R1 356.8 mm to (-253.0, 115.0), turned to 180 degrees
- moved VUL2R8 336.3 mm to (-202.0, 26.0), turned to 180 degrees
- moved VUL2R1 331.8 mm to (-194.0, 60.0), turned to 180 degrees
- moved VUL3R3 310.9 mm to (-168.0, 49.0), turned to 180 degrees
- moved BHPL2R1 302.9 mm to (-217.0, 114.0), turned to 180 degrees
- moved BCUERR1 291.0 mm to (-94.7, 162.0)
- moved VUL2R6 286.6 mm to (-203.0, 31.0), turned to 180 degrees
- moved VUMASLR5 284.5 mm to (-154.0, -45.0), turned to 180 degrees
- moved VUMASRR1 275.7 mm to (-142.0, 1.00), turned to 180 degrees
- moved VUMASLR2 273.2 mm to (-143.0, -12.0), turned to 180 degrees
- moved VUL3R2 272.2 mm to (-178.0, 59.0), turned to 180 degrees
- moved VUL2R3 271.8 mm to (-194.0, 50.0), turned to 180 degrees
- moved VUMASRR2 271.5 mm to (-141.0, -5.00), turned to 180 degrees
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Connections:
- XA1 pad 3V3: unconnected-(XA1-Pad3V3) -> (no net)
- XA1 pad A10: unconnected-(XA1-PadA10) -> (no net)
- XA1 pad A11: unconnected-(XA1-PadA11) -> (no net)
- XA1 pad A12: unconnected-(XA1-PadA12) -> (no net)
- XA1 pad A13: unconnected-(XA1-PadA13) -> (no net)
- XA1 pad A14: unconnected-(XA1-PadA14) -> (no net)
- XA1 pad A15: unconnected-(XA1-PadA15) -> (no net)
- XA1 pad A5: unconnected-(XA1-PadA5) -> (no net)
- XA1 pad A6: unconnected-(XA1-PadA6) -> (no net)
- XA1 pad A7: unconnected-(XA1-PadA7) -> (no net)
- XA1 pad A8: unconnected-(XA1-PadA8) -> (no net)
- XA1 pad A9: unconnected-(XA1-PadA9) -> (no net)
- XA1 pad AREF: unconnected-(XA1-PadAREF) -> (no net)
- XA1 pad D0: unconnected-(XA1-PadD0) -> (no net)
- XA1 pad D1: unconnected-(XA1-PadD1) -> (no net)
- XA1 pad D10: unconnected-(XA1-PadD10) -> (no net)
- XA1 pad D13: unconnected-(XA1-PadD13) -> (no net)
- XA1 pad D14: unconnected-(XA1-PadD14) -> (no net)
- XA1 pad D15: unconnected-(XA1-PadD15) -> (no net)
- XA1 pad D16: unconnected-(XA1-PadD16) -> (no net)
- XA1 pad D17: unconnected-(XA1-PadD17) -> (no net)
- XA1 pad D18: unconnected-(XA1-PadD18) -> (no net)
- XA1 pad D19: unconnected-(XA1-PadD19) -> (no net)
- XA1 pad D20: unconnected-(XA1-PadD20) -> (no net)
- XA1 pad D21: unconnected-(XA1-PadD21) -> (no net)
- XA1 pad D22: unconnected-(XA1-PadD22) -> (no net)
- XA1 pad D23: unconnected-(XA1-PadD23) -> (no net)
- XA1 pad D24: unconnected-(XA1-PadD24) -> (no net)
- XA1 pad D25: unconnected-(XA1-PadD25) -> (no net)
- XA1 pad D26: unconnected-(XA1-PadD26) -> (no net)
- XA1 pad D27: unconnected-(XA1-PadD27) -> (no net)
- XA1 pad D28: unconnected-(XA1-PadD28) -> (no net)
- XA1 pad D29: unconnected-(XA1-PadD29) -> (no net)
- XA1 pad D30: unconnected-(XA1-PadD30) -> (no net)
- XA1 pad D31: unconnected-(XA1-PadD31) -> (no net)
- XA1 pad D32: unconnected-(XA1-PadD32) -> (no net)
- XA1 pad D33: unconnected-(XA1-PadD33) -> (no net)
- XA1 pad D34: unconnected-(XA1-PadD34) -> (no net)
- XA1 pad D35: unconnected-(XA1-PadD35) -> (no net)
- XA1 pad D36: unconnected-(XA1-PadD36) -> (no net)
- XA1 pad D37: unconnected-(XA1-PadD37) -> (no net)
- XA1 pad D38: unconnected-(XA1-PadD38) -> (no net)
- XA1 pad D39: unconnected-(XA1-PadD39) -> (no net)
- XA1 pad D40: unconnected-(XA1-PadD40) -> (no net)
- XA1 pad D41: unconnected-(XA1-PadD41) -> (no net)
- XA1 pad D42: unconnected-(XA1-PadD42) -> (no net)
- XA1 pad D43: unconnected-(XA1-PadD43) -> (no net)
- XA1 pad D44: unconnected-(XA1-PadD44) -> (no net)
- XA1 pad D45: unconnected-(XA1-PadD45) -> (no net)
- XA1 pad D46: unconnected-(XA1-PadD46) -> (no net)
- XA1 pad D47: unconnected-(XA1-PadD47) -> (no net)
- XA1 pad D48: unconnected-(XA1-PadD48) -> (no net)
- XA1 pad D49: unconnected-(XA1-PadD49) -> (no net)
- XA1 pad D50: unconnected-(XA1-PadD50) -> (no net)
- XA1 pad D51: unconnected-(XA1-PadD51) -> (no net)
- XA1 pad D52: unconnected-(XA1-PadD52) -> (no net)
- XA1 pad D53: unconnected-(XA1-PadD53) -> (no net)
- XA1 pad D9: unconnected-(XA1-PadD9) -> (no net)
- XA1 pad IORF: unconnected-(XA1-PadIORF) -> (no net)
- XA1 pad RST1: unconnected-(XA1-PadRST1) -> (no net)
- XA1 pad SCL: unconnected-(XA1-PadSCL) -> (no net)
- XA1 pad SDA: unconnected-(XA1-PadSDA) -> (no net)
- XA1 pad VIN: unconnected-(XA1-PadVIN) -> (no net)

Commit message: trillbar added
Parts:
- removed IC-POTS-2, IC-SW-1, IC-SW-2, IC-SW-3: 74HC4067D,653, Package_SO:SOIC-24W_7.5x15.4mm_P1.27mm
- added PADL-D1: WS2812B, LED_SMD:LED_WS2812B_PLCC4_5.0x5.0mm_P3.2mm, F.Cu at (93.8, 208.5)
- added PADL-D2: WS2812B, LED_SMD:LED_WS2812B_PLCC4_5.0x5.0mm_P3.2mm, F.Cu at (118.9, 208.8)
- added PADL-D3: WS2812B, LED_SMD:LED_WS2812B_PLCC4_5.0x5.0mm_P3.2mm, F.Cu at (143.8, 208.7)
- added PADL-D4: WS2812B, LED_SMD:LED_WS2812B_PLCC4_5.0x5.0mm_P3.2mm, F.Cu at (168.7, 208.4)
- added PADL-D5: WS2812B, LED_SMD:LED_WS2812B_PLCC4_5.0x5.0mm_P3.2mm, F.Cu at (93.9, 183.6)
- added PADL-D6: WS2812B, LED_SMD:LED_WS2812B_PLCC4_5.0x5.0mm_P3.2mm, F.Cu at (119.0, 183.8)
- added PADL-D7: WS2812B, LED_SMD:LED_WS2812B_PLCC4_5.0x5.0mm_P3.2mm, F.Cu at (143.9, 184.0)
- added PADL-D8: WS2812B, LED_SMD:LED_WS2812B_PLCC4_5.0x5.0mm_P3.2mm, F.Cu at (169.0, 183.7)
- added PADL-IN-R1: R_Small, Resistor_SMD:R_1206_3216Metric_Pad1.30x1.75mm_HandSolder, B.Cu at (100.8, 196.5)
- added PADR-D1: WS2812B, LED_SMD:LED_WS2812B_PLCC4_5.0x5.0mm_P3.2mm, F.Cu at (334.4, 208.1)
- added PADR-D2: WS2812B, LED_SMD:LED_WS2812B_PLCC4_5.0x5.0mm_P3.2mm, F.Cu at (359.5, 208.2)
- added PADR-D3: WS2812B, LED_SMD:LED_WS2812B_PLCC4_5.0x5.0mm_P3.2mm, F.Cu at (384.4, 208.1)
- added PADR-D4: WS2812B, LED_SMD:LED_WS2812B_PLCC4_5.0x5.0mm_P3.2mm, F.Cu at (409.2, 208.3)
- added PADR-D5: WS2812B, LED_SMD:LED_WS2812B_PLCC4_5.0x5.0mm_P3.2mm, F.Cu at (334.3, 183.0)
- added PADR-D6: WS2812B, LED_SMD:LED_WS2812B_PLCC4_5.0x5.0mm_P3.2mm, F.Cu at (359.4, 183.5)
- added PADR-D7: WS2812B, LED_SMD:LED_WS2812B_PLCC4_5.0x5.0mm_P3.2mm, F.Cu at (384.3, 183.1)
- added PADR-D8: WS2812B, LED_SMD:LED_WS2812B_PLCC4_5.0x5.0mm_P3.2mm, F.Cu at (409.4, 183.0)
- added PADR-IN-R1: R_Small, Resistor_SMD:R_1206_3216Metric_Pad1.30x1.75mm_HandSolder, B.Cu at (344.7, 194.6)
- added TB1: trillbar-left, Library:trillbar, F.Cu at (133.9, 235.3)
- added TB2: trillbar-right, Library:trillbar, F.Cu at (372.5, 234.7)
- RV4, RV5: footprint Library:fader-L60 -> Library:fader-L75
- moved SW34 1010.2 mm to (408.5, 134.7)
- moved SW32 975.9 mm to (344.9, 134.8)
- moved SW33 945.0 mm to (376.7, 134.9)
- moved SW42 839.9 mm to (256.5, 70.1)
- moved SW41 807.5 mm to (222.7, 70.1)
- moved SW40 727.5 mm to (187.9, 70.1)
- moved U-LEDS1 725.8 mm to (242.5, 246.6)
- moved BPLAYRD1 478.3 mm to (338.5, 315.8)
- moved SW27 478.3 mm to (336.7, 318.6)
- moved SW17 465.6 mm to (98.9, 318.6)
- moved BPLAYLD1 465.6 mm to (100.9, 315.3)
- moved SW19 465.3 mm to (134.1, 332.1)
- moved RV4 465.2 mm to (160.2, 300.5)
- moved SW28 464.7 mm to (336.6, 289.1)
- moved BCUERD1 464.7 mm to (338.8, 286.0)
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Connections:
- net A0 renamed MPLEX-A0
- IC-POTS-1 pad 10: D4 -> MPLEX-S0
- IC-POTS-1 pad 11: D5 -> MPLEX-S1
- IC-POTS-1 pad 13: D7 -> MPLEX-S3
- IC-POTS-1 pad 14: D6 -> MPLEX-S2
- SW43 pad A: D2 -> BROWSER_A
- SW43 pad B: D3 -> BROWSER_B
- SW43 pad C: Net-(SW43-PadC) -> GND
- SW43 pad S2: Net-(SW43-PadC) -> GND
- SW44 pad A: D2 -> BROWSER_A
- SW44 pad B: D3 -> BROWSER_B
- SW44 pad C: Net-(SW44-PadC) -> GND
- SW44 pad S2: Net-(SW44-PadC) -> GND
- U-LEDS1 pad 11: D12 -> SF-CLOCK
- U-LEDS1 pad 12: D8 -> SF-LATCH
- UVU-LINE1 pad 11: D12 -> SF-CLOCK
- UVU-LINE1 pad 12: D8 -> SF-LATCH
- UVU-LINE1 pad 14: D11 -> SF-DATA
- UVU-LINE2 pad 11: D12 -> SF-CLOCK
- UVU-LINE2 pad 12: D8 -> SF-LATCH
- UVU-LINE3 pad 11: D12 -> SF-CLOCK
- UVU-LINE3 pad 12: D8 -> SF-LATCH
- UVU-MASTER-L1 pad 11: D12 -> SF-CLOCK
- UVU-MASTER-L1 pad 12: D8 -> SF-LATCH
- UVU-MASTER-R1 pad 11: D12 -> SF-CLOCK
- UVU-MASTER-R1 pad 12: D8 -> SF-LATCH
- XA1 pad A1: A1 -> GAIN-L1
- XA1 pad A10: (no net) -> PFX-1R
- XA1 pad A11: (no net) -> PFX-2R
- XA1 pad A12: (no net) -> PFX-3R
- XA1 pad A13: (no net) -> PMASTER
- XA1 pad A15: (no net) -> SF-DATA
- XA1 pad A2: A2 -> GAIN-L2
- XA1 pad A3: A3 -> GAIN-L3
- XA1 pad A4: A4 -> TRE-L1
- XA1 pad A5: (no net) -> TRE-L2
- XA1 pad A6: (no net) -> TRE-L3
- XA1 pad A7: (no net) -> PFX-1L
- XA1 pad A8: (no net) -> PFX-2L
- XA1 pad A9: (no net) -> PFX-3L
- XA1 pad D0: (no net) -> SWFX2-R
- XA1 pad D1: (no net) -> SWFX3-R
- XA1 pad D10: (no net) -> SW_BROWSER_L
- XA1 pad D11: D11 -> SW_BROWSER_R
- XA1 pad D12: D12 -> BROWSER_A
- XA1 pad D13: (no net) -> BROWSER_B
- XA1 pad D14: (no net) -> SWFX1-R
- XA1 pad D15: (no net) -> SWPAD-R5
- XA1 pad D16: (no net) -> SWPAD-R4
- XA1 pad D17: (no net) -> SWPAD-R3
- XA1 pad D18: (no net) -> SWPAD-R2
- XA1 pad D19: (no net) -> SWPAD-R1
- XA1 pad D2: D2 -> SWSEL-L3
- XA1 pad D20: (no net) -> SDA
- XA1 pad D21: (no net) -> SCL
- XA1 pad D22: (no net) -> SWPAD-R6
- XA1 pad D23: (no net) -> SWPAD-R7
- XA1 pad D24: (no net) -> SWPAD-L1
- XA1 pad D25: (no net) -> SWPAD-L2
- XA1 pad D26: (no net) -> SWPAD-L3
- XA1 pad D27: (no net) -> SWPAD-L4
- XA1 pad D28: (no net) -> SWPAD-L5
- XA1 pad D29: (no net) -> SWPAD-L6
- XA1 pad D3: D3 -> SWSEL-L2
- XA1 pad D30: (no net) -> SWPAD-L7
- XA1 pad D31: (no net) -> SWPAD-L8
- XA1 pad D32: (no net) -> SWPAD-R8
- XA1 pad D33: (no net) -> SWPLAY-L
- XA1 pad D34: (no net) -> SWCUE-L
- XA1 pad D35: (no net) -> SWSHIFT-L
- XA1 pad D36: (no net) -> SWSYNC-L
- XA1 pad D37: (no net) -> SWRANGE-L
- XA1 pad D38: (no net) -> SWPLAY-R
- XA1 pad D39: (no net) -> SWCUE-R
- XA1 pad D4: D4 -> SWSEL-L1
- XA1 pad D40: (no net) -> SWSHIFT-R
- XA1 pad D41: (no net) -> SWSYNC-R
- XA1 pad D42: (no net) -> SWRANGE-R
- XA1 pad D43: (no net) -> SWPRECUE-L1
- XA1 pad D44: (no net) -> SWPRECUE-L2
- XA1 pad D45: (no net) -> SWPRECUE-L3
- XA1 pad D46: (no net) -> SIG_PAD_LED_L
- XA1 pad D48: (no net) -> MPLEX-S0
- XA1 pad D49: (no net) -> MPLEX-S1
- XA1 pad D5: D5 -> SWFX3-L
- XA1 pad D50: (no net) -> MPLEX-S2
- XA1 pad D51: (no net) -> MPLEX-S3
- XA1 pad D52: (no net) -> SF-CLOCK
- XA1 pad D53: (no net) -> SF-LATCH
- XA1 pad D6: D6 -> SWFX2-L
- XA1 pad D7: D7 -> SWFX1-L
- XA1 pad D8: D8 -> SWBR-BACK
- XA1 pad D9: (no net) -> SWBR-PREVIEW
Routing:
- net SWPAD-L5: track 0.00 -> 393.6 mm, vias 0 -> 2
- net SWCUE-L: track 0.00 -> 351.9 mm, vias 0 -> 3
- net SWPAD-L1: track 0.00 -> 344.9 mm, vias 0 -> 6
- net SWPLAY-L: track 0.00 -> 336.9 mm, vias 0 -> 2
- net SWFX1-L: track 0.00 -> 332.6 mm
- net SWSHIFT-L: track 0.00 -> 327.8 mm, vias 0 -> 3
- net SWSYNC-L: track 0.00 -> 325.9 mm, vias 0 -> 3
- net SWPAD-L3: track 0.00 -> 321.1 mm, vias 0 -> 4
- net SWPLAY-R: track 0.00 -> 310.4 mm, vias 0 -> 7
- net SWFX2-L: track 0.00 -> 307.8 mm
- net SWFX3-L: track 0.00 -> 295.0 mm
- net SWBR-BACK: track 0.00 -> 291.3 mm
- net BROWSER_A: track 0.00 -> 291.0 mm
- net BROWSER_B: track 0.00 -> 287.8 mm
- net SWSHIFT-R: track 0.00 -> 285.8 mm, vias 0 -> 2
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