File: PCB/Kicad/multiplexers.kicad_sch (KiCad schematic)
At the start: 5 parts

Commit message: update elements WIP
Parts:
- removed U? (x5): CD74HC4067M, Package_SO:SOIC-24W_7.5x15.4mm_P1.27mm, symbol 74xx:CD74HC4067M
- added IC-POTS-1, IC-POTS-2, IC-SW-1, IC-SW-2, IC-SW-3: 74HC4067D,653, SOIC127P1032X265-24N, symbol SamacSys_Parts:74HC4067D,653
Connections:
- net A0: now also IC-POTS-1.1 (Z)
- net A1: now also IC-POTS-2.1 (Z)
- net A2: now also IC-SW-1.1 (Z)
- net A3: now also IC-SW-2.1 (Z)
- net A4: now also IC-SW-3.1 (Z)
- net BAS-L1: now also IC-POTS-1.21 (Y10)
- net BAS-L2: now also IC-POTS-1.20 (Y11)
- net BAS-L3: now also IC-POTS-1.19 (Y12)
- net D4: now also IC-POTS-1.10 (S0), IC-POTS-2.10 (S0), IC-SW-1.10 (S0), IC-SW-2.10 (S0), IC-SW-3.10 (S0)
- net D5: now also IC-POTS-1.11 (S1), IC-POTS-2.11 (S1), IC-SW-1.11 (S1), IC-SW-2.11 (S1), IC-SW-3.11 (S1)
- net D6: now also IC-POTS-1.14 (S2), IC-POTS-2.14 (S2), IC-SW-1.14 (S2), IC-SW-2.14 (S2), IC-SW-3.14 (S2)
- net D7: now also IC-POTS-1.13 (S3), IC-POTS-2.13 (S3), IC-SW-1.13 (S3), IC-SW-2.13 (S3), IC-SW-3.13 (S3)
- net FADER-L1: now also IC-POTS-1.8 (Y1)
- net FADER-L2: now also IC-POTS-1.7 (Y2)
- net FADER-L3: now also IC-POTS-1.6 (Y3)
- net FILTER-L1: now also IC-POTS-1.2 (Y7)
- net FILTER-L2: now also IC-POTS-1.23 (Y8)
- net FILTER-L3: now also IC-POTS-1.22 (Y9)
- net GAIN-L1: now also IC-POTS-2.6 (Y3)
- net GAIN-L2: now also IC-POTS-2.5 (Y4)
- net GAIN-L3: now also IC-POTS-2.4 (Y5)
- net GND: now also IC-POTS-1.12 (GND), IC-POTS-1.15 (~E), IC-POTS-2.12 (GND), IC-POTS-2.15 (~E), IC-SW-1.12 (GND), IC-SW-1.15 (~E), IC-SW-2.12 (GND), IC-SW-2.15 (~E), IC-SW-3.12 (GND), IC-SW-3.15 (~E)
- net MID-L1: now also IC-POTS-1.18 (Y13)
- net MID-L2: now also IC-POTS-1.17 (Y14)
- net MID-L3: now also IC-POTS-1.16 (Y15)
- net PFX-1L: now also IC-POTS-2.23 (Y8)
- net PFX-1R: now also IC-POTS-2.20 (Y11)
- net PFX-2L: now also IC-POTS-2.3 (Y6)
- net PFX-2R: now also IC-POTS-2.21 (Y10)
- net PFX-3L: now also IC-POTS-2.2 (Y7)
- net PFX-3R: now also IC-POTS-2.22 (Y9)
- net PITCH-L: now also IC-POTS-1.9 (Y0)
- net PITCH-R: now also IC-POTS-1.3 (Y6)
- net PMASTER: now also IC-POTS-2.19 (Y12)
- net PMIX-HP: now also IC-POTS-1.5 (Y4)
- net PVOL-HP: now also IC-POTS-1.4 (Y5)
- net SWBR-BACK-L: now also IC-SW-2.19 (Y12)
- net SWBR-BACK-R: now also IC-SW-3.19 (Y12)
- net SWBR-PREVIEW-L: now also IC-SW-2.20 (Y11)
- net SWBR-PREVIEW-R: now also IC-SW-3.20 (Y11)
- net SWCUE-L: now also IC-SW-1.2 (Y7)
- net SWCUE-R: now also IC-SW-1.23 (Y8)
- net SWFX1-L: now also IC-SW-2.23 (Y8)
- net SWFX1-R: now also IC-SW-3.23 (Y8)
- net SWFX2-L: now also IC-SW-2.22 (Y9)
- net SWFX2-R: now also IC-SW-3.22 (Y9)
- net SWFX3-L: now also IC-SW-2.21 (Y10)
- net SWFX3-R: now also IC-SW-3.21 (Y10)
- net SWPAD-L1: now also IC-SW-2.9 (Y0)
- net SWPAD-L2: now also IC-SW-2.8 (Y1)
- net SWPAD-L3: now also IC-SW-2.7 (Y2)
- net SWPAD-L4: now also IC-SW-2.6 (Y3)
- net SWPAD-L5: now also IC-SW-2.5 (Y4)
- net SWPAD-L6: now also IC-SW-2.4 (Y5)
- net SWPAD-L7: now also IC-SW-2.3 (Y6)
- net SWPAD-L8: now also IC-SW-2.2 (Y7)
- net SWPAD-R1: now also IC-SW-3.9 (Y0)
- net SWPAD-R2: now also IC-SW-3.8 (Y1)
- net SWPAD-R3: now also IC-SW-3.7 (Y2)
- net SWPAD-R4: now also IC-SW-3.6 (Y3)
- net SWPAD-R5: now also IC-SW-3.5 (Y4)
- net SWPAD-R6: now also IC-SW-3.4 (Y5)
- net SWPAD-R7: now also IC-SW-3.3 (Y6)
- net SWPAD-R8: now also IC-SW-3.2 (Y7)
- net SWPLAY-L: now also IC-SW-1.3 (Y6)
- net SWPLAY-R: now also IC-SW-1.22 (Y9)
- net SWPRECUE-L1: now also IC-SW-1.7 (Y2)
- net SWPRECUE-L2: now also IC-SW-1.8 (Y1)
- net SWPRECUE-L3: now also IC-SW-1.9 (Y0)
- net SWRANGE-L: now also IC-SW-1.4 (Y5)
- net SWRANGE-R: now also IC-SW-1.21 (Y10)
- net SWSEL-L1: now also IC-SW-2.18 (Y13)
- net SWSEL-L2: now also IC-SW-2.17 (Y14)
- net SWSEL-L3: now also IC-SW-2.16 (Y15)
- net SWSHIFT-L: now also IC-SW-1.6 (Y3)
- net SWSHIFT-R: now also IC-SW-1.19 (Y12)
- net SWSYNC-L: now also IC-SW-1.5 (Y4)
- net SWSYNC-R: now also IC-SW-1.20 (Y11)
- net TRE-L1: now also IC-POTS-2.7 (Y2)
- net TRE-L2: now also IC-POTS-2.8 (Y1)
- net TRE-L3: now also IC-POTS-2.9 (Y0)
- net VCC: now also IC-POTS-1.24 (VCC), IC-POTS-2.24 (VCC), IC-SW-1.24 (VCC), IC-SW-2.24 (VCC), IC-SW-3.24 (VCC)
- no-connect marks 0 -> 9

Commit message: progress
Parts:
- IC-POTS-1, IC-POTS-2, IC-SW-1, IC-SW-2, IC-SW-3: footprint SOIC127P1032X265-24N -> Package_SO:SOIC-24W_7.5x15.4mm_P1.27mm
Connections:
- net SWBR-BACK-L renamed SWBR-BACK
- net SWBR-BACK-R renamed SW_BROWSER_R
- net SWBR-PREVIEW-L renamed SWBR-PREVIEW
- net SWBR-PREVIEW-R renamed SW_BROWSER_L
Changed lines of the file:
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@@
     )
   )
-  (global_label "SWBR-PREVIEW-L" (shape input) (at 158.75 109.22 0)
-    (effects (font (size 1.016 1.016)) (justify left))
-    (property "Intersheet References" "${INTERSHEET_REFS}" (id 0) (at 174.5657 109.1565 0)
-      (effects (font (size 1.016 1.016)) (justify left) hide)
-    )
-  )
-  (global_label "SWBR-BACK-L" (shape input) (at 158.75 111.76 0)
-    (effects (font (size 1.016 1.016)) (justify left))
-    (property "Intersheet References" "${INTERSHEET_REFS}" (id 0) (at 172.0983 111.6965 0)
+  (global_label "SWBR-PREVIEW" (shape input) (at 158.75 109.22 0)
+    (effects (font (size 1.016 1.016)) (justify left))
+    (property "Intersheet References" "${INTERSHEET_REFS}" (id 0) (at 172.4854 109.1565 0)
+      (effects (font (size 1.016 1.016)) (justify left) hide)
+    )
+  )
+  (global_label "SWBR-BACK" (shape input) (at 158.75 111.76 0)
+    (effects (font (size 1.016 1.016)) (justify left))
+    (property "Intersheet References" "${INTERSHEET_REFS}" (id 0) (at 170.0179 111.6965 0)
       (effects (font (size 1.016 1.016)) (justify left) hide)
     )
@@
     )
   )
-  (global_label "SWBR-PREVIEW-R" (shape input) (at 215.9 109.22 0)
-    (effects (font (size 1.016 1.016)) (justify left))
-    (property "Intersheet References" "${INTERSHEET_REFS}" (id 0) (at 6.35 38.1 0)
-      (effects (font (size 1.27 1.27)) hide)
-    )
-  )
-  (global_label "SWBR-BACK-R" (shape input) (at 215.9 111.76 0)
-    (effects (font (size 1.016 1.016)) (justify left))
-    (property "Intersheet References" "${INTERSHEET_REFS}" (id 0) (at 6.35 38.1 0)
-      (effects (font (size 1.27 1.27)) hide)
+  (global_label "SW_BROWSER_L" (shape input) (at 215.9 109.22 0)
+    (effects (font (size 1.016 1.016)) (justify left))
+    (property "Intersheet References" "${INTERSHEET_REFS}" (id 0) (at 229.4902 109.1565 0)
+      (effects (font (size 1.016 1.016)) (justify left) hide)
+    )
+  )
+  (global_label "SW_BROWSER_R" (shape input) (at 215.9 111.76 0)
+    (effects (font (size 1.016 1.016)) (justify left))
+    (property "Intersheet References" "${INTERSHEET_REFS}" (id 0) (at 229.6837 111.6965 0)
+      (effects (font (size 1.016 1.016)) (justify left) hide)
     )
   )
@@
     (property "Reference" "IC-POTS-1" (id 0) (at 92.71 44.45 0))
     (property "Value" "74HC4067D,653" (id 1) (at 92.71 46.99 0))
-    (property "Footprint" "SOIC127P1032X265-24N" (id 2) (at 101.6 48.26 0)
+    (property "Footprint" "Package_SO:SOIC-24W_7.5x15.4mm_P1.27mm" (id 2) (at 101.6 48.26 0)
       (effects (font (size 1.27 1.27)) (justify left) hide)
     )
@@
     (property "Reference" "IC-SW-1" (id 0) (at 92.71 92.71 0))
     (property "Value" "74HC4067D,653" (id 1) (at 92.71 95.25 0))
-    (property "Footprint" "SOIC127P1032X265-24N" (id 2) (at 101.6 96.52 0)
+    (property "Footprint" "Package_SO:SOIC-24W_7.5x15.4mm_P1.27mm" (id 2) (at 101.6 96.52 0)
       (effects (font (size 1.27 1.27)) (justify left) hide)
     )
@@
     (property "Reference" "IC-SW-2" (id 0) (at 146.05 92.71 0))
     (property "Value" "74HC4067D,653" (id 1) (at 146.05 95.25 0))
-    (property "Footprint" "SOIC127P1032X265-24N" (id 2) (at 154.94 96.52 0)
+    (property "Footprint" "Package_SO:SOIC-24W_7.5x15.4mm_P1.27mm" (id 2) (at 154.94 96.52 0)
       (effects (font (size 1.27 1.27)) (justify left) hide)
     )
@@
     (property "Reference" "IC-POTS-2" (id 0) (at 147.32 44.45 0))
     (property "Value" "74HC4067D,653" (id 1) (at 147.32 46.99 0))
-    (property "Footprint" "SOIC127P1032X265-24N" (id 2) (at 156.21 48.26 0)
+    (property "Footprint" "Package_SO:SOIC-24W_7.5x15.4mm_P1.27mm" (id 2) (at 156.21 48.26 0)
       (effects (font (size 1.27 1.27)) (justify left) hide)
     )
@@
     (property "Reference" "IC-SW-3" (id 0) (at 203.2 92.71 0))
     (property "Value" "74HC4067D,653" (id 1) (at 203.2 95.25 0))
-    (property "Footprint" "SOIC127P1032X265-24N" (id 2) (at 212.09 96.52 0)
-      (effects (font (size 1.27 1.27)) (justify left) hide)
-    )
+    (property "Footprint" "Package_SO:SOIC-24W_7.5x15.4mm_P1.27mm" (id 2) (at 212.09 96.52 0)
+      (effects (font (size 1.27 1.27)) (justify left) hide)
+    )

Commit message: trillbar added
Parts:
- removed IC-SW-1, IC-SW-2, IC-SW-3: 74HC4067D,653, Package_SO:SOIC-24W_7.5x15.4mm_P1.27mm, symbol SamacSys_Parts:74HC4067D,653
Connections:
- net A0 renamed MPLEX-A0
- net A1 renamed MPLEX-A1
- net D4 renamed MPLEX-S0
- net D5 renamed MPLEX-S1
- net D6 renamed MPLEX-S2
- net D7 renamed MPLEX-S3
- no-connect marks 9 -> 3
