File: PCB/Kicad/switchers.kicad_sch (KiCad schematic)
At the start: 44 parts

Commit message: update elements WIP
Parts:
- gave numbers to parts that had none: 44

Commit message: progress
Parts:
- removed SW11, SW12, SW13, SW14, SW15, SW16, SW3, SW4, SW5, SW6, SW7, SW8: SW_Push, symbol Switch:SW_Push
- added SWPAD-L3, SWPAD-L4, SWPAD-L5, SWPAD-L6, SWPAD-L7, SWPAD-L8, SWPAD-R3, SWPAD-R4, SWPAD-R5, SWPAD-R6, SWPAD-R7, SWPAD-R8: SW_Push, Button_Switch_THT:SW_PUSH_6mm_H5mm, symbol Switch:SW_Push
- ENCLEFT4001: renamed from SW43; footprint (none) -> Rotary_Encoder:RotaryEncoder_Alps_EC11E_Vertical_H20mm_CircularMountingHoles
- ENCRIGHT4001: renamed from SW44; footprint (none) -> Rotary_Encoder:RotaryEncoder_Alps_EC11E_Vertical_H20mm_CircularMountingHoles
- SWBRBACKL4001: renamed from SW26; footprint (none) -> Button_Switch_THT:SW_PUSH_6mm_H5mm
- SWBRBACKR4001: renamed from SW36; footprint (none) -> Button_Switch_THT:SW_PUSH_6mm_H5mm
- SWBRPREVL4001: renamed from SW25; footprint (none) -> Button_Switch_THT:SW_PUSH_6mm_H5mm
- SWBRPREVR4001: renamed from SW35; footprint (none) -> Button_Switch_THT:SW_PUSH_6mm_H5mm
- SWCUEL4001: renamed from SW18; footprint (none) -> Button_Switch_THT:SW_PUSH_6mm_H5mm
- SWCUER4001: renamed from SW28; footprint (none) -> Button_Switch_THT:SW_PUSH_6mm_H5mm
- SWFX1L4001: renamed from SW22; footprint (none) -> Button_Switch_THT:SW_PUSH_6mm_H5mm
- SWFX1R4001: renamed from SW32; footprint (none) -> Button_Switch_THT:SW_PUSH_6mm_H5mm
- SWFX2L4001: renamed from SW23; footprint (none) -> Button_Switch_THT:SW_PUSH_6mm_H5mm
- SWFX2R4001: renamed from SW33; footprint (none) -> Button_Switch_THT:SW_PUSH_6mm_H5mm
- SWFX3L4001: renamed from SW24; footprint (none) -> Button_Switch_THT:SW_PUSH_6mm_H5mm
- SWFX3R4001: renamed from SW34; footprint (none) -> Button_Switch_THT:SW_PUSH_6mm_H5mm
- SWPAD-L1: renamed from SW1; footprint (none) -> Button_Switch_THT:SW_PUSH_6mm_H5mm
- SWPAD-L2: renamed from SW2; footprint (none) -> Button_Switch_THT:SW_PUSH_6mm_H5mm
- SWPAD-R1: renamed from SW9; footprint (none) -> Button_Switch_THT:SW_PUSH_6mm_H5mm
- SWPAD-R2: renamed from SW10; footprint (none) -> Button_Switch_THT:SW_PUSH_6mm_H5mm
- SWPLAYL4001: renamed from SW17; footprint (none) -> Button_Switch_THT:SW_PUSH_6mm_H5mm
- SWPLAYR4001: renamed from SW27; footprint (none) -> Button_Switch_THT:SW_PUSH_6mm_H5mm
- SWPRECUEL1: renamed from SW37; footprint (none) -> Button_Switch_THT:SW_PUSH_6mm_H5mm
- SWPRECUEL2: renamed from SW38; footprint (none) -> Button_Switch_THT:SW_PUSH_6mm_H5mm
- SWPRECUEL3: renamed from SW39; footprint (none) -> Button_Switch_THT:SW_PUSH_6mm_H5mm
- SWRANGEL4001: renamed from SW21; footprint (none) -> Button_Switch_THT:SW_PUSH_6mm_H5mm
- SWRANGER4001: renamed from SW31; footprint (none) -> Button_Switch_THT:SW_PUSH_6mm_H5mm
- SWSEL1: renamed from SW40; footprint (none) -> Button_Switch_THT:SW_PUSH_6mm_H5mm
- SWSEL2: renamed from SW41; footprint (none) -> Button_Switch_THT:SW_PUSH_6mm_H5mm
- SWSEL3: renamed from SW42; footprint (none) -> Button_Switch_THT:SW_PUSH_6mm_H5mm
- SWSHIFTL4001: renamed from SW19; footprint (none) -> Button_Switch_THT:SW_PUSH_6mm_H5mm
- SWSHIFTR4001: renamed from SW29; footprint (none) -> Button_Switch_THT:SW_PUSH_6mm_H5mm
- SWSYNCL4001: renamed from SW20; footprint (none) -> Button_Switch_THT:SW_PUSH_6mm_H5mm
- SWSYNCR4001: renamed from SW30; footprint (none) -> Button_Switch_THT:SW_PUSH_6mm_H5mm
Connections:
- net GND: now also SWPAD-L3.1, SWPAD-L4.1, SWPAD-L5.1, SWPAD-L6.1, SWPAD-L7.1, SWPAD-L8.1, SWPAD-R3.1, SWPAD-R4.1, SWPAD-R5.1, SWPAD-R6.1, SWPAD-R7.1, SWPAD-R8.1
- net SWPAD-L3: now also SWPAD-L3.2
- net SWPAD-L4: now also SWPAD-L4.2
- net SWPAD-L5: now also SWPAD-L5.2
- net SWPAD-L6: now also SWPAD-L6.2
- net SWPAD-L7: now also SWPAD-L7.2
- net SWPAD-L8: now also SWPAD-L8.2
- net SWPAD-R3: now also SWPAD-R3.2
- net SWPAD-R4: now also SWPAD-R4.2
- net SWPAD-R6: now also SWPAD-R6.2
- net SWPAD-R7: now also SWPAD-R7.2
- net SWPAD-R8: now also SWPAD-R8.2
- new net SWPAD-R5: SWPAD-R5.2

Commit message: mod layout
Parts:
- SW1: renamed from SWPAD-L1; value SW_Push -> SWPADL1; footprint Button_Switch_THT:SW_PUSH_6mm_H5mm -> Library:sw-pad
- SW10: renamed from SWPAD-R2; value SW_Push -> SWPADR2; footprint Button_Switch_THT:SW_PUSH_6mm_H5mm -> Library:sw-pad
- SW11: renamed from SWPAD-R3; value SW_Push -> SWPADR3; footprint Button_Switch_THT:SW_PUSH_6mm_H5mm -> Library:sw-pad
- SW12: renamed from SWPAD-R4; value SW_Push -> SWPADR4; footprint Button_Switch_THT:SW_PUSH_6mm_H5mm -> Library:sw-pad
- SW13: renamed from SWPAD-R5; value SW_Push -> SWPADR5; footprint Button_Switch_THT:SW_PUSH_6mm_H5mm -> Library:sw-pad
- SW14: renamed from SWPAD-R6; value SW_Push -> SWPADR6; footprint Button_Switch_THT:SW_PUSH_6mm_H5mm -> Library:sw-pad
- SW15: renamed from SWPAD-R7; value SW_Push -> SWPADR7; footprint Button_Switch_THT:SW_PUSH_6mm_H5mm -> Library:sw-pad
- SW16: renamed from SWPAD-R8; value SW_Push -> SWPADR8; footprint Button_Switch_THT:SW_PUSH_6mm_H5mm -> Library:sw-pad
- SW17: renamed from SWPLAYL4001; value SW_Push -> SWPLAYL
- SW18: renamed from SWCUEL4001; value SW_Push -> SWCUEL
- SW19: renamed from SWSHIFTL4001; value SW_Push -> SWSHIFTL
- SW2: renamed from SWPAD-L2; value SW_Push -> SWPADL2; footprint Button_Switch_THT:SW_PUSH_6mm_H5mm -> Library:sw-pad
- SW20: renamed from SWSYNCL4001; value SW_Push -> SWSYNCL
- SW21: renamed from SWRANGEL4001; value SW_Push -> SWRANGEL
- SW22: renamed from SWFX1L4001; value SW_Push -> SWFX1L
- SW23: renamed from SWFX2L4001; value SW_Push -> SWFX2L
- SW24: renamed from SWFX3L4001; value SW_Push -> SWFX3L
- SW25: renamed from SWBRPREVL4001; value SW_Push -> SWBR-PREVL
- SW26: renamed from SWBRBACKL4001; value SW_Push -> SWBR-BACKL
- SW27: renamed from SWPLAYR4001; value SW_Push -> SWPLAYR
- SW28: renamed from SWCUER4001; value SW_Push -> SWCUER
- SW29: renamed from SWSHIFTR4001; value SW_Push -> SWSHIFTR
- SW3: renamed from SWPAD-L3; value SW_Push -> SWPADL3; footprint Button_Switch_THT:SW_PUSH_6mm_H5mm -> Library:sw-pad
- SW30: renamed from SWSYNCR4001; value SW_Push -> SWSYNCR
- SW31: renamed from SWRANGER4001; value SW_Push -> SWRANGER
- SW32: renamed from SWFX1R4001; value SW_Push -> SWFX1R
- SW33: renamed from SWFX2R4001; value SW_Push -> SWFX2R
- SW34: renamed from SWFX3R4001; value SW_Push -> SWFX3R
- SW35: renamed from SWBRPREVR4001; value SW_Push -> SWBR-PREVR
- SW36: renamed from SWBRBACKR4001; value SW_Push -> SWBR-BACKR
- SW37: renamed from SWPRECUEL1; value SW_Push -> SWPCUEL1
- SW38: renamed from SWPRECUEL2; value SW_Push -> SWPCUEL2
- SW39: renamed from SWPRECUEL3; value SW_Push -> SWPCUEL3
- SW4: renamed from SWPAD-L4; value SW_Push -> SWPADL4; footprint Button_Switch_THT:SW_PUSH_6mm_H5mm -> Library:sw-pad
- SW40: renamed from SWSEL1; value SW_Push -> SWSEL1
- SW41: renamed from SWSEL2; value SW_Push -> SWSEL2
- SW42: renamed from SWSEL3; value SW_Push -> SWSEL3
- SW43: renamed from ENCLEFT4001; value RotaryEncoder_Switch -> BROWSER-L; footprint Rotary_Encoder:RotaryEncoder_Alps_EC11E_Vertical_H20mm_CircularMountingHoles -> Rotary_Encoder:RotaryEncoder_Alps_EC11E-Switch_Vertical_H20mm_CircularMountingHoles
- SW44: renamed from ENCRIGHT4001; value RotaryEncoder_Switch -> BROWSER-R; footprint Rotary_Encoder:RotaryEncoder_Alps_EC11E_Vertical_H20mm_CircularMountingHoles -> Rotary_Encoder:RotaryEncoder_Alps_EC11E-Switch_Vertical_H20mm_CircularMountingHoles
- SW5: renamed from SWPAD-L5; value SW_Push -> SWPADL5; footprint Button_Switch_THT:SW_PUSH_6mm_H5mm -> Library:sw-pad
- SW6: renamed from SWPAD-L6; value SW_Push -> SWPADL6; footprint Button_Switch_THT:SW_PUSH_6mm_H5mm -> Library:sw-pad
- SW7: renamed from SWPAD-L7; value SW_Push -> SWPADL7; footprint Button_Switch_THT:SW_PUSH_6mm_H5mm -> Library:sw-pad
- SW8: renamed from SWPAD-L8; value SW_Push -> SWPADL8; footprint Button_Switch_THT:SW_PUSH_6mm_H5mm -> Library:sw-pad
- SW9: renamed from SWPAD-R1; value SW_Push -> SWPADR1; footprint Button_Switch_THT:SW_PUSH_6mm_H5mm -> Library:sw-pad

Commit message: trillbar added
Connections:
- net GND: now also SW43.C, SW43.S2, SW44.C, SW44.S2
- net D2 renamed BROWSER_A
- net D3 renamed BROWSER_B
Changed lines of the file:
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@@
     (stroke (width 0) (type solid) (color 0 0 0 0))
   )
-  (wire (pts (xy 223.52 72.39) (xy 223.52 80.01))
-    (stroke (width 0) (type solid) (color 0 0 0 0))
-  )
-  (wire (pts (xy 223.52 80.01) (xy 246.38 80.01))
-    (stroke (width 0) (type solid) (color 0 0 0 0))
-  )
-  (wire (pts (xy 223.52 99.06) (xy 223.52 106.68))
-    (stroke (width 0) (type solid) (color 0 0 0 0))
-  )
-  (wire (pts (xy 223.52 106.68) (xy 246.38 106.68))
-    (stroke (width 0) (type solid) (color 0 0 0 0))
-  )
-  (wire (pts (xy 231.14 72.39) (xy 223.52 72.39))
-    (stroke (width 0) (type solid) (color 0 0 0 0))
-  )
-  (wire (pts (xy 231.14 99.06) (xy 223.52 99.06))
-    (stroke (width 0) (type solid) (color 0 0 0 0))
-  )
-  (wire (pts (xy 246.38 74.93) (xy 246.38 80.01))
-    (stroke (width 0) (type solid) (color 0 0 0 0))
-  )
-  (wire (pts (xy 246.38 101.6) (xy 246.38 106.68))
-    (stroke (width 0) (type solid) (color 0 0 0 0))
-  )
   (global_label "SWPAD-L1" (shape input) (at 40.64 33.02 0)
     (effects (font (size 1.016 1.016)) (justify left))
@@
     )
   )
-  (global_label "D2" (shape input) (at 231.14 69.85 180)
-    (effects (font (size 1.524 1.524)) (justify right))
-    (property "Intersheet References" "${INTERSHEET_REFS}" (id 0) (at 483.87 144.78 0)
-      (effects (font (size 1.27 1.27)) hide)
-    )
-  )
-  (global_label "D3" (shape input) (at 231.14 74.93 180)
-    (effects (font (size 1.524 1.524)) (justify right))
-    (property "Intersheet References" "${INTERSHEET_REFS}" (id 0) (at 1.905 -30.48 0)
-      (effects (font (size 1.27 1.27)) hide)
-    )
-  )
-  (global_label "D2" (shape input) (at 231.14 96.52 180)
-    (effects (font (size 1.524 1.524)) (justify right))
-    (property "Intersheet References" "${INTERSHEET_REFS}" (id 0) (at 483.87 171.45 0)
-      (effects (font (size 1.27 1.27)) hide)
-    )
-  )
-  (global_label "D3" (shape input) (at 231.14 101.6 180)
-    (effects (font (size 1.524 1.524)) (justify right))
-    (property "Intersheet References" "${INTERSHEET_REFS}" (id 0) (at 1.905 -3.81 0)
-      (effects (font (size 1.27 1.27)) hide)
+  (global_label "BROWSER_A" (shape input) (at 231.14 69.85 180)
+    (effects (font (size 1.016 1.016)) (justify right))
+    (property "Intersheet References" "${INTERSHEET_REFS}" (id 0) (at 220.4043 69.7865 0)
+      (effects (font (size 1.016 1.016)) (justify right) hide)
+    )
+  )
+  (global_label "GND" (shape input) (at 231.14 72.39 180)
+    (effects (font (size 1.016 1.016)) (justify right))
+    (property "Intersheet References" "${INTERSHEET_REFS}" (id 0) (at 226.1132 72.3265 0)
+      (effects (font (size 1.016 1.016)) (justify right) hide)
+    )
+  )
+  (global_label "BROWSER_B" (shape input) (at 231.14 74.93 180)
+    (effects (font (size 1.016 1.016)) (justify right))
+    (property "Intersheet References" "${INTERSHEET_REFS}" (id 0) (at 220.2591 74.8665 0)
+      (effects (font (size 1.016 1.016)) (justify right) hide)
+    )
+  )
+  (global_label "BROWSER_A" (shape input) (at 231.14 96.52 180)
+    (effects (font (size 1.016 1.016)) (justify right))
+    (property "Intersheet References" "${INTERSHEET_REFS}" (id 0) (at 220.4043 96.4565 0)
+      (effects (font (size 1.016 1.016)) (justify right) hide)
+    )
+  )
+  (global_label "GND" (shape input) (at 231.14 99.06 180)
+    (effects (font (size 1.016 1.016)) (justify right))
+    (property "Intersheet References" "${INTERSHEET_REFS}" (id 0) (at 226.1132 98.9965 0)
+      (effects (font (size 1.016 1.016)) (justify right) hide)
+    )
+  )
+  (global_label "BROWSER_B" (shape input) (at 231.14 101.6 180)
+    (effects (font (size 1.016 1.016)) (justify right))
+    (property "Intersheet References" "${INTERSHEET_REFS}" (id 0) (at 220.2591 101.5365 0)
+      (effects (font (size 1.016 1.016)) (justify right) hide)
     )
   )
   (global_label "SW_BROWSER_L" (shape input) (at 246.38 69.85 0)
-    (effects (font (size 1.524 1.524)) (justify left))
-    (property "Intersheet References" "${INTERSHEET_REFS}" (id 0) (at 266.7653 69.7548 0)
-      (effects (font (size 1.524 1.524)) (justify left) hide)
+    (effects (font (size 1.016 1.016)) (justify left))
+    (property "Intersheet References" "${INTERSHEET_REFS}" (id 0) (at 259.9702 69.7865 0)
+      (effects (font (size 1.016 1.016)) (justify left) hide)
+    )
+  )
+  (global_label "GND" (shape input) (at 246.38 74.93 0)
+    (effects (font (size 1.016 1.016)) (justify left))
+    (property "Intersheet References" "${INTERSHEET_REFS}" (id 0) (at 251.4068 74.8665 0)
+      (effects (font (size 1.016 1.016)) (justify left) hide)
     )
   )
   (global_label "SW_BROWSER_R" (shape input) (at 246.38 96.52 0)
-    (effects (font (size 1.524 1.524)) (justify left))
-    (property "Intersheet References" "${INTERSHEET_REFS}" (id 0) (at 267.0556 96.4248 0)
-      (effects (font (size 1.524 1.524)) (justify left) hide)
-    )
-  )
+    (effects (font (size 1.016 1.016)) (justify left))
+    (property "Intersheet References" "${INTERSHEET_REFS}" (id 0) (at 260.1637 96.4565 0)
+      (effects (font (size 1.016 1.016)) (justify left) hide)
+    )
+  )
+  (global_label "GND" (shape input) (at 246.38 101.6 0)
+    (effects (font (size 1.016 1.016)) (justify left))
+    (property "Intersheet References" "${INTERSHEET_REFS}" (id 0) (at 251.4068 101.5365 0)
+      (effects (font (size 1.016 1.016)) (justify left) hide)
+    )
+  )

Commit message: placed 3d model components
Parts:
- SW43, SW44: footprint Rotary_Encoder:RotaryEncoder_Alps_EC11E-Switch_Vertical_H20mm_CircularMountingHoles -> Library:RotaryEncoder_Alps_EC11E-Switch_Vertical_H20mm_CircularMountingHoles
Changed lines of the file:
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@@
     (property "Reference" "SW43" (id 0) (at 238.76 63.5 0))
     (property "Value" "BROWSER-L" (id 1) (at 238.76 66.04 0))
-    (property "Footprint" "Rotary_Encoder:RotaryEncoder_Alps_EC11E-Switch_Vertical_H20mm_CircularMountingHoles" (id 2) (at 234.95 68.326 0)
+    (property "Footprint" "Library:RotaryEncoder_Alps_EC11E-Switch_Vertical_H20mm_CircularMountingHoles" (id 2) (at 234.95 68.326 0)
       (effects (font (size 1.27 1.27)) hide)
     )
@@
     (property "Reference" "SW44" (id 0) (at 238.76 90.17 0))
     (property "Value" "BROWSER-R" (id 1) (at 238.76 92.71 0))
-    (property "Footprint" "Rotary_Encoder:RotaryEncoder_Alps_EC11E-Switch_Vertical_H20mm_CircularMountingHoles" (id 2) (at 234.95 94.996 0)
+    (property "Footprint" "Library:RotaryEncoder_Alps_EC11E-Switch_Vertical_H20mm_CircularMountingHoles" (id 2) (at 234.95 94.996 0)
       (effects (font (size 1.27 1.27)) hide)
     )
