File: PCB/Kicad/switchers.kicad_sch (KiCad schematic)
At the start: 44 parts, among them SW1 SWPADL1, SW10 SWPADR2, SW11 SWPADR3, SW12 SWPADR4, SW13 SWPADR5, SW14 SWPADR6, SW15 SWPADR7, SW16 SWPADR8, SW17 SWPLAYL, SW18 SWCUEL, SW19 SWSHIFTL, SW2 SWPADL2, SW20 SWSYNCL, SW21 SWRANGEL, SW22 SWFX1L, SW23 SWFX2L, SW24 SWFX3L, SW25 SWBR-PREVL, SW26 SWBR-BACKL, SW27 SWPLAYR, SW28 SWCUER, SW29 SWSHIFTR, SW3 SWPADL3, SW30 SWSYNCR, SW31 SWRANGER, SW32 SWFX1R, SW33 SWFX2R, SW34 SWFX3R, SW35 SWBR-PREVR, SW36 SWBR-BACKR, SW37 SWPCUEL1, SW38 SWPCUEL2, SW39 SWPCUEL3, SW4 SWPADL4, SW40 SWSEL1, SW41 SWSEL2, SW42 SWSEL3, SW43 BROWSER-L, SW44 BROWSER-R, SW5 SWPADL5, SW6 SWPADL6, SW7 SWPADL7, SW8 SWPADL8, SW9 SWPADR1

Commit message: sr wip
Parts:
- removed SW41: SWSEL2, Library:SW_PUSH_6mm_H5mm, symbol Switch:SW_Push
- removed SW42: SWSEL3, Library:SW_PUSH_6mm_H5mm, symbol Switch:SW_Push
Changed lines of the file:
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@@
-    (stroke (width 0) (type solid) (color 0 0 0 0))
-  )
-  (wire (pts (xy 168.91 97.79) (xy 166.37 97.79))
-    (stroke (width 0) (type solid) (color 0 0 0 0))
-  )
-  (wire (pts (xy 168.91 114.3) (xy 166.37 114.3))
     (stroke (width 0) (type solid) (color 0 0 0 0))
   )
@@
   )
   (global_label "SWSEL-L1" (shape input) (at 179.07 82.55 0)
-    (effects (font (size 1.016 1.016)) (justify left))
-    (property "Intersheet References" "${INTERSHEET_REFS}" (id 0) (at 0 0 0)
-      (effects (font (size 1.27 1.27)) hide)
-    )
-  )
-  (global_label "SWSEL-L2" (shape input) (at 179.07 97.79 0)
-    (effects (font (size 1.016 1.016)) (justify left))
-    (property "Intersheet References" "${INTERSHEET_REFS}" (id 0) (at 0 0 0)
-      (effects (font (size 1.27 1.27)) hide)
-    )
-  )
-  (global_label "SWSEL-L3" (shape input) (at 179.07 114.3 0)
     (effects (font (size 1.016 1.016)) (justify left))
     (property "Intersheet References" "${INTERSHEET_REFS}" (id 0) (at 0 0 0)
@@
     (pin "1")
   )
-  (symbol (lib_id "power:GND") (at 166.37 97.79 0) (unit 1)
-    (in_bom yes) (on_board yes)
-    (property "Reference" "#PWR0136" (id 0) (at 166.37 104.14 0)
-      (effects (font (size 1.27 1.27)) hide)
-    )
-    (property "Value" "GND" (id 1) (at 166.497 102.1842 0))
-    (property "Footprint" "" (id 2) (at 166.37 97.79 0)
-      (effects (font (size 1.27 1.27)) hide)
-    )
-    (property "Datasheet" "" (id 3) (at 166.37 97.79 0)
-      (effects (font (size 1.27 1.27)) hide)
-    )
-    (pin "1")
-  )
-  (symbol (lib_id "power:GND") (at 166.37 114.3 0) (unit 1)
-    (in_bom yes) (on_board yes)
-    (property "Reference" "#PWR0135" (id 0) (at 166.37 120.65 0)
-      (effects (font (size 1.27 1.27)) hide)
-    )
-    (property "Value" "GND" (id 1) (at 166.497 118.6942 0))
-    (property "Footprint" "" (id 2) (at 166.37 114.3 0)
-      (effects (font (size 1.27 1.27)) hide)
-    )
-    (property "Datasheet" "" (id 3) (at 166.37 114.3 0)
-      (effects (font (size 1.27 1.27)) hide)
-    )
-    (pin "1")
-  )
   (symbol (lib_id "Switch:SW_Push") (at 35.56 33.02 0) (unit 1)
     (in_bom yes) (on_board yes)
@@
       (effects (font (size 1.27 1.27)) hide)
     )
-    (pin "1")
-    (pin "2")
-  )
-  (symbol (lib_id "Switch:SW_Push") (at 173.99 97.79 0) (unit 1)
-    (in_bom yes) (on_board yes)
-    (property "Reference" "SW41" (id 0) (at 173.99 90.551 0))
-    (property "Value" "SWSEL2" (id 1) (at 173.99 92.8624 0))
-    (property "Footprint" "Library:SW_PUSH_6mm_H5mm" (id 2) (at 173.99 92.71 0)
-      (effects (font (size 1.27 1.27)) hide)
-    )
-    (property "Datasheet" "~" (id 3) (at 173.99 92.71 0)
-      (effects (font (size 1.27 1.27)) hide)
-    )
-    (pin "1")
-    (pin "2")
-  )
-  (symbol (lib_id "Switch:SW_Push") (at 173.99 114.3 0) (unit 1)
-    (in_bom yes) (on_board yes)
-    (property "Reference" "SW42" (id 0) (at 173.99 107.061 0))
-    (property "Value" "SWSEL3" (id 1) (at 173.99 109.3724 0))
-    (property "Footprint" "Library:SW_PUSH_6mm_H5mm" (id 2) (at 173.99 109.22 0)
-      (effects (font (size 1.27 1.27)) hide)
-    )
-    (property "Datasheet" "~" (id 3) (at 173.99 109.22 0)
-      (effects (font (size 1.27 1.27)) hide)
-    )

Commit message: routing
Parts:
- SW21: renamed from SW40; value SWSEL1 -> SWDECK
- renumbered SW38 to SW10, SW3 to SW11, SW19 to SW12, SW29 to SW13, SW39 to SW14, SW11 to SW15, SW43 to SW16, SW4 to SW17, SW12 to SW18, SW20 to SW19, SW9 to SW2, SW30 to SW20, SW5 to SW22, SW13 to SW23, SW21 to SW24, SW31 to SW25, SW44 to SW26, SW14 to SW27, SW6 to SW28, SW22 to SW29, SW17 to SW3, SW32 to SW30, SW15 to SW31, SW7 to SW32, SW23 to SW33, SW33 to SW34, SW16 to SW35, SW24 to SW36, SW34 to SW37, SW8 to SW38, SW25 to SW39, SW27 to SW4, SW35 to SW40, SW26 to SW41, SW36 to SW42, SW37 to SW5, SW2 to SW6, SW10 to SW7, SW18 to SW8, SW28 to SW9
Connections:
- net SWSEL-L1 renamed SW-DECK-SEL

Commit message: schematic updated
Parts:
- added SW43: SWLOOPL, Library:SW_PUSH_6mm_H8mm, symbol Switch:SW_Push
- added SW44: SWLOOPR, Library:SW_PUSH_6mm_H8mm, symbol Switch:SW_Push
- SW10, SW12, SW13, SW14, SW19, SW20, SW21, SW24, SW25, SW29, SW3, SW30, SW33, SW34, SW36, SW37, SW39, SW4, SW40, SW41, SW42, SW5, SW8, SW9: footprint Library:SW_PUSH_6mm_H5mm -> Library:SW_PUSH_6mm_H8mm
Connections:
- net GND: now also SW43.1, SW44.1
- net BROWSER_A renamed L_BROWSER_A
- net L_BROWSER_A: no longer SW26.A
- net BROWSER_B renamed L_BROWSER_B
- net L_BROWSER_B: no longer SW26.B
- new net R_BROWSER_A: SW26.A
- new net R_BROWSER_B: SW26.B
- new net SWLOOP-L: SW43.2
- new net SWLOOP-R: SW44.2

Commit message: SCHEMATIC FINISHED
Parts:
- removed SW1: SWPADL1, Library:sw-pad, symbol Switch:SW_Push
- removed SW10: SWPCUEL2, Library:SW_PUSH_6mm_H8mm, symbol Switch:SW_Push
- removed SW11: SWPADL3, Library:sw-pad, symbol Switch:SW_Push
- removed SW12: SWSHIFTL, Library:SW_PUSH_6mm_H8mm, symbol Switch:SW_Push
- removed SW13: SWSHIFTR, Library:SW_PUSH_6mm_H8mm, symbol Switch:SW_Push
- removed SW14: SWPCUEL3, Library:SW_PUSH_6mm_H8mm, symbol Switch:SW_Push
- removed SW15: SWPADR3, Library:sw-pad, symbol Switch:SW_Push
- removed SW16: BROWSER-L, Library:RotaryEncoder_Alps_EC11E-Switch_Vertical_H20mm_CircularMountingHoles, symbol Device:RotaryEncoder_Switch
- removed SW17: SWPADL4, Library:sw-pad, symbol Switch:SW_Push
- removed SW18: SWPADR4, Library:sw-pad, symbol Switch:SW_Push
- removed SW19: SWSYNCL, Library:SW_PUSH_6mm_H8mm, symbol Switch:SW_Push
- removed SW2: SWPADR1, Library:sw-pad, symbol Switch:SW_Push
- removed SW20: SWSYNCR, Library:SW_PUSH_6mm_H8mm, symbol Switch:SW_Push
- removed SW21: SWDECK, Library:SW_PUSH_6mm_H8mm, symbol Switch:SW_Push
- removed SW22: SWPADL5, Library:sw-pad, symbol Switch:SW_Push
- removed SW23: SWPADR5, Library:sw-pad, symbol Switch:SW_Push
- removed SW24: SWRANGEL, Library:SW_PUSH_6mm_H8mm, symbol Switch:SW_Push
- removed SW25: SWRANGER, Library:SW_PUSH_6mm_H8mm, symbol Switch:SW_Push
- removed SW26: BROWSER-R, Library:RotaryEncoder_Alps_EC11E-Switch_Vertical_H20mm_CircularMountingHoles, symbol Device:RotaryEncoder_Switch
- removed SW27: SWPADR6, Library:sw-pad, symbol Switch:SW_Push
- removed SW28: SWPADL6, Library:sw-pad, symbol Switch:SW_Push
- removed SW29: SWFX1L, Library:SW_PUSH_6mm_H8mm, symbol Switch:SW_Push
- removed SW3: SWPLAYL, Library:SW_PUSH_6mm_H8mm, symbol Switch:SW_Push
- removed SW30: SWFX1R, Library:SW_PUSH_6mm_H8mm, symbol Switch:SW_Push
- removed SW31: SWPADR7, Library:sw-pad, symbol Switch:SW_Push
- removed SW32: SWPADL7, Library:sw-pad, symbol Switch:SW_Push
- removed SW33: SWFX2L, Library:SW_PUSH_6mm_H8mm, symbol Switch:SW_Push
- removed SW34: SWFX2R, Library:SW_PUSH_6mm_H8mm, symbol Switch:SW_Push
- removed SW35: SWPADR8, Library:sw-pad, symbol Switch:SW_Push
- removed SW36: SWFX3L, Library:SW_PUSH_6mm_H8mm, symbol Switch:SW_Push
- removed SW37: SWFX3R, Library:SW_PUSH_6mm_H8mm, symbol Switch:SW_Push
- removed SW38: SWPADL8, Library:sw-pad, symbol Switch:SW_Push
- removed SW39: SWBR-PREVL, Library:SW_PUSH_6mm_H8mm, symbol Switch:SW_Push
- removed SW4: SWPLAYR, Library:SW_PUSH_6mm_H8mm, symbol Switch:SW_Push
- removed SW40: SWBR-PREVR, Library:SW_PUSH_6mm_H8mm, symbol Switch:SW_Push
- removed SW41: SWBR-BACKL, Library:SW_PUSH_6mm_H8mm, symbol Switch:SW_Push
- removed SW42: SWBR-BACKR, Library:SW_PUSH_6mm_H8mm, symbol Switch:SW_Push
- removed SW43: SWLOOPL, Library:SW_PUSH_6mm_H8mm, symbol Switch:SW_Push
- removed SW44: SWLOOPR, Library:SW_PUSH_6mm_H8mm, symbol Switch:SW_Push
- removed SW5: SWPCUEL1, Library:SW_PUSH_6mm_H8mm, symbol Switch:SW_Push
- removed SW6: SWPADL2, Library:sw-pad, symbol Switch:SW_Push
- removed SW7: SWPADR2, Library:sw-pad, symbol Switch:SW_Push
- removed SW8: SWCUEL, Library:SW_PUSH_6mm_H8mm, symbol Switch:SW_Push
- removed SW9: SWCUER, Library:SW_PUSH_6mm_H8mm, symbol Switch:SW_Push
