File: PCB/Kicad/shift-registers.kicad_sch (KiCad schematic)
At the start: 6 parts

Commit message: update elements WIP
Parts:
- renumbered U-LEDS to U-LEDS1, UVU-MASTER-L to UVU-MASTER-L1, UVU-MASTER-R to UVU-MASTER-R1
Connections:
- net LEDCUER: now also U-LEDS1.2 (QC); no longer U-LEDS1.6 (QG)
- net LEDHPL1: now also U-LEDS1.7 (QH); no longer U-LEDS1.1 (QB)
- net LEDHPL2: now also U-LEDS1.6 (QG); no longer U-LEDS1.2 (QC)
- net LEDHPL3: now also U-LEDS1.5 (QF); no longer U-LEDS1.3 (QD)
- net LEDPLAYL: now also U-LEDS1.3 (QD); no longer U-LEDS1.5 (QF)
- net LEDPLAYR: now also U-LEDS1.1 (QB); no longer U-LEDS1.7 (QH)
- net VUL1-0: now also UVU-LINE1.15 (QA); no longer UVU-LINE1.7 (QH)
- net VUL1-1: now also UVU-LINE1.1 (QB); no longer UVU-LINE1.6 (QG)
- net VUL1-2: now also UVU-LINE1.2 (QC); no longer UVU-LINE1.5 (QF)
- net VUL1-3: now also UVU-LINE1.3 (QD); no longer UVU-LINE1.4 (QE)
- net VUL1-4: now also UVU-LINE1.4 (QE); no longer UVU-LINE1.3 (QD)
- net VUL1-5: now also UVU-LINE1.5 (QF); no longer UVU-LINE1.2 (QC)
- net VUL1-6: now also UVU-LINE1.6 (QG); no longer UVU-LINE1.1 (QB)
- net VUL1-7: now also UVU-LINE1.7 (QH); no longer UVU-LINE1.15 (QA)
- net VUL2-0: now also UVU-LINE2.15 (QA); no longer UVU-LINE2.7 (QH)
- net VUL2-1: now also UVU-LINE2.1 (QB); no longer UVU-LINE2.6 (QG)
- net VUL2-2: now also UVU-LINE2.2 (QC); no longer UVU-LINE2.5 (QF)
- net VUL2-3: now also UVU-LINE2.3 (QD); no longer UVU-LINE2.4 (QE)
- net VUL2-4: now also UVU-LINE2.4 (QE); no longer UVU-LINE2.3 (QD)
- net VUL2-5: now also UVU-LINE2.5 (QF); no longer UVU-LINE2.2 (QC)
- net VUL2-6: now also UVU-LINE2.6 (QG); no longer UVU-LINE2.1 (QB)
- net VUL2-7: now also UVU-LINE2.7 (QH); no longer UVU-LINE2.15 (QA)
- net VUL3-0: now also UVU-LINE3.15 (QA); no longer UVU-LINE3.7 (QH)
- net VUL3-1: now also UVU-LINE3.1 (QB); no longer UVU-LINE3.6 (QG)
- net VUL3-2: now also UVU-LINE3.2 (QC); no longer UVU-LINE3.5 (QF)
- net VUL3-3: now also UVU-LINE3.3 (QD); no longer UVU-LINE3.4 (QE)
- net VUL3-4: now also UVU-LINE3.4 (QE); no longer UVU-LINE3.3 (QD)
- net VUL3-5: now also UVU-LINE3.5 (QF); no longer UVU-LINE3.2 (QC)
- net VUL3-6: now also UVU-LINE3.6 (QG); no longer UVU-LINE3.1 (QB)
- net VUL3-7: now also UVU-LINE3.7 (QH); no longer UVU-LINE3.15 (QA)
- net VUMASL-0: now also UVU-MASTER-L1.15 (QA); no longer UVU-MASTER-L1.7 (QH)
- net VUMASL-1: now also UVU-MASTER-L1.1 (QB); no longer UVU-MASTER-L1.6 (QG)
- net VUMASL-2: now also UVU-MASTER-L1.2 (QC); no longer UVU-MASTER-L1.5 (QF)
- net VUMASL-3: now also UVU-MASTER-L1.3 (QD); no longer UVU-MASTER-L1.4 (QE)
- net VUMASL-4: now also UVU-MASTER-L1.4 (QE); no longer UVU-MASTER-L1.3 (QD)
- net VUMASL-5: now also UVU-MASTER-L1.5 (QF); no longer UVU-MASTER-L1.2 (QC)
- net VUMASL-6: now also UVU-MASTER-L1.6 (QG); no longer UVU-MASTER-L1.1 (QB)
- net VUMASL-7: now also UVU-MASTER-L1.7 (QH); no longer UVU-MASTER-L1.15 (QA)
- net VUMASR-0: now also UVU-MASTER-R1.15 (QA); no longer UVU-MASTER-R1.7 (QH)
- net VUMASR-1: now also UVU-MASTER-R1.1 (QB); no longer UVU-MASTER-R1.6 (QG)
- net VUMASR-2: now also UVU-MASTER-R1.2 (QC); no longer UVU-MASTER-R1.5 (QF)
- net VUMASR-3: now also UVU-MASTER-R1.3 (QD); no longer UVU-MASTER-R1.4 (QE)
- net VUMASR-4: now also UVU-MASTER-R1.4 (QE); no longer UVU-MASTER-R1.3 (QD)
- net VUMASR-5: now also UVU-MASTER-R1.5 (QF); no longer UVU-MASTER-R1.2 (QC)
- net VUMASR-6: now also UVU-MASTER-R1.6 (QG); no longer UVU-MASTER-R1.1 (QB)
- net VUMASR-7: now also UVU-MASTER-R1.7 (QH); no longer UVU-MASTER-R1.15 (QA)
- no-connect marks 0 -> 1
Other:
- moved on the sheet: U-LEDS1, UVU-LINE1, UVU-LINE2, UVU-LINE3, UVU-MASTER-L1, UVU-MASTER-R1

Commit message: progress
Parts:
- U-LEDS1, UVU-LINE1, UVU-LINE2, UVU-LINE3, UVU-MASTER-L1, UVU-MASTER-R1: footprint (none) -> Package_DIP:DIP-16_W7.62mm_LongPads
Connections:
- net 595_OUT: no longer names the net of U-LEDS1.9 (QH')
- no-connect marks 1 -> 2
Changed lines of the file:
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@@
   (paper "A4")
   (no_connect (at 257.81 85.09))
+  (no_connect (at 257.81 107.95))
   (wire (pts (xy 52.07 107.95) (xy 63.5 107.95))
     (stroke (width 0) (type solid) (color 0 0 0 0))
@@
     (property "Intersheet References" "${INTERSHEET_REFS}" (id 0) (at 192.278 187.198 0)
       (effects (font (size 1.27 1.27)) hide)
-    )
-  )
-  (global_label "595_OUT" (shape input) (at 257.81 107.95 0)
-    (effects (font (size 1.016 1.016)) (justify left))
-    (property "Intersheet References" "${INTERSHEET_REFS}" (id 0) (at 266.3202 107.8865 0)
-      (effects (font (size 1.016 1.016)) (justify left) hide)
     )
   )
@@
     (property "Reference" "UVU-LINE1" (id 0) (at 41.91 72.39 0))
     (property "Value" "74HC595" (id 1) (at 40.64 102.87 0))
-    (property "Footprint" "" (id 2) (at 41.91 95.25 0)
+    (property "Footprint" "Package_DIP:DIP-16_W7.62mm_LongPads" (id 2) (at 41.91 95.25 0)
       (effects (font (size 1.27 1.27)) hide)
     )
@@
     (property "Reference" "UVU-LINE2" (id 0) (at 81.28 72.644 0))
     (property "Value" "74HC595" (id 1) (at 80.01 103.124 0))
-    (property "Footprint" "" (id 2) (at 81.28 95.25 0)
+    (property "Footprint" "Package_DIP:DIP-16_W7.62mm_LongPads" (id 2) (at 81.28 95.25 0)
       (effects (font (size 1.27 1.27)) hide)
     )
@@
     (property "Reference" "UVU-LINE3" (id 0) (at 123.19 72.39 0))
     (property "Value" "74HC595" (id 1) (at 121.92 102.87 0))
-    (property "Footprint" "" (id 2) (at 123.19 95.25 0)
+    (property "Footprint" "Package_DIP:DIP-16_W7.62mm_LongPads" (id 2) (at 123.19 95.25 0)
       (effects (font (size 1.27 1.27)) hide)
     )
@@
     (property "Reference" "UVU-MASTER-L1" (id 0) (at 161.29 72.39 0))
     (property "Value" "74HC595" (id 1) (at 160.02 102.87 0))
-    (property "Footprint" "" (id 2) (at 161.29 95.25 0)
+    (property "Footprint" "Package_DIP:DIP-16_W7.62mm_LongPads" (id 2) (at 161.29 95.25 0)
       (effects (font (size 1.27 1.27)) hide)
     )
@@
     (property "Reference" "UVU-MASTER-R1" (id 0) (at 200.66 72.39 0))
     (property "Value" "74HC595" (id 1) (at 199.39 102.87 0))
-    (property "Footprint" "" (id 2) (at 200.66 95.25 0)
+    (property "Footprint" "Package_DIP:DIP-16_W7.62mm_LongPads" (id 2) (at 200.66 95.25 0)
       (effects (font (size 1.27 1.27)) hide)
     )
@@
     (property "Reference" "U-LEDS1" (id 0) (at 247.65 72.39 0))
     (property "Value" "74HC595" (id 1) (at 246.38 102.87 0))
-    (property "Footprint" "" (id 2) (at 247.65 95.25 0)
-      (effects (font (size 1.27 1.27)) hide)
-    )
+    (property "Footprint" "Package_DIP:DIP-16_W7.62mm_LongPads" (id 2) (at 247.65 95.25 0)
+      (effects (font (size 1.27 1.27)) hide)
+    )

Commit message: Arduino mega retrofit WIP
Parts:
- U-LEDS1, UVU-LINE1, UVU-LINE2, UVU-LINE3, UVU-MASTER-L1, UVU-MASTER-R1: footprint Package_DIP:DIP-16_W7.62mm_LongPads -> Package_SO:SO-16_3.9x9.9mm_P1.27mm
Changed lines of the file:
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@@
     (property "Reference" "UVU-LINE1" (id 0) (at 41.91 72.39 0))
     (property "Value" "74HC595" (id 1) (at 40.64 102.87 0))
-    (property "Footprint" "Package_DIP:DIP-16_W7.62mm_LongPads" (id 2) (at 41.91 95.25 0)
+    (property "Footprint" "Package_SO:SO-16_3.9x9.9mm_P1.27mm" (id 2) (at 41.91 95.25 0)
       (effects (font (size 1.27 1.27)) hide)
     )
@@
     (property "Reference" "UVU-LINE2" (id 0) (at 81.28 72.644 0))
     (property "Value" "74HC595" (id 1) (at 80.01 103.124 0))
-    (property "Footprint" "Package_DIP:DIP-16_W7.62mm_LongPads" (id 2) (at 81.28 95.25 0)
+    (property "Footprint" "Package_SO:SO-16_3.9x9.9mm_P1.27mm" (id 2) (at 81.28 95.25 0)
       (effects (font (size 1.27 1.27)) hide)
     )
@@
     (property "Reference" "UVU-LINE3" (id 0) (at 123.19 72.39 0))
     (property "Value" "74HC595" (id 1) (at 121.92 102.87 0))
-    (property "Footprint" "Package_DIP:DIP-16_W7.62mm_LongPads" (id 2) (at 123.19 95.25 0)
+    (property "Footprint" "Package_SO:SO-16_3.9x9.9mm_P1.27mm" (id 2) (at 123.19 95.25 0)
       (effects (font (size 1.27 1.27)) hide)
     )
@@
     (property "Reference" "UVU-MASTER-L1" (id 0) (at 161.29 72.39 0))
     (property "Value" "74HC595" (id 1) (at 160.02 102.87 0))
-    (property "Footprint" "Package_DIP:DIP-16_W7.62mm_LongPads" (id 2) (at 161.29 95.25 0)
+    (property "Footprint" "Package_SO:SO-16_3.9x9.9mm_P1.27mm" (id 2) (at 161.29 95.25 0)
       (effects (font (size 1.27 1.27)) hide)
     )
@@
     (property "Reference" "UVU-MASTER-R1" (id 0) (at 200.66 72.39 0))
     (property "Value" "74HC595" (id 1) (at 199.39 102.87 0))
-    (property "Footprint" "Package_DIP:DIP-16_W7.62mm_LongPads" (id 2) (at 200.66 95.25 0)
+    (property "Footprint" "Package_SO:SO-16_3.9x9.9mm_P1.27mm" (id 2) (at 200.66 95.25 0)
       (effects (font (size 1.27 1.27)) hide)
     )
@@
     (property "Reference" "U-LEDS1" (id 0) (at 247.65 72.39 0))
     (property "Value" "74HC595" (id 1) (at 246.38 102.87 0))
-    (property "Footprint" "Package_DIP:DIP-16_W7.62mm_LongPads" (id 2) (at 247.65 95.25 0)
+    (property "Footprint" "Package_SO:SO-16_3.9x9.9mm_P1.27mm" (id 2) (at 247.65 95.25 0)
       (effects (font (size 1.27 1.27)) hide)
     )

Commit message: trillbar added
Connections:
- net D11 renamed SF-DATA
- net D12 renamed SF-CLOCK
- net D8 renamed SF-LATCH
Other:
- moved on the sheet: U-LEDS1, UVU-MASTER-L1, UVU-MASTER-R1

Commit message: board updated
Connections:
- net LEDCUEL: now also U-LEDS1.1 (QB); no longer U-LEDS1.4 (QE)
- net LEDCUER: now also U-LEDS1.7 (QH); no longer U-LEDS1.2 (QC)
- net LEDHPL1: now also U-LEDS1.3 (QD); no longer U-LEDS1.7 (QH)
- net LEDHPL2: now also U-LEDS1.4 (QE); no longer U-LEDS1.6 (QG)
- net LEDPLAYL: now also U-LEDS1.2 (QC); no longer U-LEDS1.3 (QD)
- net LEDPLAYR: now also U-LEDS1.6 (QG); no longer U-LEDS1.1 (QB)
- net SF-DATA: now also UVU-MASTER-R1.14 (SER); no longer UVU-LINE1.14 (SER)
- net at UVU-LINE1.9 (QH'): now also U-LEDS1.14 (SER); no longer UVU-LINE2.14 (SER)
- net at UVU-LINE2.9 (QH'): now also UVU-LINE1.14 (SER); no longer UVU-LINE3.14 (SER)
- net at UVU-LINE3.9 (QH'): now also UVU-LINE2.14 (SER); no longer UVU-MASTER-L1.14 (SER)
- net at UVU-MASTER-L1.9 (QH'): now also UVU-LINE3.14 (SER); no longer UVU-MASTER-R1.14 (SER)
- net at UVU-MASTER-R1.9 (QH'): now also UVU-MASTER-L1.14 (SER); no longer U-LEDS1.14 (SER)
Other:
- moved on the sheet: U-LEDS1, UVU-LINE1, UVU-LINE2, UVU-LINE3, UVU-MASTER-L1, UVU-MASTER-R1

Commit message: fixing 3dmodels
Parts:
- U-LEDS1, UVU-LINE1, UVU-LINE2, UVU-LINE3, UVU-MASTER-L1, UVU-MASTER-R1: footprint Package_SO:SO-16_3.9x9.9mm_P1.27mm -> Library:SO-16_3.9x9.9mm_P1.27mm
Changed lines of the file:
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@@
     (property "Reference" "UVU-MASTER-R1" (id 0) (at 36.83 72.39 0))
     (property "Value" "74HC595" (id 1) (at 35.56 102.87 0))
-    (property "Footprint" "Package_SO:SO-16_3.9x9.9mm_P1.27mm" (id 2) (at 36.83 95.25 0)
+    (property "Footprint" "Library:SO-16_3.9x9.9mm_P1.27mm" (id 2) (at 36.83 95.25 0)
       (effects (font (size 1.27 1.27)) hide)
     )
@@
     (property "Reference" "UVU-MASTER-L1" (id 0) (at 83.185 73.025 0))
     (property "Value" "74HC595" (id 1) (at 81.915 103.505 0))
-    (property "Footprint" "Package_SO:SO-16_3.9x9.9mm_P1.27mm" (id 2) (at 83.185 95.885 0)
+    (property "Footprint" "Library:SO-16_3.9x9.9mm_P1.27mm" (id 2) (at 83.185 95.885 0)
       (effects (font (size 1.27 1.27)) hide)
     )
@@
     (property "Reference" "UVU-LINE3" (id 0) (at 128.27 73.025 0))
     (property "Value" "74HC595" (id 1) (at 127 103.505 0))
-    (property "Footprint" "Package_SO:SO-16_3.9x9.9mm_P1.27mm" (id 2) (at 128.27 95.885 0)
+    (property "Footprint" "Library:SO-16_3.9x9.9mm_P1.27mm" (id 2) (at 128.27 95.885 0)
       (effects (font (size 1.27 1.27)) hide)
     )
@@
     (property "Reference" "UVU-LINE2" (id 0) (at 174.625 73.279 0))
     (property "Value" "74HC595" (id 1) (at 173.355 103.759 0))
-    (property "Footprint" "Package_SO:SO-16_3.9x9.9mm_P1.27mm" (id 2) (at 174.625 95.885 0)
+    (property "Footprint" "Library:SO-16_3.9x9.9mm_P1.27mm" (id 2) (at 174.625 95.885 0)
       (effects (font (size 1.27 1.27)) hide)
     )
@@
     (property "Reference" "UVU-LINE1" (id 0) (at 217.805 74.295 0))
     (property "Value" "74HC595" (id 1) (at 216.535 104.775 0))
-    (property "Footprint" "Package_SO:SO-16_3.9x9.9mm_P1.27mm" (id 2) (at 217.805 97.155 0)
+    (property "Footprint" "Library:SO-16_3.9x9.9mm_P1.27mm" (id 2) (at 217.805 97.155 0)
       (effects (font (size 1.27 1.27)) hide)
     )
@@
     (property "Reference" "U-LEDS1" (id 0) (at 259.08 74.295 0))
     (property "Value" "74HC595" (id 1) (at 257.81 104.775 0))
-    (property "Footprint" "Package_SO:SO-16_3.9x9.9mm_P1.27mm" (id 2) (at 259.08 97.155 0)
+    (property "Footprint" "Library:SO-16_3.9x9.9mm_P1.27mm" (id 2) (at 259.08 97.155 0)
       (effects (font (size 1.27 1.27)) hide)
     )

Commit message: sr wip
Parts:
- added U-LEDSR1: 74HC595, Library:SO-16_3.9x9.9mm_P1.27mm, symbol 74xx:74HC595
Connections:
- net +5V: now also U-LEDSR1.16 (VCC)
- net GND: now also U-LEDSR1.13 (~OE), U-LEDSR1.8 (GND)
- net LEDCUER: now also U-LEDSR1.3 (QD); no longer U-LEDS1.7 (QH)
- net LEDHPL1: now also U-LEDS1.6 (QG); no longer U-LEDS1.3 (QD)
- net LEDHPL2: now also U-LEDS1.7 (QH); no longer U-LEDS1.4 (QE)
- net LEDHPL3: now also U-LEDSR1.1 (QB); no longer U-LEDS1.5 (QF)
- net LEDPLAYR: now also U-LEDSR1.2 (QC); no longer U-LEDS1.6 (QG)
- net SF-CLOCK: now also U-LEDSR1.11 (SRCLK)
- net SF-LATCH: now also U-LEDSR1.12 (RCLK)
- net VCC: now also U-LEDSR1.10 (~SRCLR)
- net at UVU-LINE1.9 (QH'): no longer U-LEDS1.14 (SER)
- net SF-DATA renamed VU-SF-DATA
- new net: U-LEDS1.14 (SER), U-LEDSR1.9 (QH')
- new net BTNLED-SF-DATA: U-LEDSR1.14 (SER)
- new net LEDFX1L: U-LEDS1.3 (QD)
- new net LEDFX1R: U-LEDSR1.6 (QG)
- new net LEDFX2L: U-LEDS1.4 (QE)
- new net LEDFX2R: U-LEDSR1.5 (QF)
- new net LEDFX3L: U-LEDS1.5 (QF)
- new net LEDFX3R: U-LEDSR1.4 (QE)
- no-connect marks 2 -> 4
Other:
- moved on the sheet: U-LEDS1, UVU-LINE1, UVU-LINE2, UVU-LINE3, UVU-MASTER-L1, UVU-MASTER-R1
