File: PCB/Kicad/Mixduino.kicad_pcb (KiCad board)
At the start: 2 copper layers, 360 x 260 mm, 206 parts, among them SW1 SWPADL1, SW10 SWPADR2, SW11 SWPADR3, SW12 SWPADR4, SW13 SWPADR5, SW14 SWPADR6, SW15 SWPADR7, SW16 SWPADR8, SW17 SWPLAYL, SW18 SWCUEL, SW19 SWSHIFTL, SW2 SWPADL2, SW20 SWSYNCL, SW21 SWRANGEL, SW22 SWFX1L, SW23 SWFX2L, SW24 SWFX3L, SW25 SWBR-PREVL, SW26 SWBR-BACKL, SW27 SWPLAYR, SW28 SWCUER, SW29 SWSHIFTR, SW3 SWPADL3, SW30 SWSYNCR, SW31 SWRANGER, SW32 SWFX1R, SW33 SWFX2R, SW34 SWFX3R, SW35 SWBR-PREVR, SW36 SWBR-BACKR, SW37 SWPCUEL1, SW38 SWPCUEL2, SW39 SWPCUEL3, SW4 SWPADL4, SW40 SWSEL1, SW43 BROWSER-L, SW44 BROWSER-R, SW5 SWPADL5, SW6 SWPADL6, SW7 SWPADL7, SW8 SWPADL8, SW9 SWPADR1

Commit message: routing
Parts:
- removed BCUELD1, BCUERD1, BHPL1D1, BHPL2D1, FX2LD1, FX2RD1, FX3LD1, FX3RD1: LED_ALT, Library:LED_YELLOW
- removed BCUELR1, BCUERR1, BHPL1R1, BHPL2R1, BPLAYLR1, BPLAYRR1, FX1LR1, FX1RR1, FX2LR1, FX2RR1, FX3LR1, FX3RR1, PADL-IN-R1, PADR-IN-R1, VUL1R1, VUL1R2, VUL1R3, VUL1R4, VUL1R5, VUL1R6, VUL1R7, VUL1R8, VUL2R1, VUL2R2, VUL2R3, VUL2R4, VUL2R5, VUL2R6, VUL2R7, VUL2R8, VUL3R1, VUL3R2, VUL3R3, VUL3R4, VUL3R5, VUL3R6, VUL3R7, VUL3R8, VUMASLR1, VUMASLR2, VUMASLR3, VUMASLR4, VUMASLR5, VUMASLR6, VUMASLR7, VUMASLR8, VUMASRR1, VUMASRR2, VUMASRR3, VUMASRR4, VUMASRR5, VUMASRR6, VUMASRR7, VUMASRR8: R_Small, Library:R_1206_3216Metric_Pad1.30x1.75mm_HandSolder
- removed BPLAYLD1, BPLAYRD1, FX1LD1, FX1RD1: LED_ALT, Library:LED_GREEN
- removed PADL-D1, PADL-D2, PADL-D3, PADL-D4, PADL-D5, PADL-D6, PADL-D7, PADL-D8, PADR-D1, PADR-D2, PADR-D3, PADR-D4, PADR-D5, PADR-D6, PADR-D7, PADR-D8: WS2812B, Library:LED_WS2812B_PLCC4_5.0x5.0mm_P3.2mm
- removed SW43: BROWSER-L, Library:RotaryEncoder_Alps_EC11E-Switch_Vertical_H20mm_CircularMountingHoles
- removed SW44: BROWSER-R, Library:RotaryEncoder_Alps_EC11E-Switch_Vertical_H20mm_CircularMountingHoles
- removed VUL1D1, VUL1D2, VUL1D3, VUL1D4, VUL1D5, VUL2D1, VUL2D2, VUL2D3, VUL2D4, VUL2D5, VUL3D1, VUL3D2, VUL3D3, VUL3D4, VUL3D5, VUMASLD1, VUMASLD2, VUMASLD3, VUMASLD4, VUMASLD5, VUMASRD1, VUMASRD2, VUMASRD3, VUMASRD4, VUMASRD5: LED_Filled, Library:LED_GREEN
- removed VUL1D6, VUL1D7, VUL2D6, VUL2D7, VUL3D6, VUL3D7, VUMASLD6, VUMASLD7, VUMASRD6, VUMASRD7: LED_Filled, Library:LED_YELLOW
- removed VUL1D8, VUL2D8, VUL3D8, VUMASLD8, VUMASRD8: LED_Filled, Library:LED_RED
- added C1: 100nF, Capacitor_SMD:C_1206_3216Metric_Pad1.33x1.80mm_HandSolder, B.Cu at (439.2, 240.0)
- added C10: 100nF, Capacitor_SMD:C_1206_3216Metric_Pad1.33x1.80mm_HandSolder, B.Cu at (387.5, 181.7)
- added C11: 100nF, Capacitor_SMD:C_1206_3216Metric_Pad1.33x1.80mm_HandSolder, B.Cu at (136.9, 162.1)
- added C12: 100nF, Capacitor_SMD:C_1206_3216Metric_Pad1.33x1.80mm_HandSolder, B.Cu at (137.0, 187.1)
- added C13: 100nF, Capacitor_SMD:C_1206_3216Metric_Pad1.33x1.80mm_HandSolder, B.Cu at (437.4, 156.1)
- added C14: 100nF, Capacitor_SMD:C_1206_3216Metric_Pad1.33x1.80mm_HandSolder, B.Cu at (348.8, 193.9)
- added C15: 100nF, Capacitor_SMD:C_1206_3216Metric_Pad1.33x1.80mm_HandSolder, B.Cu at (212.1, 162.1)
- added C16: 100nF, Capacitor_SMD:C_1206_3216Metric_Pad1.33x1.80mm_HandSolder, B.Cu at (459.0, 179.8)
- added C17: 100nF, Capacitor_SMD:C_1206_3216Metric_Pad1.33x1.80mm_HandSolder, B.Cu at (437.4, 181.3)
- added C18: 100nF, Capacitor_SMD:C_1206_3216Metric_Pad1.33x1.80mm_HandSolder, B.Cu at (186.9, 187.2)
- added C19: 100nF, Capacitor_SMD:C_1206_3216Metric_Pad1.33x1.80mm_HandSolder, B.Cu at (462.5, 156.2)
- added C2: 100nF, Capacitor_SMD:C_1206_3216Metric_Pad1.33x1.80mm_HandSolder, B.Cu at (412.3, 155.9)
- added C20: 100nF, Capacitor_SMD:C_1206_3216Metric_Pad1.33x1.80mm_HandSolder, B.Cu at (162.1, 187.2)
- added C21: 100nF, Capacitor_SMD:C_1206_3216Metric_Pad1.33x1.80mm_HandSolder, B.Cu at (439.2, 254.3)
- added C3: 100nF, Capacitor_SMD:C_1206_3216Metric_Pad1.33x1.80mm_HandSolder, B.Cu at (412.4, 181.0)
- added C4: 100nF, Capacitor_SMD:C_1206_3216Metric_Pad1.33x1.80mm_HandSolder, B.Cu at (162.1, 162.1)
- added C5: 100nF, Capacitor_SMD:C_1206_3216Metric_Pad1.33x1.80mm_HandSolder, B.Cu at (212.1, 187.2)
- added C6: 100nF, Capacitor_SMD:C_1206_3216Metric_Pad1.33x1.80mm_HandSolder, B.Cu at (187.2, 162.1)
- added C7: 100nF, Capacitor_SMD:C_1206_3216Metric_Pad1.33x1.80mm_HandSolder, B.Cu at (387.4, 155.9)
- added C8: 100nF, Capacitor_SMD:C_1206_3216Metric_Pad1.33x1.80mm_HandSolder, B.Cu at (189.5, 240.8)
- added C9: 100nF, Capacitor_SMD:C_1206_3216Metric_Pad1.33x1.80mm_HandSolder, B.Cu at (189.5, 255.3)
- added D1: VUL1D1, Library:LED_GREEN, F.Cu at (262.3, 170.0)
- added D10: LCUE-D, Library:LED_YELLOW, F.Cu at (141.9, 259.1)
- added D11: LFX1-D, Library:LED_GREEN, F.Cu at (136.0, 69.1)
- added D12: LFX2-D, Library:LED_YELLOW, F.Cu at (178.2, 69.2)
- added D13: LFX3-D, Library:LED_YELLOW, F.Cu at (219.0, 69.1)
- added D14: VUL2D1, Library:LED_GREEN, F.Cu at (296.5, 170.0)
- added D15: VUL2D2, Library:LED_GREEN, F.Cu at (296.6, 165.0)
- added D16: VUL2D3, Library:LED_GREEN, F.Cu at (296.6, 160.0)
- added D17: VUL2D4, Library:LED_GREEN, F.Cu at (296.5, 154.9)
- added D18: VUL2D5, Library:LED_GREEN, F.Cu at (296.6, 149.9)
- added D19: VUL2D6, Library:LED_YELLOW, F.Cu at (296.5, 145.0)
- added D2: VUL1D2, Library:LED_GREEN, F.Cu at (262.2, 165.0)
- added D20: VUL2D7, Library:LED_YELLOW, F.Cu at (296.4, 140.0)
- added D21: VUL2D8, Library:LED_RED, F.Cu at (296.5, 134.9)
- added D22: L1HP-D, Library:LED_YELLOW, F.Cu at (252.9, 228.7)
- added D24: L3HP-D, Library:LED_YELLOW, F.Cu at (321.1, 228.9)
- added D25: RPLAY-D, Library:LED_GREEN, F.Cu at (391.7, 289.6)
- added D26: RCUE-D, Library:LED_YELLOW, F.Cu at (391.7, 259.8)
- added D27: RFX1-D, Library:LED_GREEN, F.Cu at (386.1, 66.3)
- added D28: RFX2-D, Library:LED_YELLOW, F.Cu at (427.6, 66.6)
- added D29: RFX3-D, Library:LED_YELLOW, F.Cu at (468.7, 66.6)
- added D3: VUL1D3, Library:LED_GREEN, F.Cu at (262.2, 160.0)
- added D30: VUL3D1, Library:LED_GREEN, F.Cu at (330.5, 169.9)
- added D31: VUL3D2, Library:LED_GREEN, F.Cu at (330.6, 164.9)
- added D32: VUL3D3, Library:LED_GREEN, F.Cu at (330.6, 159.9)
- added D33: VUL3D4, Library:LED_GREEN, F.Cu at (330.6, 154.9)
- added D34: VUL3D5, Library:LED_GREEN, F.Cu at (330.5, 149.9)
- added D35: VUL3D6, Library:LED_YELLOW, F.Cu at (330.5, 144.9)
- added D36: VUL3D7, Library:LED_YELLOW, F.Cu at (330.5, 139.9)
- added D37: VUL3D8, Library:LED_RED, F.Cu at (330.5, 134.9)
- added D38: VUMASLD1, Library:LED_GREEN, F.Cu at (344.3, 119.5)
- added D39: VUMASLD2, Library:LED_GREEN, F.Cu at (344.3, 114.5)
- added D4: VUL1D4, Library:LED_GREEN, F.Cu at (262.3, 155.0)
- added D40: VUMASLD3, Library:LED_GREEN, F.Cu at (344.3, 109.5)
- added D41: VUMASLD4, Library:LED_GREEN, F.Cu at (344.2, 104.5)
- added D42: VUMASLD5, Library:LED_GREEN, F.Cu at (344.3, 99.5)
- added D43: VUMASLD6, Library:LED_YELLOW, F.Cu at (344.3, 94.5)
- added D44: VUMASLD7, Library:LED_YELLOW, F.Cu at (344.2, 89.5)
- added D45: VUMASLD8, Library:LED_RED, F.Cu at (344.2, 84.5)
- added D46: VUMASRD1, Library:LED_GREEN, F.Cu at (356.3, 119.5)
- added D47: VUMASRD2, Library:LED_GREEN, F.Cu at (356.2, 114.5)
- added D48: VUMASRD3, Library:LED_GREEN, F.Cu at (356.2, 109.5)
- added D49: VUMASRD4, Library:LED_GREEN, F.Cu at (356.2, 104.5)
- added D5: VUL1D5, Library:LED_GREEN, F.Cu at (262.3, 150.0)
- added D50: VUMASRD5, Library:LED_GREEN, F.Cu at (356.2, 99.5)
- added D51: VUMASRD6, Library:LED_YELLOW, F.Cu at (356.2, 94.5)
- added D52: VUMASRD7, Library:LED_YELLOW, F.Cu at (356.2, 89.5)
- added D53: VUMASRD8, Library:LED_RED, F.Cu at (356.2, 84.5)
- added D6: VUL1D6, Library:LED_YELLOW, F.Cu at (262.3, 145.0)
- added D7: VUL1D7, Library:LED_YELLOW, F.Cu at (262.2, 140.0)
- added D8: VUL1D8, Library:LED_RED, F.Cu at (262.2, 135.0)
- added D9: LPLAY-D, Library:LED_GREEN, F.Cu at (141.8, 289.1)
- added NP1: PADL-D1, Library:LED_WS2812B_PLCC4_5.0x5.0mm_P3.2mm, F.Cu at (137.0, 162.1)
- added NP10: L-SYNC-D, Library:LED_WS2812B_PLCC4_5.0x5.0mm_P3.2mm, F.Cu at (189.4, 247.7)
- added NP11: PADR-D8, Library:LED_WS2812B_PLCC4_5.0x5.0mm_P3.2mm, F.Cu at (462.5, 187.1)
- added NP12: PADR-D7, Library:LED_WS2812B_PLCC4_5.0x5.0mm_P3.2mm, F.Cu at (437.5, 187.1)
- added NP13: PADR-D6, Library:LED_WS2812B_PLCC4_5.0x5.0mm_P3.2mm, F.Cu at (412.5, 187.1)
- added NP14: PADR-D5, Library:LED_WS2812B_PLCC4_5.0x5.0mm_P3.2mm, F.Cu at (387.5, 187.1)
- added NP15: PADR-D4, Library:LED_WS2812B_PLCC4_5.0x5.0mm_P3.2mm, F.Cu at (462.5, 162.1)
- added NP16: PADR-D3, Library:LED_WS2812B_PLCC4_5.0x5.0mm_P3.2mm, F.Cu at (437.5, 162.1)
- added NP17: PADR-D2, Library:LED_WS2812B_PLCC4_5.0x5.0mm_P3.2mm, F.Cu at (412.5, 162.1)
- added NP18: PADR-D1, Library:LED_WS2812B_PLCC4_5.0x5.0mm_P3.2mm, F.Cu at (387.5, 162.1)
- added NP19: DECK-SWITCHER-D, Library:LED_WS2812B_PLCC4_5.0x5.0mm_P3.2mm, F.Cu at (348.6, 199.7)
- added NP2: PADL-D2, Library:LED_WS2812B_PLCC4_5.0x5.0mm_P3.2mm, F.Cu at (162.0, 162.1)
- added NP20: R-RNG-D, Library:LED_WS2812B_PLCC4_5.0x5.0mm_P3.2mm, F.Cu at (439.2, 233.7)
- added NP21: R-SYNC-D, Library:LED_WS2812B_PLCC4_5.0x5.0mm_P3.2mm, F.Cu at (439.3, 247.9)
- added NP3: PADL-D3, Library:LED_WS2812B_PLCC4_5.0x5.0mm_P3.2mm, F.Cu at (187.0, 162.1)
- added NP4: PADL-D4, Library:LED_WS2812B_PLCC4_5.0x5.0mm_P3.2mm, F.Cu at (212.0, 162.1)
- added NP5: PADL-D5, Library:LED_WS2812B_PLCC4_5.0x5.0mm_P3.2mm, F.Cu at (137.0, 187.1)
- added NP6: PADL-D6, Library:LED_WS2812B_PLCC4_5.0x5.0mm_P3.2mm, F.Cu at (162.0, 187.1)
- added NP7: PADL-D7, Library:LED_WS2812B_PLCC4_5.0x5.0mm_P3.2mm, F.Cu at (187.0, 187.1)
- added NP8: PADL-D8, Library:LED_WS2812B_PLCC4_5.0x5.0mm_P3.2mm, F.Cu at (212.0, 187.1)
- added NP9: L-RNG-D, Library:LED_WS2812B_PLCC4_5.0x5.0mm_P3.2mm, F.Cu at (189.4, 233.8)
- added NPR1: L-NP-SIG_R, Library:R_1206_3216Metric_Pad1.30x1.75mm_HandSolder, B.Cu at (142.1, 145.8)
- added NPR2: R-NP-SIG_R, Library:R_1206_3216Metric_Pad1.30x1.75mm_HandSolder, B.Cu at (466.4, 177.6)
- added R1: VUL1R1, Library:R_1206_3216Metric_Pad1.30x1.75mm_HandSolder, B.Cu at (266.6, 169.9)
- added R10: LCUE-R, Library:R_1206_3216Metric_Pad1.30x1.75mm_HandSolder, B.Cu at (143.5, 263.1)
- added R11: LFX1R, Library:R_1206_3216Metric_Pad1.30x1.75mm_HandSolder, B.Cu at (140.2, 67.8)
- added R12: LFX2R, Library:R_1206_3216Metric_Pad1.30x1.75mm_HandSolder, B.Cu at (182.1, 67.8)
- added R13: LFX3R, Library:R_1206_3216Metric_Pad1.30x1.75mm_HandSolder, B.Cu at (223.0, 67.8)
- added R14: VUL2R1, Library:R_1206_3216Metric_Pad1.30x1.75mm_HandSolder, B.Cu at (301.0, 169.9)
- added R15: VUL2R2, Library:R_1206_3216Metric_Pad1.30x1.75mm_HandSolder, B.Cu at (301.0, 165.1)
- added R16: VUL2R3, Library:R_1206_3216Metric_Pad1.30x1.75mm_HandSolder, B.Cu at (301.0, 160.0)
- added R17: VUL2R4, Library:R_1206_3216Metric_Pad1.30x1.75mm_HandSolder, B.Cu at (301.0, 154.9)
- added R18: VUL2R5, Library:R_1206_3216Metric_Pad1.30x1.75mm_HandSolder, B.Cu at (301.0, 149.9)
- added R19: VUL2R6, Library:R_1206_3216Metric_Pad1.30x1.75mm_HandSolder, B.Cu at (301.0, 145.0)
- added R2: VUL1R2, Library:R_1206_3216Metric_Pad1.30x1.75mm_HandSolder, B.Cu at (266.6, 165.0)
- added R20: VUL2R7, Library:R_1206_3216Metric_Pad1.30x1.75mm_HandSolder, B.Cu at (301.0, 140.0)
- added R21: VUL2R8, Library:R_1206_3216Metric_Pad1.30x1.75mm_HandSolder, B.Cu at (301.0, 134.9)
- added R22: L1HP-R, Library:R_1206_3216Metric_Pad1.30x1.75mm_HandSolder, B.Cu at (256.3, 227.3)
- added R24: L3HP-R, Library:R_1206_3216Metric_Pad1.30x1.75mm_HandSolder, B.Cu at (324.6, 227.8)
- added R25: RPLAY-R, Library:R_1206_3216Metric_Pad1.30x1.75mm_HandSolder, B.Cu at (393.2, 293.9)
- added R26: RCUE-R, Library:R_1206_3216Metric_Pad1.30x1.75mm_HandSolder, B.Cu at (393.1, 263.8)
- added R27: RFX1-R, Library:R_1206_3216Metric_Pad1.30x1.75mm_HandSolder, B.Cu at (389.4, 67.8)
- added R28: RFX2-R, Library:R_1206_3216Metric_Pad1.30x1.75mm_HandSolder, B.Cu at (431.0, 67.8)
- added R29: RFX3-R, Library:R_1206_3216Metric_Pad1.30x1.75mm_HandSolder, B.Cu at (471.9, 68.1)
- added R3: VUL1R3, Library:R_1206_3216Metric_Pad1.30x1.75mm_HandSolder, B.Cu at (266.6, 160.0)
- added R30: VUL3R1, Library:R_1206_3216Metric_Pad1.30x1.75mm_HandSolder, B.Cu at (335.0, 169.9)
- added R31: VUL3R2, Library:R_1206_3216Metric_Pad1.30x1.75mm_HandSolder, B.Cu at (335.0, 164.8)
- added R32: VUL3R3, Library:R_1206_3216Metric_Pad1.30x1.75mm_HandSolder, B.Cu at (335.0, 160.0)
- added R33: VUL3R4, Library:R_1206_3216Metric_Pad1.30x1.75mm_HandSolder, B.Cu at (335.0, 154.9)
- added R34: VUL3R5, Library:R_1206_3216Metric_Pad1.30x1.75mm_HandSolder, B.Cu at (335.0, 149.9)
- added R35: VUL3R6, Library:R_1206_3216Metric_Pad1.30x1.75mm_HandSolder, B.Cu at (335.0, 144.8)
- added R36: VUL3R7, Library:R_1206_3216Metric_Pad1.30x1.75mm_HandSolder, B.Cu at (335.0, 139.7)
- added R37: VUL3R8, Library:R_1206_3216Metric_Pad1.30x1.75mm_HandSolder, B.Cu at (335.0, 134.9)
- added R38: VUMASLR1, Library:R_1206_3216Metric_Pad1.30x1.75mm_HandSolder, B.Cu at (348.2, 119.6)
- added R39: VUMASLR2, Library:R_1206_3216Metric_Pad1.30x1.75mm_HandSolder, B.Cu at (348.2, 114.6)
- added R4: VUL1R4, Library:R_1206_3216Metric_Pad1.30x1.75mm_HandSolder, B.Cu at (266.5, 155.0)
- added R40: VUMASLR3, Library:R_1206_3216Metric_Pad1.30x1.75mm_HandSolder, B.Cu at (348.2, 109.5)
- added R41: VUMASLR4, Library:R_1206_3216Metric_Pad1.30x1.75mm_HandSolder, B.Cu at (348.2, 104.4)
- added R42: VUMASLR5, Library:R_1206_3216Metric_Pad1.30x1.75mm_HandSolder, B.Cu at (348.2, 99.3)
- added R43: VUMASLR6, Library:R_1206_3216Metric_Pad1.30x1.75mm_HandSolder, B.Cu at (348.2, 94.5)
- added R44: VUMASLR7, Library:R_1206_3216Metric_Pad1.30x1.75mm_HandSolder, B.Cu at (348.2, 89.7)
- added R45: VUMASLR8, Library:R_1206_3216Metric_Pad1.30x1.75mm_HandSolder, B.Cu at (348.2, 84.6)
- added R46: VUMASRR1, Library:R_1206_3216Metric_Pad1.30x1.75mm_HandSolder, B.Cu at (360.5, 119.6)
- added R47: VUMASRR2, Library:R_1206_3216Metric_Pad1.30x1.75mm_HandSolder, B.Cu at (360.5, 114.6)
- added R48: VUMASRR3, Library:R_1206_3216Metric_Pad1.30x1.75mm_HandSolder, B.Cu at (360.5, 109.5)
- added R49: VUMASRR4, Library:R_1206_3216Metric_Pad1.30x1.75mm_HandSolder, B.Cu at (360.4, 104.4)
- added R5: VUL1R5, Library:R_1206_3216Metric_Pad1.30x1.75mm_HandSolder, B.Cu at (266.5, 150.0)
- added R50: VUMASRR5, Library:R_1206_3216Metric_Pad1.30x1.75mm_HandSolder, B.Cu at (360.4, 99.3)
- added R51: VUMASRR6, Library:R_1206_3216Metric_Pad1.30x1.75mm_HandSolder, B.Cu at (360.4, 94.5)
- added R52: VUMASRR7, Library:R_1206_3216Metric_Pad1.30x1.75mm_HandSolder, B.Cu at (360.4, 89.4)
- added R53: VUMASRR8, Library:R_1206_3216Metric_Pad1.30x1.75mm_HandSolder, B.Cu at (360.4, 84.6)
- added R6: VUL1R6, Library:R_1206_3216Metric_Pad1.30x1.75mm_HandSolder, B.Cu at (266.5, 144.9)
- added R7: VUL1R7, Library:R_1206_3216Metric_Pad1.30x1.75mm_HandSolder, B.Cu at (266.6, 140.0)
- added R8: VUL1R8, Library:R_1206_3216Metric_Pad1.30x1.75mm_HandSolder, B.Cu at (266.4, 135.0)
- added R9: LPLAY-R, Library:R_1206_3216Metric_Pad1.30x1.75mm_HandSolder, B.Cu at (143.3, 292.9)
- added SW41: SWBR-BACKL, Library:SW_PUSH_6mm_H5mm, F.Cu at (159.8, 117.3)
- added SW42: SWBR-BACKR, Library:SW_PUSH_6mm_H5mm, F.Cu at (409.8, 117.2)
- D23: value LED_ALT -> L2HP-D
- R23: value R_Small -> L2HP-R
- RV10: value PFX1L -> MIDL2
- RV11: value PFX1R -> TREL2
- RV12: value PVOL-HP -> GAINL2
- RV13: value BASL1 -> FADERL3; footprint Library:Potentiometer_Bourns_PTV09A-1_Single_Vertical -> Library:fader-L60
- RV14: value BASL2 -> FILTERL3
- RV16: value PFX2L -> MIDL3
- RV17: value PFX2R -> TREL3
- RV18: value PMASTER -> GAINL3
- RV19: value MIDL1 -> PITCH-L; footprint Library:Potentiometer_Bourns_PTV09A-1_Single_Vertical -> Library:fader-L75
- RV2: value FADERL2 -> FILTERL1; footprint Library:fader-L60 -> Library:Potentiometer_Bourns_PTV09A-1_Single_Vertical
- RV20: value MIDL2 -> PFX1L
- RV21: value MIDL3 -> PFX2L
- RV23: value PFX3R -> PITH-R; footprint Library:Potentiometer_Bourns_PTV09A-1_Single_Vertical -> Library:fader-L75
- RV24: value TREL1 -> PFX1R
- RV25: value TREL2 -> PFX2R
- RV26: value TREL3 -> PFX3R
- RV27: value GAINL1 -> PMIX-HP
- RV28: value GAINL2 -> PVOL-HP
- RV29: value GAINL3 -> PMASTER
- RV3: value FADERL3 -> BASL1; footprint Library:fader-L60 -> Library:Potentiometer_Bourns_PTV09A-1_Single_Vertical
- RV4: value PITCH-L -> MIDL1; footprint Library:fader-L75 -> Library:Potentiometer_Bourns_PTV09A-1_Single_Vertical
- RV5: value PITH-R -> TREL1; footprint Library:fader-L75 -> Library:Potentiometer_Bourns_PTV09A-1_Single_Vertical
- RV6: value PMIX-HP -> GAINL1
- RV7: value FILTERL1 -> FADERL2; footprint Library:Potentiometer_Bourns_PTV09A-1_Single_Vertical -> Library:fader-L60
- RV9: value FILTERL3 -> BASL2
- SW10: value SWPADR2 -> SWPCUEL2; footprint Library:sw-pad -> Library:SW_PUSH_6mm_H5mm
- SW11: value SWPADR3 -> SWPADL3
- SW12: value SWPADR4 -> SWSHIFTL; footprint Library:sw-pad -> Library:SW_PUSH_6mm_H5mm
- SW13: value SWPADR5 -> SWSHIFTR; footprint Library:sw-pad -> Library:SW_PUSH_6mm_H5mm
- SW14: value SWPADR6 -> SWPCUEL3; footprint Library:sw-pad -> Library:SW_PUSH_6mm_H5mm
- SW15: value SWPADR7 -> SWPADR3
- SW16: value SWPADR8 -> BROWSER-L; footprint Library:sw-pad -> Library:RotaryEncoder_Alps_EC11E-Switch_Vertical_H20mm_CircularMountingHoles
- SW17: value SWPLAYL -> SWPADL4; footprint Library:SW_PUSH_6mm_H5mm -> Library:sw-pad
- SW18: value SWCUEL -> SWPADR4; footprint Library:SW_PUSH_6mm_H5mm -> Library:sw-pad
- SW19: value SWSHIFTL -> SWSYNCL
- SW2: value SWPADL2 -> SWPADR1
- SW20: value SWSYNCL -> SWSYNCR
- SW21: value SWRANGEL -> SWDECK
- SW22: value SWFX1L -> SWPADL5; footprint Library:SW_PUSH_6mm_H5mm -> Library:sw-pad
- SW23: value SWFX2L -> SWPADR5; footprint Library:SW_PUSH_6mm_H5mm -> Library:sw-pad
- SW24: value SWFX3L -> SWRANGEL
- SW25: value SWBR-PREVL -> SWRANGER
- SW26: value SWBR-BACKL -> BROWSER-R; footprint Library:SW_PUSH_6mm_H5mm -> Library:RotaryEncoder_Alps_EC11E-Switch_Vertical_H20mm_CircularMountingHoles
- SW27: value SWPLAYR -> SWPADR6; footprint Library:SW_PUSH_6mm_H5mm -> Library:sw-pad
- SW28: value SWCUER -> SWPADL6; footprint Library:SW_PUSH_6mm_H5mm -> Library:sw-pad
- SW29: value SWSHIFTR -> SWFX1L
- SW3: value SWPADL3 -> SWPLAYL; footprint Library:sw-pad -> Library:SW_PUSH_6mm_H5mm
- SW30: value SWSYNCR -> SWFX1R
- SW31: value SWRANGER -> SWPADR7; footprint Library:SW_PUSH_6mm_H5mm -> Library:sw-pad
- SW32: value SWFX1R -> SWPADL7; footprint Library:SW_PUSH_6mm_H5mm -> Library:sw-pad
- SW33: value SWFX2R -> SWFX2L
- SW34: value SWFX3R -> SWFX2R
- SW35: value SWBR-PREVR -> SWPADR8; footprint Library:SW_PUSH_6mm_H5mm -> Library:sw-pad
- SW36: value SWBR-BACKR -> SWFX3L
- SW37: value SWPCUEL1 -> SWFX3R
- SW38: value SWPCUEL2 -> SWPADL8; footprint Library:SW_PUSH_6mm_H5mm -> Library:sw-pad
- SW39: value SWPCUEL3 -> SWBR-PREVL
- SW4: value SWPADL4 -> SWPLAYR; footprint Library:sw-pad -> Library:SW_PUSH_6mm_H5mm
- SW40: value SWSEL1 -> SWBR-PREVR
- SW5: value SWPADL5 -> SWPCUEL1; footprint Library:sw-pad -> Library:SW_PUSH_6mm_H5mm
- SW6: value SWPADL6 -> SWPADL2
- SW7: value SWPADL7 -> SWPADR2
- SW8: value SWPADL8 -> SWCUEL; footprint Library:sw-pad -> Library:SW_PUSH_6mm_H5mm
- SW9: value SWPADR1 -> SWCUER; footprint Library:sw-pad -> Library:SW_PUSH_6mm_H5mm
- moved SW29 379.0 mm to (127.2, 71.2), turned to 90 degrees
- moved SW18 334.7 mm to (462.5, 162.1)
- moved SW12 311.4 mm to (181.7, 296.7)
- moved SW16 297.1 mm to (176.5, 106.5), turned to -90 degrees
- moved SW25 273.9 mm to (433.8, 230.8), turned to -90 degrees
- moved SW37 266.9 mm to (459.9, 71.2), turned to 90 degrees
- moved RV5 260.2 mm to (251.5, 109.4), turned to 90 degrees
- moved SW11 250.5 mm to (187.0, 162.1)
- moved SW20 249.8 mm to (429.3, 251.2), turned to 90 degrees
- moved SW33 249.4 mm to (169.2, 71.2), turned to 90 degrees
- moved SW23 242.3 mm to (387.5, 187.1), turned to 0 degrees
- moved RV6 238.2 mm to (251.5, 75.4)
- moved RV27 237.9 mm to (351.5, 291.4)
- moved SW28 236.6 mm to (162.0, 187.1)
- moved SW7 226.9 mm to (412.5, 162.1)
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Connections:
- D23 pad 2: LEDHPL3 -> LEDHPL2
- RV10 pad 2: PFX-1L -> MID-L2
- RV11 pad 2: PFX-1R -> TRE-L2
- RV12 pad 2: PVOL-HP -> GAIN-L2
- RV13 pad 2: BAS-L1 -> FADER-L3
- RV14 pad 2: BAS-L2 -> FILTER-L3
- RV16 pad 2: PFX-2L -> MID-L3
- RV17 pad 2: PFX-2R -> TRE-L3
- RV18 pad 2: PMASTER -> GAIN-L3
- RV19 pad 2: MID-L1 -> PITCH-L
- RV2 pad 2: FADER-L2 -> FILTER-L1
- RV20 pad 2: MID-L2 -> PFX-1L
- RV21 pad 2: MID-L3 -> PFX-2L
- RV23 pad 2: PFX-3R -> PITCH-R
- RV24 pad 2: TRE-L1 -> PFX-1R
- RV25 pad 2: TRE-L2 -> PFX-2R
- RV26 pad 2: TRE-L3 -> PFX-3R
- RV27 pad 2: GAIN-L1 -> PMIX-HP
- RV28 pad 2: GAIN-L2 -> PVOL-HP
- RV29 pad 2: GAIN-L3 -> PMASTER
- RV3 pad 2: FADER-L3 -> BAS-L1
- RV4 pad 2: PITCH-L -> MID-L1
- RV5 pad 2: PITCH-R -> TRE-L1
- RV6 pad 2: PMIX-HP -> GAIN-L1
- RV7 pad 2: FILTER-L1 -> FADER-L2
- RV9 pad 2: FILTER-L3 -> BAS-L2
- SW10 pad 2: SWPAD-R2 -> SWPRECUE-L2
- SW11 pad 2: SWPAD-R3 -> SWPAD-L3
- SW12 pad 2: SWPAD-R4 -> SWSHIFT
- SW13 pad 2: SWPAD-R5 -> SWSHIFT
- SW14 pad 2: SWPAD-R6 -> SWPRECUE-L3
- SW15 pad 2: SWPAD-R7 -> SWPAD-R3
- SW17 pad 2: SWPLAY-L -> SWPAD-L4
- SW18 pad 2: SWCUE-L -> SWPAD-R4
- SW19 pad 2: SWSHIFT -> SWSYNC-L
- SW2 pad 2: SWPAD-L2 -> SWPAD-R1
- SW20 pad 2: SWSYNC-L -> SWSYNC-R
- SW21 pad 2: SWRANGE-L -> SW-DECK-SEL
- SW22 pad 2: SWFX1-L -> SWPAD-L5
- SW23 pad 2: SWFX2-L -> SWPAD-R5
- SW24 pad 2: SWFX3-L -> SWRANGE-L
- SW25 pad 2: SWBR-PREVIEW -> SWRANGE-R
- SW27 pad 2: SWPLAY-R -> SWPAD-R6
- SW28 pad 2: SWCUE-R -> SWPAD-L6
- SW29 pad 2: SWSHIFT -> SWFX1-L
- SW3 pad 2: SWPAD-L3 -> SWPLAY-L
- SW30 pad 2: SWSYNC-R -> SWFX1-R
- SW31 pad 2: SWRANGE-R -> SWPAD-R7
- SW32 pad 2: SWFX1-R -> SWPAD-L7
- SW33 pad 2: SWFX2-R -> SWFX2-L
- SW34 pad 2: SWFX3-R -> SWFX2-R
- SW35 pad 2: SWBR-PREVIEW -> SWPAD-R8
- SW36 pad 2: SWBR-BACK -> SWFX3-L
- SW37 pad 2: SWPRECUE-L1 -> SWFX3-R
- SW38 pad 2: SWPRECUE-L2 -> SWPAD-L8
- SW39 pad 2: SWPRECUE-L3 -> SWBR-PREVIEW
- SW4 pad 2: SWPAD-L4 -> SWPLAY-R
- SW40 pad 2: SWSEL-L1 -> SWBR-PREVIEW
- SW5 pad 2: SWPAD-L5 -> SWPRECUE-L1
- SW6 pad 2: SWPAD-L6 -> SWPAD-L2
- SW7 pad 2: SWPAD-L7 -> SWPAD-R2
- SW8 pad 2: SWPAD-L8 -> SWCUE-L
- SW9 pad 2: SWPAD-R1 -> SWCUE-R
- U-LEDS1 pad 15: unconnected-(U-LEDS1-Pad15) -> (no net)
- U-LEDS1 pad 9: unconnected-(U-LEDS1-Pad9) -> (no net)
- U-LEDSR1 pad 15: unconnected-(U-LEDSR1-Pad15) -> (no net)
- U-LEDSR1 pad 7: unconnected-(U-LEDSR1-Pad7) -> (no net)
- UVU-LINE1 pad 1: VUL1-1 -> VUL3-1
- UVU-LINE1 pad 15: VUL1-0 -> VUL3-0
- UVU-LINE1 pad 2: VUL1-2 -> VUL3-2
- UVU-LINE1 pad 3: VUL1-3 -> VUL3-3
- UVU-LINE1 pad 4: VUL1-4 -> VUL3-4
- UVU-LINE1 pad 5: VUL1-5 -> VUL3-5
- UVU-LINE1 pad 6: VUL1-6 -> VUL3-6
- UVU-LINE1 pad 7: VUL1-7 -> VUL3-7
- UVU-LINE1 pad 9: unconnected-(UVU-LINE1-Pad9) -> Net-(UVU-LINE1-Pad9)
- UVU-LINE2 pad 14: Net-(UVU-LINE2-Pad14) -> Net-(UVU-LINE1-Pad9)
- UVU-LINE2 pad 9: Net-(UVU-LINE1-Pad14) -> Net-(UVU-LINE2-Pad9)
- UVU-LINE3 pad 1: VUL3-1 -> VUL1-1
- UVU-LINE3 pad 14: Net-(UVU-LINE3-Pad14) -> Net-(UVU-LINE2-Pad9)
- UVU-LINE3 pad 15: VUL3-0 -> VUL1-0
- UVU-LINE3 pad 2: VUL3-2 -> VUL1-2
- UVU-LINE3 pad 3: VUL3-3 -> VUL1-3
- UVU-LINE3 pad 4: VUL3-4 -> VUL1-4
- UVU-LINE3 pad 5: VUL3-5 -> VUL1-5
- UVU-LINE3 pad 6: VUL3-6 -> VUL1-6
- UVU-LINE3 pad 7: VUL3-7 -> VUL1-7
- UVU-LINE3 pad 9: Net-(UVU-LINE2-Pad14) -> (no net)
- UVU-MASTER-L1 pad 9: Net-(UVU-LINE3-Pad14) -> Net-(UVU-LINE1-Pad14)
- XA1 pad 3V3: unconnected-(XA1-Pad3V3) -> (no net)
- XA1 pad A13: unconnected-(XA1-PadA13) -> (no net)
- XA1 pad A14: unconnected-(XA1-PadA14) -> (no net)
- XA1 pad AREF: unconnected-(XA1-PadAREF) -> (no net)
- XA1 pad D0: SIG_PAD_LED_L -> (no net)
- XA1 pad D2: unconnected-(XA1-PadD2) -> NP_SIG_LEFT
- XA1 pad D23: SWPAD-L4 -> NP_SIG_RIGTH
- XA1 pad D4: SWSEL-L1 -> SW-DECK-SEL
- XA1 pad D46: SIG_PAD_LED_R -> SWPAD-L4
- XA1 pad IORF: unconnected-(XA1-PadIORF) -> (no net)
- XA1 pad RST1: unconnected-(XA1-PadRST1) -> (no net)
- XA1 pad SCL: unconnected-(XA1-PadSCL) -> (no net)
- XA1 pad SDA: unconnected-(XA1-PadSDA) -> (no net)
- XA1 pad VIN: unconnected-(XA1-PadVIN) -> (no net)
Routing:
- net SWPAD-L1: track 0.00 -> 343.8 mm, vias 0 -> 10
- net SWFX1-L: track 339.6 -> 0.00 mm
- net SWPAD-L6: track 0.00 -> 333.4 mm, vias 0 -> 10
- net SWFX2-L: track 299.9 -> 0.00 mm
- net SWPAD-L3: track 0.00 -> 293.1 mm, vias 0 -> 10
- net SWFX3-L: track 261.1 -> 0.00 mm
- net SWPAD-L4: track 0.00 -> 229.1 mm, vias 0 -> 2
- net LEDFX3R: track 0.00 -> 192.2 mm, vias 0 -> 8
- net LEDPLAYL: track 0.00 -> 182.8 mm
- net MPLEX-A0: track 178.2 -> 0.00 mm, vias 4 -> 0
- net LEDPLAYR: track 0.00 -> 173.7 mm, vias 0 -> 6
- net Net-(UVU-LINE1-Pad14): track 0.00 -> 164.1 mm, vias 0 -> 8
- net LEDCUEL: track 0.00 -> 152.5 mm
- net Net-(U-LEDS1-Pad14): track 0.00 -> 152.5 mm, vias 0 -> 4
- net LEDFX1L: track 0.00 -> 150.7 mm, vias 0 -> 2
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