File: PCB/Kicad/Mixduino.kicad_pcb (KiCad board)
At the start: 2 copper layers, 360 x 260 mm, 242 parts, among them SW1 SWPADL1, SW10 SWPCUEL2, SW11 SWPADL3, SW12 SWSHIFTL, SW13 SWSHIFTR, SW14 SWPCUEL3, SW15 SWPADR3, SW16 BROWSER-L, SW17 SWPADL4, SW18 SWPADR4, SW19 SWSYNCL, SW2 SWPADR1, SW20 SWSYNCR, SW21 SWDECK, SW22 SWPADL5, SW23 SWPADR5, SW24 SWRANGEL, SW25 SWRANGER, SW26 BROWSER-R, SW27 SWPADR6, SW28 SWPADL6, SW29 SWFX1L, SW3 SWPLAYL, SW30 SWFX1R, SW31 SWPADR7, SW32 SWPADL7, SW33 SWFX2L, SW34 SWFX2R, SW35 SWPADR8, SW36 SWFX3L, SW37 SWFX3R, SW38 SWPADL8, SW39 SWBR-PREVL, SW4 SWPLAYR, SW40 SWBR-PREVR, SW41 SWBR-BACKL, SW42 SWBR-BACKR, SW43 SWLOOPL, SW44 SWLOOPR, SW5 SWPCUEL1, SW6 SWPADL2, SW7 SWPADR2, SW8 SWCUEL, SW9 SWCUER

Commit message: schematic updated
Parts:
- moved IC-MPLEX-1 43.9 mm to (300.2, 211.8)
- moved NPR2 16.0 mm to (393.9, 152.2), turned to 180 degrees
- moved IC-MPLEX-2 5.67 mm to (203.7, 212.1), turned to 90 degrees
- moved NPR1 3.09 mm to (144.7, 153.2), turned to 180 degrees
- turned R54 to -90 degrees
Connections:
- IC-MPLEX-1 pad 16: MID-L3 -> FADER-L3
- IC-MPLEX-1 pad 17: MID-L2 -> PMIX-HP
- IC-MPLEX-1 pad 18: MID-L1 -> PVOL-HP
- IC-MPLEX-1 pad 19: BAS-L3 -> PITCH-R
- IC-MPLEX-1 pad 2: FILTER-L1 -> BAS-L2
- IC-MPLEX-1 pad 20: BAS-L2 -> FILTER-L3
- IC-MPLEX-1 pad 21: BAS-L1 -> BAS-L3
- IC-MPLEX-1 pad 22: FILTER-L3 -> MID-L3
- IC-MPLEX-1 pad 23: FILTER-L2 -> MID-L2
- IC-MPLEX-1 pad 3: PITCH-R -> MID-L1
- IC-MPLEX-1 pad 4: PVOL-HP -> BAS-L1
- IC-MPLEX-1 pad 5: PMIX-HP -> FILTER-L2
- IC-MPLEX-1 pad 6: FADER-L3 -> FILTER-L1
- IC-MPLEX-1 pad 7: FADER-L2 -> PITCH-L
- IC-MPLEX-1 pad 9: PITCH-L -> FADER-L2
- IC-MPLEX-2 pad 16: SWPRECUE-L1 -> SWPAD-L8
- IC-MPLEX-2 pad 17: SWPRECUE-L2 -> SWPAD-L4
- IC-MPLEX-2 pad 18: SWPRECUE-L3 -> SWPAD-L3
- IC-MPLEX-2 pad 19: SWCUE-L -> SWPAD-L7
- IC-MPLEX-2 pad 2: SWPAD-L1 -> SWCUE-L
- IC-MPLEX-2 pad 20: SWPLAY-L -> SWPAD-L2
- IC-MPLEX-2 pad 21: SWRANGE-L -> SWPAD-L6
- IC-MPLEX-2 pad 22: SWSHIFT -> SWPAD-L1
- IC-MPLEX-2 pad 23: SWSYNC-L -> SWPAD-L5
- IC-MPLEX-2 pad 3: SWPAD-L2 -> SWPLAY-L
- IC-MPLEX-2 pad 4: SWPAD-L3 -> SWRANGE-L
- IC-MPLEX-2 pad 5: SWPAD-L4 -> SWSYNC-L
- IC-MPLEX-2 pad 6: SWPAD-L5 -> SWLOOP-L
- IC-MPLEX-2 pad 7: SWPAD-L6 -> SWSHIFT
- IC-MPLEX-2 pad 8: SWPAD-L7 -> SWPRECUE-L1
- IC-MPLEX-2 pad 9: SWPAD-L8 -> SWPRECUE-L2
- NP10 pad 2: (no net) -> unconnected-(NP10-Pad2)
- NP11 pad 2: Net-(NP11-Pad2) -> unconnected-(NP11-Pad2)
- NP12 pad 2: Net-(NP12-Pad2) -> Net-(NP11-Pad4)
- NP12 pad 4: Net-(NP11-Pad2) -> Net-(NP12-Pad4)
- NP13 pad 2: Net-(NP13-Pad2) -> Net-(NP12-Pad4)
- NP13 pad 4: Net-(NP12-Pad2) -> Net-(NP13-Pad4)
- NP14 pad 2: Net-(NP14-Pad2) -> Net-(NP13-Pad4)
- NP14 pad 4: Net-(NP13-Pad2) -> Net-(NP14-Pad4)
- NP15 pad 2: Net-(NP15-Pad2) -> Net-(NP14-Pad4)
- NP15 pad 4: Net-(NP14-Pad2) -> Net-(NP15-Pad4)
- NP16 pad 2: Net-(NP16-Pad2) -> Net-(NP15-Pad4)
- NP16 pad 4: Net-(NP15-Pad2) -> Net-(NP16-Pad4)
- NP17 pad 2: Net-(NP17-Pad2) -> Net-(NP16-Pad4)
- NP17 pad 4: Net-(NP16-Pad2) -> Net-(NP17-Pad4)
- NP18 pad 2: (no net) -> Net-(NP17-Pad4)
- NP18 pad 4: Net-(NP17-Pad2) -> Net-(NP18-Pad4)
- NP21 pad 2: (no net) -> unconnected-(NP21-Pad2)
- NP8 pad 2: (no net) -> unconnected-(NP8-Pad2)
- NPR2 pad 2: Net-(NP11-Pad4) -> Net-(NP18-Pad4)
- U-LEDS1 pad 9: (no net) -> unconnected-(U-LEDS1-Pad9)
- U-LEDSR1 pad 7: (no net) -> unconnected-(U-LEDSR1-Pad7)
- UVU-LINE1 pad 9: (no net) -> unconnected-(UVU-LINE1-Pad9)
- XA1 pad 3V3: (no net) -> unconnected-(XA1-Pad3V3)
- XA1 pad A10: GAIN-L1 -> PFX-3L
- XA1 pad A15: (no net) -> unconnected-(XA1-PadA15)
- XA1 pad A2: PFX-3L -> PFX-1R
- XA1 pad A3: PFX-2L -> GAIN-L3
- XA1 pad A4: PFX-1L -> GAIN-L2
- XA1 pad A5: PFX-3R -> GAIN-L1
- XA1 pad A6: PFX-2R -> PFX-3R
- XA1 pad A7: PFX-1R -> PFX-2R
- XA1 pad A8: GAIN-L3 -> PFX-1L
- XA1 pad A9: GAIN-L2 -> PFX-2L
- XA1 pad AREF: (no net) -> unconnected-(XA1-PadAREF)
- XA1 pad D0: (no net) -> unconnected-(XA1-PadD0)
- XA1 pad D1: (no net) -> unconnected-(XA1-PadD1)
- XA1 pad D14: (no net) -> unconnected-(XA1-PadD14)
- XA1 pad D15: (no net) -> unconnected-(XA1-PadD15)
- XA1 pad D16: (no net) -> unconnected-(XA1-PadD16)
- XA1 pad D17: (no net) -> unconnected-(XA1-PadD17)
- XA1 pad D18: (no net) -> unconnected-(XA1-PadD18)
- XA1 pad D19: (no net) -> unconnected-(XA1-PadD19)
- XA1 pad D22: SWLOOP-L -> unconnected-(XA1-PadD22)
- XA1 pad D25: SWPAD-R8 -> SWPAD-R4
- XA1 pad D27: SWPAD-R4 -> SWPAD-R8
- XA1 pad D4: SW-DECK-SEL -> L_BROWSER_A
- XA1 pad D41: L_BROWSER_B -> SW-DECK-SEL
- XA1 pad D43: L_BROWSER_A -> FB-LATCH
- XA1 pad D45: (no net) -> SWPRECUE-L3
- XA1 pad D46: (no net) -> unconnected-(XA1-PadD46)
- XA1 pad D5: FB-LATCH -> L_BROWSER_B
- XA1 pad IORF: (no net) -> unconnected-(XA1-PadIORF)
- XA1 pad RST1: (no net) -> unconnected-(XA1-PadRST1)
- XA1 pad SCL: (no net) -> unconnected-(XA1-PadSCL)
- XA1 pad SDA: (no net) -> unconnected-(XA1-PadSDA)
- XA1 pad VIN: (no net) -> unconnected-(XA1-PadVIN)
Routing:
- net SWSHIFT: track 0.00 -> 343.6 mm
- net PITCH-R: track 0.00 -> 160.7 mm
- net PMIX-HP: track 0.00 -> 103.6 mm
- net SWPLAY-L: track 0.00 -> 103.3 mm
- net PITCH-L: track 0.00 -> 100.0 mm
- net MID-L1: track 0.00 -> 96.3 mm
- net SWPAD-L1: track 0.00 -> 91.8 mm
- net MID-L2: track 0.00 -> 81.7 mm
- net SWCUE-L: track 0.00 -> 72.9 mm
- net PVOL-HP: track 0.00 -> 72.0 mm
- net MID-L3: track 0.00 -> 70.3 mm
- net SWPAD-L2: track 0.00 -> 70.2 mm
- net SWLOOP-L: track 0.00 -> 67.5 mm
- net SWPAD-L5: track 0.00 -> 66.2 mm
- net VUMASL-0: track 0.00 -> 65.5 mm
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