File: PCB/Kicad/Mixduino.kicad_pcb (KiCad board)
At the start: 2 copper layers, 360 x 260 mm, 336 parts, among them Q1 MMBTA05L, Q2 MMBTA05L, Q3 MMBTA05L, Q4 MMBTA05L, SW1 BROWSER-L, SW10 SWFX2L, SW11 SWFX1R, SW12 SWFX3L, SW13 SWCUEL, SW14 SWPLAYL, SW15 SWRANGEL, SW16 SWSYNCL, SW17 SWLOOPL, SW18 SWSHIFTL, SW19 SWSHIFTR, SW2 BROWSER-R, SW20 SWPCUEL1, SW21 SWPCUEL2, SW22 SWCUER, SW23 SWPLAYR, SW24 SWRANGER, SW25 SWLOOPR, SW26 SWPCUEL3, SW27 SWSYNCR, SW28 SWDECKSEL, SW29 SWPADL5, SW3 SWBR-BACKR, SW30 SWPADL1, SW31 SWPADL6, SW32 SWPADL2, SW33 SWPADL7, SW34 SWPADL3, SW35 SWPADL4, SW36 SWPADL8, SW37 SWPADR5, SW38 SWPADR1, SW39 SWPADR6, SW4 SWBR-BACKL, SW40 SWPADR2, SW41 SWPADR7, SW42 SWPADR3, SW43 SWPADR4, SW44 SWPADR8, SW5 SWBR-PREVR, SW6 SWBR-PREVL, SW7 SWFX2R, SW8 SWFX3R, SW9 SWFX1L, U1 SR1-L1, U10 SR2-MR, U2 SR2-L1, U3 SR1-L2, U4 SR2-L2, U5 SR1-L3, U6 SR2-L3, U7 SR1-ML, U8 SR2-ML, U9 SR1-MR

Commit message: routing WIP
Parts:
- moved SR-FB-RIGHT1 7.96 mm to (370.2, 200.7)
- moved U1 6.91 mm to (220.0, 122.1)
- moved U2 6.91 mm to (220.0, 154.8)
- moved U3 2.19 mm to (254.7, 122.7)
- moved U4 1.84 mm to (254.9, 154.8)
- moved U9 1.21 mm to (349.8, 122.2)
- moved R37 0.43 mm to (239.0, 165.6), turned to 180 degrees
- moved NPR1 0.21 mm to (144.5, 153.2)
- moved R33 0.20 mm to (238.9, 147.7), turned to 180 degrees
- moved R13 0.15 mm to (160.2, 286.3)
- turned R24 to 180 degrees
- turned R25 to 180 degrees
- turned R26 to 180 degrees
- turned R27 to 180 degrees
- turned R28 to 180 degrees
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Connections:
- RV5 pad 2: Net-(IC-MPLEX-1-Pad3) -> Net-(IC-MPLEX-1-Pad2)
- RV9 pad 2: Net-(IC-MPLEX-1-Pad2) -> Net-(IC-MPLEX-1-Pad3)
- SR-FB-RIGHT1 pad 1: Net-(R12-Pad1) -> Net-(R18-Pad1)
- SR-FB-RIGHT1 pad 2: Net-(R18-Pad1) -> Net-(R12-Pad1)
- SW3 pad 2: Net-(SW10-Pad2) -> Net-(SW3-Pad2)
- SW4 pad 2: Net-(SW4-Pad2) -> Net-(SW3-Pad2)
- SW41 pad 1: Net-(IC-MPLEX-2-Pad20) -> Net-(IC-MPLEX-2-Pad21)
- SW42 pad 1: Net-(IC-MPLEX-2-Pad21) -> Net-(IC-MPLEX-2-Pad20)
- XA1 pad D14: L2VU-LATCH -> Net-(SW5-Pad2)
- XA1 pad D15: L2VU-SIG -> Net-(SW3-Pad2)
- XA1 pad D18: R_BROWSER_A -> R_BROWSER_B
- XA1 pad D19: R_BROWSER_B -> R_BROWSER_A
- XA1 pad D31: Net-(SW5-Pad2) -> L2VU-SIG
- XA1 pad D38: Net-(SW10-Pad2) -> L2VU-LATCH
- XA1 pad D9: Net-(SW4-Pad2) -> Net-(SW10-Pad2)
Routing:
- net MPLEX-S0: track 0.00 -> 725.0 mm, vias 0 -> 10
- net MPLEX-S1: track 0.00 -> 717.3 mm, vias 0 -> 8
- net MPLEX-S2: track 0.00 -> 707.1 mm, vias 0 -> 7
- net MPLEX-S3: track 0.00 -> 667.9 mm, vias 0 -> 8
- net SRCLK: track 0.00 -> 466.6 mm, vias 0 -> 12
- net L_BROWSER_A: track 0.00 -> 422.6 mm, vias 0 -> 5
- net L_BROWSER_B: track 0.00 -> 405.3 mm, vias 0 -> 5
- net Net-(SW3-Pad2): track 0.00 -> 403.7 mm, vias 0 -> 6
- net Net-(SW5-Pad2): track 0.00 -> 384.4 mm, vias 0 -> 4
- net SW_BROWSER_L: track 0.00 -> 377.2 mm, vias 0 -> 2
- net Net-(SW9-Pad2): track 0.00 -> 374.6 mm
- net Net-(IC-MPLEX-3-Pad7): track 0.00 -> 369.2 mm, vias 0 -> 3
- net NP_DATA: track 0.00 -> 356.4 mm, vias 0 -> 5
- net Net-(SW10-Pad2): track 0.00 -> 350.3 mm
- net L1VU-LATCH: track 0.00 -> 316.7 mm, vias 0 -> 3
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Other:
- rule pad_to_mask_clearance: 0 -> 0.05
