File: PCB/Kicad/Mixduino.kicad_sch (KiCad schematic)
At the start: 3 parts

Commit message: SCHEMATIC FINISHED
Parts:
- added RV1: PFX1R, Library:Potentiometer_Bourns_PTV09A-1_Single_Vertical, symbol Device:R_Potentiometer
- added RV2: PMASTER, Library:Potentiometer_Bourns_PTV09A-1_Single_Vertical, symbol Device:R_Potentiometer
- added SW1: BROWSER-L, Library:RotaryEncoder_Alps_EC11E-Switch_Vertical_H20mm_CircularMountingHoles, symbol Device:RotaryEncoder_Switch
- added SW10: SWFX2L, Library:SW_PUSH_6mm_H8mm, symbol mixduino-mk2:SW_Push
- added SW11: SWFX1R, Library:SW_PUSH_6mm_H8mm, symbol mixduino-mk2:SW_Push
- added SW12: SWFX3L, Library:SW_PUSH_6mm_H8mm, symbol mixduino-mk2:SW_Push
- added SW2: BROWSER-R, Library:RotaryEncoder_Alps_EC11E-Switch_Vertical_H20mm_CircularMountingHoles, symbol Device:RotaryEncoder_Switch
- added SW3: SWBR-BACKR, Library:SW_PUSH_6mm_H8mm, symbol mixduino-mk2:SW_Push
- added SW4: SWBR-BACKL, Library:SW_PUSH_6mm_H8mm, symbol mixduino-mk2:SW_Push
- added SW5: SWBR-PREVR, Library:SW_PUSH_6mm_H8mm, symbol mixduino-mk2:SW_Push
- added SW6: SWBR-PREVL, Library:SW_PUSH_6mm_H8mm, symbol mixduino-mk2:SW_Push
- added SW7: SWFX2R, Library:SW_PUSH_6mm_H8mm, symbol mixduino-mk2:SW_Push
- added SW8: SWFX3R, Library:SW_PUSH_6mm_H8mm, symbol mixduino-mk2:SW_Push
- added SW9: SWFX1L, Library:SW_PUSH_6mm_H8mm, symbol mixduino-mk2:SW_Push
Connections:
- net SWFX1-L is gone; now on net SW_BROWSER_R: XA1.D7
- net +5V: now also RV1.1, RV2.1
- net GND: now also RV1.3, RV2.3, SW1.C, SW1.S2, SW10.1, SW11.1, SW12.1, SW2.C, SW2.S2, SW3.1, SW4.1, SW5.1, SW6.1, SW7.1, SW8.1, SW9.1
- net L_BROWSER_A: now also SW1.A
- net L_BROWSER_B: now also SW1.B
- net R_BROWSER_A: now also SW2.A
- net R_BROWSER_B: now also SW2.B
- net SW_BROWSER_L: now also SW1.S1
- net SW_BROWSER_R: now also SW2.S1; no longer XA1.D32
- net MPLEX-A3: now reaches XA1.A3
- net MPLEX-A4: now reaches XA1.A4
- net at XA1.D12: now also SW12.2
- net L2VU-LATCH: now reaches XA1.D14 (D14_TX3)
- net L2VU-SIG: now reaches XA1.D15 (D15_RX3)
- net L1VU-LATCH: now reaches XA1.D16 (D16_TX2)
- net L1VU-SIG: now reaches XA1.D17 (D17_RX2)
- net MRVU-LATCH: now reaches XA1.D26
- net MRVU-SIG: now reaches XA1.D28
- net at XA1.D31: now also SW5.2, SW6.2
- net L3VU-SIG: now reaches XA1.D34
- net L3VU-LATCH: now reaches XA1.D36
- net FB-L-SIG: now reaches XA1.D37
- net FB-L-LATCH: now reaches XA1.D39
- net FB-R-SIG: now reaches XA1.D42
- net FB-R-LATCH: now reaches XA1.D44
- net BTNLED-SF-DATA: no longer names the net of XA1.D51
- net FB-LATCH: no longer names the net of XA1.D43
- net MPLEX-A0 renamed MPLEX-A2
- net PFX-1R: no longer names the net of XA1.A0
- net PFX-1R: now also RV1.2
- net PMASTER: no longer names the net of XA1.A14
- net PMASTER: now also RV2.2
- net SF-CLOCK renamed SRCLK
- net SWBR-BACK: no longer names the net of XA1.D38
- net SWBR-BACK: now also SW3.2, SW4.2
- net SWBR-PREVIEW renamed MLVU-LATCH
- net SWFX1-R: no longer names the net of XA1.D11
- net SWFX1-R: now also SW11.2
- net SWFX2-L: no longer names the net of XA1.D8
- net SWFX2-L: now also SW9.2
- net SWFX2-R: no longer names the net of XA1.D4
- net SWFX2-R: now also SW7.2
- net SWFX3-L: no longer names the net of XA1.D9
- net SWFX3-L: now also SW10.2
- net SWFX3-R: no longer names the net of XA1.D5
- net SWFX3-R: now also SW8.2
- net VU-LATCH: no longer names the net of XA1.D50
- net VU-SF-DATA: no longer names the net of XA1.D48
- new net MLVU-SIG: XA1.D32
- no-connect marks 21 -> 35
Other:
- sheet LedsSheet renamed VU Leds
- sheet MultiplexersSheet renamed MPX SW BTNS
- sheet PotenciometersSheet renamed TOP POTS
- sheet ShiftRegistersSheet renamed FEEDBACK Leds
- removed sheet SwitchersSheet
- added sheet BOTTOM POTS (BOTTOM-POTS.kicad_sch)
- sheet FEEDBACK Leds: file shift-registers.kicad_sch -> fb-leds.kicad_sch
- sheet MPX SW BTNS: file multiplexers.kicad_sch -> MPX-SW-BTNS.kicad_sch
- sheet TOP POTS: file potenciometers.kicad_sch -> TOP-POTS.kicad_sch
- sheet VU Leds: file leds.kicad_sch -> vu-leds.kicad_sch
- moved on the sheet: TB1, TB2
