File: PCB/Kicad/leds.kicad_sch (KiCad schematic)
At the start: 94 parts

Commit message: fixing 3dmodels
Parts:
- BCUELD1, BCUERD1, BHPL1D1, BHPL2D1, D23, VUL1D6, VUL1D7, VUL2D6, VUL2D7, VUL3D6, VUL3D7, VUMASLD6, VUMASLD7, VUMASRD6, VUMASRD7: footprint LED_THT:LED_Rectangular_W3.0mm_H2.0mm -> Library:LED_YELLOW
- BCUELR1, BCUERR1, BHPL1R1, BHPL2R1, BPLAYLR1, BPLAYRR1, R23, VUL1R1, VUL1R2, VUL1R3, VUL1R4, VUL1R5, VUL1R6, VUL1R7, VUL1R8, VUL2R1, VUL2R2, VUL2R3, VUL2R4, VUL2R5, VUL2R6, VUL2R7, VUL2R8, VUL3R1, VUL3R2, VUL3R3, VUL3R4, VUL3R5, VUL3R6, VUL3R7, VUL3R8, VUMASLR1, VUMASLR2, VUMASLR3, VUMASLR4, VUMASLR5, VUMASLR6, VUMASLR7, VUMASLR8, VUMASRR1, VUMASRR2, VUMASRR3, VUMASRR4, VUMASRR5, VUMASRR6, VUMASRR7, VUMASRR8: footprint Resistor_SMD:R_1206_3216Metric_Pad1.30x1.75mm_HandSolder -> Library:R_1206_3216Metric_Pad1.30x1.75mm_HandSolder
- BPLAYLD1, BPLAYRD1, VUL1D1, VUL1D2, VUL1D3, VUL1D4, VUL1D5, VUL2D1, VUL2D2, VUL2D3, VUL2D4, VUL2D5, VUL3D1, VUL3D2, VUL3D3, VUL3D4, VUL3D5, VUMASLD1, VUMASLD2, VUMASLD3, VUMASLD4, VUMASLD5, VUMASRD1, VUMASRD2, VUMASRD3, VUMASRD4, VUMASRD5: footprint LED_THT:LED_Rectangular_W3.0mm_H2.0mm -> Library:LED_GREEN
- VUL1D8, VUL2D8, VUL3D8, VUMASLD8, VUMASRD8: footprint LED_THT:LED_Rectangular_W3.0mm_H2.0mm -> Library:LED_RED

Commit message: sr wip
Parts:
- added FX1LD1, FX1RD1: LED_ALT, Library:LED_GREEN, symbol Device:LED_Filled
- added FX1LR1, FX1RR1, FX2LR1, FX2RR1, FX3LR1, FX3RR1: R_Small, Library:R_1206_3216Metric_Pad1.30x1.75mm_HandSolder, symbol Device:R_Small
- added FX2LD1, FX2RD1, FX3LD1, FX3RD1: LED_ALT, Library:LED_YELLOW, symbol Device:LED_Filled
Connections:
- net GND: now also FX1LR1.2, FX1RR1.2, FX2LR1.2, FX2RR1.2, FX3LR1.2, FX3RR1.2
- new net: FX2RD1.1 (K), FX2RR1.1
- new net: FX3RD1.1 (K), FX3RR1.1
- new net: FX2LD1.1 (K), FX2LR1.1
- new net: FX1LD1.1 (K), FX1LR1.1
- new net: FX3LD1.1 (K), FX3LR1.1
- new net: FX1RD1.1 (K), FX1RR1.1
- new net LEDFX1L: FX1LD1.2 (A)
- new net LEDFX1R: FX1RD1.2 (A)
- new net LEDFX2L: FX2LD1.2 (A)
- new net LEDFX2R: FX2RD1.2 (A)
- new net LEDFX3L: FX3LD1.2 (A)
- new net LEDFX3R: FX3RD1.2 (A)
Other:
- moved on the sheet: BCUELD1, BCUELR1, BCUERD1, BCUERR1, BPLAYLD1, BPLAYLR1, BPLAYRD1, BPLAYRR1

Commit message: routing
Parts:
- removed VUL2D1, VUL2D2, VUL2D3, VUL2D4, VUL2D5, VUL3D1, VUL3D2, VUL3D3, VUL3D4, VUL3D5: LED_Filled, Library:LED_GREEN, symbol Device:LED_Filled
- removed VUL2D6, VUL2D7, VUL3D6, VUL3D7: LED_Filled, Library:LED_YELLOW, symbol Device:LED_Filled
- removed VUL2D8, VUL3D8: LED_Filled, Library:LED_RED, symbol Device:LED_Filled
- removed VUL2R1, VUL2R2, VUL2R3, VUL2R4, VUL2R5, VUL2R6, VUL2R7, VUL2R8, VUL3R1, VUL3R2, VUL3R3, VUL3R4, VUL3R5, VUL3R6, VUL3R7, VUL3R8: R_Small, Library:R_1206_3216Metric_Pad1.30x1.75mm_HandSolder, symbol Device:R_Small
- added D14: VUL2D1, Library:LED_GREEN, symbol Device:LED_Filled
- added D15: VUL2D2, Library:LED_GREEN, symbol Device:LED_Filled
- added D16: VUL2D3, Library:LED_GREEN, symbol Device:LED_Filled
- added D17: VUL2D4, Library:LED_GREEN, symbol Device:LED_Filled
- added D18: VUL2D5, Library:LED_GREEN, symbol Device:LED_Filled
- added D19: VUL2D6, Library:LED_YELLOW, symbol Device:LED_Filled
- added D20: VUL2D7, Library:LED_YELLOW, symbol Device:LED_Filled
- added D21: VUL2D8, Library:LED_RED, symbol Device:LED_Filled
- added D30: VUL3D1, Library:LED_GREEN, symbol Device:LED_Filled
- added D31: VUL3D2, Library:LED_GREEN, symbol Device:LED_Filled
- added D32: VUL3D3, Library:LED_GREEN, symbol Device:LED_Filled
- added D33: VUL3D4, Library:LED_GREEN, symbol Device:LED_Filled
- added D34: VUL3D5, Library:LED_GREEN, symbol Device:LED_Filled
- added D35: VUL3D6, Library:LED_YELLOW, symbol Device:LED_Filled
- added D36: VUL3D7, Library:LED_YELLOW, symbol Device:LED_Filled
- added D37: VUL3D8, Library:LED_RED, symbol Device:LED_Filled
- added R14: VUL2R1, Library:R_1206_3216Metric_Pad1.30x1.75mm_HandSolder, symbol Device:R_Small
- added R15: VUL2R2, Library:R_1206_3216Metric_Pad1.30x1.75mm_HandSolder, symbol Device:R_Small
- added R16: VUL2R3, Library:R_1206_3216Metric_Pad1.30x1.75mm_HandSolder, symbol Device:R_Small
- added R17: VUL2R4, Library:R_1206_3216Metric_Pad1.30x1.75mm_HandSolder, symbol Device:R_Small
- added R18: VUL2R5, Library:R_1206_3216Metric_Pad1.30x1.75mm_HandSolder, symbol Device:R_Small
- added R19: VUL2R6, Library:R_1206_3216Metric_Pad1.30x1.75mm_HandSolder, symbol Device:R_Small
- added R20: VUL2R7, Library:R_1206_3216Metric_Pad1.30x1.75mm_HandSolder, symbol Device:R_Small
- added R21: VUL2R8, Library:R_1206_3216Metric_Pad1.30x1.75mm_HandSolder, symbol Device:R_Small
- added R30: VUL3R1, Library:R_1206_3216Metric_Pad1.30x1.75mm_HandSolder, symbol Device:R_Small
- added R31: VUL3R2, Library:R_1206_3216Metric_Pad1.30x1.75mm_HandSolder, symbol Device:R_Small
- added R32: VUL3R3, Library:R_1206_3216Metric_Pad1.30x1.75mm_HandSolder, symbol Device:R_Small
- added R33: VUL3R4, Library:R_1206_3216Metric_Pad1.30x1.75mm_HandSolder, symbol Device:R_Small
- added R34: VUL3R5, Library:R_1206_3216Metric_Pad1.30x1.75mm_HandSolder, symbol Device:R_Small
- added R35: VUL3R6, Library:R_1206_3216Metric_Pad1.30x1.75mm_HandSolder, symbol Device:R_Small
- added R36: VUL3R7, Library:R_1206_3216Metric_Pad1.30x1.75mm_HandSolder, symbol Device:R_Small
- added R37: VUL3R8, Library:R_1206_3216Metric_Pad1.30x1.75mm_HandSolder, symbol Device:R_Small
- D1: renamed from VUL1D1; value LED_Filled -> VUL1D1
- D10: renamed from BCUELD1; value LED_ALT -> LCUE-D
- D11: renamed from FX1LD1; value LED_ALT -> LFX1-D
- D12: renamed from FX2LD1; value LED_ALT -> LFX2-D
- D13: renamed from FX3LD1; value LED_ALT -> LFX3-D
- D2: renamed from VUL1D2; value LED_Filled -> VUL1D2
- D22: renamed from BHPL1D1; value LED_ALT -> L1HP-D
- D23: renamed from BHPL2D1; value LED_ALT -> L2HP-D
- D24: renamed from D23; value LED_ALT -> L3HP-D
- D25: renamed from BPLAYRD1; value LED_ALT -> RPLAY-D
- D26: renamed from BCUERD1; value LED_ALT -> RCUE-D
- D27: renamed from FX1RD1; value LED_ALT -> RFX1-D
- D28: renamed from FX2RD1; value LED_ALT -> RFX2-D
- D29: renamed from FX3RD1; value LED_ALT -> RFX3-D
- D3: renamed from VUL1D3; value LED_Filled -> VUL1D3
- D38: renamed from VUMASLD1; value LED_Filled -> VUMASLD1
- D39: renamed from VUMASLD2; value LED_Filled -> VUMASLD2
- D4: renamed from VUL1D4; value LED_Filled -> VUL1D4
- D40: renamed from VUMASLD3; value LED_Filled -> VUMASLD3
- D41: renamed from VUMASLD4; value LED_Filled -> VUMASLD4
- D42: renamed from VUMASLD5; value LED_Filled -> VUMASLD5
- D43: renamed from VUMASLD6; value LED_Filled -> VUMASLD6
- D44: renamed from VUMASLD7; value LED_Filled -> VUMASLD7
- D45: renamed from VUMASLD8; value LED_Filled -> VUMASLD8
- D46: renamed from VUMASRD1; value LED_Filled -> VUMASRD1
- D47: renamed from VUMASRD2; value LED_Filled -> VUMASRD2
- D48: renamed from VUMASRD3; value LED_Filled -> VUMASRD3
- D49: renamed from VUMASRD4; value LED_Filled -> VUMASRD4
- D5: renamed from VUL1D5; value LED_Filled -> VUL1D5
- D50: renamed from VUMASRD5; value LED_Filled -> VUMASRD5
- D51: renamed from VUMASRD6; value LED_Filled -> VUMASRD6
- D52: renamed from VUMASRD7; value LED_Filled -> VUMASRD7
- D53: renamed from VUMASRD8; value LED_Filled -> VUMASRD8
- D6: renamed from VUL1D6; value LED_Filled -> VUL1D6
- D7: renamed from VUL1D7; value LED_Filled -> VUL1D7
- D8: renamed from VUL1D8; value LED_Filled -> VUL1D8
- D9: renamed from BPLAYLD1; value LED_ALT -> LPLAY-D
- R1: renamed from VUL1R1; value R_Small -> VUL1R1
- R10: renamed from BCUELR1; value R_Small -> LCUE-R
- R11: renamed from FX1LR1; value R_Small -> LFX1R
- R12: renamed from FX2LR1; value R_Small -> LFX2R
- R13: renamed from FX3LR1; value R_Small -> LFX3R
- R2: renamed from VUL1R2; value R_Small -> VUL1R2
- R22: renamed from BHPL1R1; value R_Small -> L1HP-R
- R23: renamed from BHPL2R1; value R_Small -> L2HP-R
- R24: renamed from R23; value R_Small -> L3HP-R
- R25: renamed from BPLAYRR1; value R_Small -> RPLAY-R
- R26: renamed from BCUERR1; value R_Small -> RCUE-R
- R27: renamed from FX1RR1; value R_Small -> RFX1-R
- R28: renamed from FX2RR1; value R_Small -> RFX2-R
- R29: renamed from FX3RR1; value R_Small -> RFX3-R
- R3: renamed from VUL1R3; value R_Small -> VUL1R3
- R38: renamed from VUMASLR1; value R_Small -> VUMASLR1
- R39: renamed from VUMASLR2; value R_Small -> VUMASLR2
- R4: renamed from VUL1R4; value R_Small -> VUL1R4
- R40: renamed from VUMASLR3; value R_Small -> VUMASLR3
- R41: renamed from VUMASLR4; value R_Small -> VUMASLR4
- R42: renamed from VUMASLR5; value R_Small -> VUMASLR5
- R43: renamed from VUMASLR6; value R_Small -> VUMASLR6
- R44: renamed from VUMASLR7; value R_Small -> VUMASLR7
- R45: renamed from VUMASLR8; value R_Small -> VUMASLR8
- R46: renamed from VUMASRR1; value R_Small -> VUMASRR1
- R47: renamed from VUMASRR2; value R_Small -> VUMASRR2
- R48: renamed from VUMASRR3; value R_Small -> VUMASRR3
- R49: renamed from VUMASRR4; value R_Small -> VUMASRR4
- R5: renamed from VUL1R5; value R_Small -> VUL1R5
- R50: renamed from VUMASRR5; value R_Small -> VUMASRR5
- R51: renamed from VUMASRR6; value R_Small -> VUMASRR6
- R52: renamed from VUMASRR7; value R_Small -> VUMASRR7
- R53: renamed from VUMASRR8; value R_Small -> VUMASRR8
- R6: renamed from VUL1R6; value R_Small -> VUL1R6
- R7: renamed from VUL1R7; value R_Small -> VUL1R7
- R8: renamed from VUL1R8; value R_Small -> VUL1R8
- R9: renamed from BPLAYLR1; value R_Small -> LPLAY-R
Connections:
- net GND: now also R14.2, R15.2, R16.2, R17.2, R18.2, R19.2, R20.2, R21.2, R30.2, R31.2, R32.2, R33.2, R34.2, R35.2, R36.2, R37.2
- net VUL2-0: now also D14.2 (A)
- net VUL2-1: now also D15.2 (A)
- net VUL2-2: now also D16.2 (A)
- net VUL2-3: now also D17.2 (A)
- net VUL2-4: now also D18.2 (A)
- net VUL2-5: now also D19.2 (A)
- net VUL2-6: now also D20.2 (A)
- net VUL2-7: now also D21.2 (A)
- net VUL3-0: now also D30.2 (A)
- net VUL3-1: now also D31.2 (A)
- net VUL3-2: now also D32.2 (A)
- net VUL3-3: now also D33.2 (A)
- net VUL3-4: now also D34.2 (A)
- net VUL3-5: now also D35.2 (A)
- net VUL3-6: now also D36.2 (A)
- net VUL3-7: now also D37.2 (A)
- new net: D19.1 (K), R19.1
- new net: D17.1 (K), R17.1
- new net: D21.1 (K), R21.1
- new net: D35.1 (K), R35.1
- new net: D37.1 (K), R37.1
- new net: D36.1 (K), R36.1
- new net: D20.1 (K), R20.1
- new net: D15.1 (K), R15.1
- new net: D33.1 (K), R33.1
- new net: D18.1 (K), R18.1
- new net: D32.1 (K), R32.1
- new net: D34.1 (K), R34.1
- new net: D14.1 (K), R14.1
- new net: D30.1 (K), R30.1
- new net: D16.1 (K), R16.1
- new net: D31.1 (K), R31.1

Commit message: schematic updated
Parts:
- added D54: L-LOOP-D, Library:LED_YELLOW, symbol Device:LED_Filled
- added D55: R-LOOP-D, Library:LED_YELLOW, symbol Device:LED_Filled
- added R54: L-LOOP-R, Library:R_1206_3216Metric_Pad1.30x1.75mm_HandSolder, symbol Device:R_Small
- added R55: R-LOOP-R, Library:R_1206_3216Metric_Pad1.30x1.75mm_HandSolder, symbol Device:R_Small
Connections:
- net GND: now also R54.2, R55.2
- new net: D54.1 (K), R54.1
- new net: D55.1 (K), R55.1
- new net LEDLOOPL: D54.2 (A)
- new net LEDLOOPR: D55.2 (A)
Other:
- moved on the sheet: D22, D23, D24, R22, R23, R24

Commit message: SCHEMATIC FINISHED
Parts:
- removed D1: VUL1D1, Library:LED_GREEN, symbol Device:LED_Filled
- removed D10: LCUE-D, Library:LED_YELLOW, symbol Device:LED_Filled
- removed D11: LFX1-D, Library:LED_GREEN, symbol Device:LED_Filled
- removed D12: LFX2-D, Library:LED_YELLOW, symbol Device:LED_Filled
- removed D13: LFX3-D, Library:LED_YELLOW, symbol Device:LED_Filled
- removed D14: VUL2D1, Library:LED_GREEN, symbol Device:LED_Filled
- removed D15: VUL2D2, Library:LED_GREEN, symbol Device:LED_Filled
- removed D16: VUL2D3, Library:LED_GREEN, symbol Device:LED_Filled
- removed D17: VUL2D4, Library:LED_GREEN, symbol Device:LED_Filled
- removed D18: VUL2D5, Library:LED_GREEN, symbol Device:LED_Filled
- removed D19: VUL2D6, Library:LED_YELLOW, symbol Device:LED_Filled
- removed D2: VUL1D2, Library:LED_GREEN, symbol Device:LED_Filled
- removed D20: VUL2D7, Library:LED_YELLOW, symbol Device:LED_Filled
- removed D21: VUL2D8, Library:LED_RED, symbol Device:LED_Filled
- removed D22: L1HP-D, Library:LED_YELLOW, symbol Device:LED_Filled
- removed D23: L2HP-D, Library:LED_YELLOW, symbol Device:LED_Filled
- removed D24: L3HP-D, Library:LED_YELLOW, symbol Device:LED_Filled
- removed D25: RPLAY-D, Library:LED_GREEN, symbol Device:LED_Filled
- removed D26: RCUE-D, Library:LED_YELLOW, symbol Device:LED_Filled
- removed D27: RFX1-D, Library:LED_GREEN, symbol Device:LED_Filled
- removed D28: RFX2-D, Library:LED_YELLOW, symbol Device:LED_Filled
- removed D29: RFX3-D, Library:LED_YELLOW, symbol Device:LED_Filled
- removed D3: VUL1D3, Library:LED_GREEN, symbol Device:LED_Filled
- removed D30: VUL3D1, Library:LED_GREEN, symbol Device:LED_Filled
- removed D31: VUL3D2, Library:LED_GREEN, symbol Device:LED_Filled
- removed D32: VUL3D3, Library:LED_GREEN, symbol Device:LED_Filled
- removed D33: VUL3D4, Library:LED_GREEN, symbol Device:LED_Filled
- removed D34: VUL3D5, Library:LED_GREEN, symbol Device:LED_Filled
- removed D35: VUL3D6, Library:LED_YELLOW, symbol Device:LED_Filled
- removed D36: VUL3D7, Library:LED_YELLOW, symbol Device:LED_Filled
- removed D37: VUL3D8, Library:LED_RED, symbol Device:LED_Filled
- removed D38: VUMASLD1, Library:LED_GREEN, symbol Device:LED_Filled
- removed D39: VUMASLD2, Library:LED_GREEN, symbol Device:LED_Filled
- removed D4: VUL1D4, Library:LED_GREEN, symbol Device:LED_Filled
- removed D40: VUMASLD3, Library:LED_GREEN, symbol Device:LED_Filled
- removed D41: VUMASLD4, Library:LED_GREEN, symbol Device:LED_Filled
- removed D42: VUMASLD5, Library:LED_GREEN, symbol Device:LED_Filled
- removed D43: VUMASLD6, Library:LED_YELLOW, symbol Device:LED_Filled
- removed D44: VUMASLD7, Library:LED_YELLOW, symbol Device:LED_Filled
- removed D45: VUMASLD8, Library:LED_RED, symbol Device:LED_Filled
- removed D46: VUMASRD1, Library:LED_GREEN, symbol Device:LED_Filled
- removed D47: VUMASRD2, Library:LED_GREEN, symbol Device:LED_Filled
- removed D48: VUMASRD3, Library:LED_GREEN, symbol Device:LED_Filled
- removed D49: VUMASRD4, Library:LED_GREEN, symbol Device:LED_Filled
- removed D5: VUL1D5, Library:LED_GREEN, symbol Device:LED_Filled
- removed D50: VUMASRD5, Library:LED_GREEN, symbol Device:LED_Filled
- removed D51: VUMASRD6, Library:LED_YELLOW, symbol Device:LED_Filled
- removed D52: VUMASRD7, Library:LED_YELLOW, symbol Device:LED_Filled
- removed D53: VUMASRD8, Library:LED_RED, symbol Device:LED_Filled
- removed D54: L-LOOP-D, Library:LED_YELLOW, symbol Device:LED_Filled
- removed D55: R-LOOP-D, Library:LED_YELLOW, symbol Device:LED_Filled
- removed D6: VUL1D6, Library:LED_YELLOW, symbol Device:LED_Filled
- removed D7: VUL1D7, Library:LED_YELLOW, symbol Device:LED_Filled
- removed D8: VUL1D8, Library:LED_RED, symbol Device:LED_Filled
- removed D9: LPLAY-D, Library:LED_GREEN, symbol Device:LED_Filled
- removed R1: VUL1R1, Library:R_1206_3216Metric_Pad1.30x1.75mm_HandSolder, symbol Device:R_Small
- removed R10: LCUE-R, Library:R_1206_3216Metric_Pad1.30x1.75mm_HandSolder, symbol Device:R_Small
- removed R11: LFX1R, Library:R_1206_3216Metric_Pad1.30x1.75mm_HandSolder, symbol Device:R_Small
- removed R12: LFX2R, Library:R_1206_3216Metric_Pad1.30x1.75mm_HandSolder, symbol Device:R_Small
- removed R13: LFX3R, Library:R_1206_3216Metric_Pad1.30x1.75mm_HandSolder, symbol Device:R_Small
- removed R14: VUL2R1, Library:R_1206_3216Metric_Pad1.30x1.75mm_HandSolder, symbol Device:R_Small
- removed R15: VUL2R2, Library:R_1206_3216Metric_Pad1.30x1.75mm_HandSolder, symbol Device:R_Small
- removed R16: VUL2R3, Library:R_1206_3216Metric_Pad1.30x1.75mm_HandSolder, symbol Device:R_Small
- removed R17: VUL2R4, Library:R_1206_3216Metric_Pad1.30x1.75mm_HandSolder, symbol Device:R_Small
- removed R18: VUL2R5, Library:R_1206_3216Metric_Pad1.30x1.75mm_HandSolder, symbol Device:R_Small
- removed R19: VUL2R6, Library:R_1206_3216Metric_Pad1.30x1.75mm_HandSolder, symbol Device:R_Small
- removed R2: VUL1R2, Library:R_1206_3216Metric_Pad1.30x1.75mm_HandSolder, symbol Device:R_Small
- removed R20: VUL2R7, Library:R_1206_3216Metric_Pad1.30x1.75mm_HandSolder, symbol Device:R_Small
- removed R21: VUL2R8, Library:R_1206_3216Metric_Pad1.30x1.75mm_HandSolder, symbol Device:R_Small
- removed R22: L1HP-R, Library:R_1206_3216Metric_Pad1.30x1.75mm_HandSolder, symbol Device:R_Small
- removed R23: L2HP-R, Library:R_1206_3216Metric_Pad1.30x1.75mm_HandSolder, symbol Device:R_Small
- removed R24: L3HP-R, Library:R_1206_3216Metric_Pad1.30x1.75mm_HandSolder, symbol Device:R_Small
- removed R25: RPLAY-R, Library:R_1206_3216Metric_Pad1.30x1.75mm_HandSolder, symbol Device:R_Small
- removed R26: RCUE-R, Library:R_1206_3216Metric_Pad1.30x1.75mm_HandSolder, symbol Device:R_Small
- removed R27: RFX1-R, Library:R_1206_3216Metric_Pad1.30x1.75mm_HandSolder, symbol Device:R_Small
- removed R28: RFX2-R, Library:R_1206_3216Metric_Pad1.30x1.75mm_HandSolder, symbol Device:R_Small
- removed R29: RFX3-R, Library:R_1206_3216Metric_Pad1.30x1.75mm_HandSolder, symbol Device:R_Small
- removed R3: VUL1R3, Library:R_1206_3216Metric_Pad1.30x1.75mm_HandSolder, symbol Device:R_Small
- removed R30: VUL3R1, Library:R_1206_3216Metric_Pad1.30x1.75mm_HandSolder, symbol Device:R_Small
- removed R31: VUL3R2, Library:R_1206_3216Metric_Pad1.30x1.75mm_HandSolder, symbol Device:R_Small
- removed R32: VUL3R3, Library:R_1206_3216Metric_Pad1.30x1.75mm_HandSolder, symbol Device:R_Small
- removed R33: VUL3R4, Library:R_1206_3216Metric_Pad1.30x1.75mm_HandSolder, symbol Device:R_Small
- removed R34: VUL3R5, Library:R_1206_3216Metric_Pad1.30x1.75mm_HandSolder, symbol Device:R_Small
- removed R35: VUL3R6, Library:R_1206_3216Metric_Pad1.30x1.75mm_HandSolder, symbol Device:R_Small
- removed R36: VUL3R7, Library:R_1206_3216Metric_Pad1.30x1.75mm_HandSolder, symbol Device:R_Small
- removed R37: VUL3R8, Library:R_1206_3216Metric_Pad1.30x1.75mm_HandSolder, symbol Device:R_Small
- removed R38: VUMASLR1, Library:R_1206_3216Metric_Pad1.30x1.75mm_HandSolder, symbol Device:R_Small
- removed R39: VUMASLR2, Library:R_1206_3216Metric_Pad1.30x1.75mm_HandSolder, symbol Device:R_Small
- removed R4: VUL1R4, Library:R_1206_3216Metric_Pad1.30x1.75mm_HandSolder, symbol Device:R_Small
- removed R40: VUMASLR3, Library:R_1206_3216Metric_Pad1.30x1.75mm_HandSolder, symbol Device:R_Small
- removed R41: VUMASLR4, Library:R_1206_3216Metric_Pad1.30x1.75mm_HandSolder, symbol Device:R_Small
- removed R42: VUMASLR5, Library:R_1206_3216Metric_Pad1.30x1.75mm_HandSolder, symbol Device:R_Small
- removed R43: VUMASLR6, Library:R_1206_3216Metric_Pad1.30x1.75mm_HandSolder, symbol Device:R_Small
- removed R44: VUMASLR7, Library:R_1206_3216Metric_Pad1.30x1.75mm_HandSolder, symbol Device:R_Small
- removed R45: VUMASLR8, Library:R_1206_3216Metric_Pad1.30x1.75mm_HandSolder, symbol Device:R_Small
- removed R46: VUMASRR1, Library:R_1206_3216Metric_Pad1.30x1.75mm_HandSolder, symbol Device:R_Small
- removed R47: VUMASRR2, Library:R_1206_3216Metric_Pad1.30x1.75mm_HandSolder, symbol Device:R_Small
- removed R48: VUMASRR3, Library:R_1206_3216Metric_Pad1.30x1.75mm_HandSolder, symbol Device:R_Small
- removed R49: VUMASRR4, Library:R_1206_3216Metric_Pad1.30x1.75mm_HandSolder, symbol Device:R_Small
- removed R5: VUL1R5, Library:R_1206_3216Metric_Pad1.30x1.75mm_HandSolder, symbol Device:R_Small
- removed R50: VUMASRR5, Library:R_1206_3216Metric_Pad1.30x1.75mm_HandSolder, symbol Device:R_Small
- removed R51: VUMASRR6, Library:R_1206_3216Metric_Pad1.30x1.75mm_HandSolder, symbol Device:R_Small
- removed R52: VUMASRR7, Library:R_1206_3216Metric_Pad1.30x1.75mm_HandSolder, symbol Device:R_Small
- removed R53: VUMASRR8, Library:R_1206_3216Metric_Pad1.30x1.75mm_HandSolder, symbol Device:R_Small
- removed R54: L-LOOP-R, Library:R_1206_3216Metric_Pad1.30x1.75mm_HandSolder, symbol Device:R_Small
- removed R55: R-LOOP-R, Library:R_1206_3216Metric_Pad1.30x1.75mm_HandSolder, symbol Device:R_Small
- removed R6: VUL1R6, Library:R_1206_3216Metric_Pad1.30x1.75mm_HandSolder, symbol Device:R_Small
- removed R7: VUL1R7, Library:R_1206_3216Metric_Pad1.30x1.75mm_HandSolder, symbol Device:R_Small
- removed R8: VUL1R8, Library:R_1206_3216Metric_Pad1.30x1.75mm_HandSolder, symbol Device:R_Small
- removed R9: LPLAY-R, Library:R_1206_3216Metric_Pad1.30x1.75mm_HandSolder, symbol Device:R_Small
Other:
- added sheet VU Line 1 Sheet (VU-L1.kicad_sch)
- added sheet VU Line 2 (VU-L3.kicad_sch)
- added sheet VU Line 3  (VU-L3.kicad_sch)
- added sheet VU Master Left (VU-ML.kicad_sch)
- added sheet VU Master Right (VU-MR.kicad_sch)
- note removed: "LINE 1"
- note removed: "LINE 2"
- note removed: "LINE 3"
- note removed: "MASTER LEFT"
- note removed: "MASTER RIGHT"
