File: PCB/Kicad/neopixels.kicad_sch (KiCad schematic)
At the start: 22 parts

Commit message: SCHEMATIC FINISHED
Parts:
- renumbered NP4 to NP10, NP14 to NP11, NP5 to NP12, NP6 to NP13, NP15 to NP14, NP7 to NP15, NP8 to NP17, NP17 to NP18, NP9 to NP19, NP19 to NP2, NP10 to NP20, NP18 to NP21, NP11 to NP3, NP2 to NP4, NP20 to NP5, NP12 to NP6, NP3 to NP7, NP21 to NP8, NP13 to NP9
Connections:
- no-connect marks 2 -> 1
Changed lines of the file:
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@@
-(kicad_sch (version 20210615) (generator eeschema)
+(kicad_sch (version 20210621) (generator eeschema)
   (paper "A4")
-  (no_connect (at 48.895 99.695))
-  (no_connect (at 110.49 132.715))
+  (no_connect (at 107.95 132.715))
   (wire (pts (xy 24.765 64.135) (xy 28.575 64.135))
     (stroke (width 0) (type solid) (color 0 0 0 0))
@@
   )
   (wire (pts (xy 93.98 64.135) (xy 99.695 64.135))
-    (stroke (width 0) (type solid) (color 0 0 0 0))
-  )
-  (wire (pts (xy 107.95 132.715) (xy 110.49 132.715))
     (stroke (width 0) (type solid) (color 0 0 0 0))
   )
@@
   (symbol (lib_id "mixduino-mk2:WS2812B") (at 48.895 132.715 0) (unit 1)
     (in_bom yes) (on_board yes)
-    (property "Reference" "NP19" (id 0) (at 53.975 127 0)
+    (property "Reference" "NP2" (id 0) (at 53.975 127 0)
       (effects (font (size 1.27 1.27)) (justify right bottom))
     )
@@
   (symbol (lib_id "mixduino-mk2:WS2812B") (at 49.53 99.695 180) (unit 1)
     (in_bom yes) (on_board yes)
-    (property "Reference" "NP11" (id 0) (at 44.45 105.41 0)
+    (property "Reference" "NP3" (id 0) (at 44.45 105.41 0)
       (effects (font (size 1.27 1.27)) (justify right bottom))
     )
@@
   (symbol (lib_id "mixduino-mk2:WS2812B") (at 65.405 64.135 0) (unit 1)
     (in_bom yes) (on_board yes)
-    (property "Reference" "NP2" (id 0) (at 70.485 58.42 0)
+    (property "Reference" "NP4" (id 0) (at 70.485 58.42 0)
       (effects (font (size 1.27 1.27)) (justify right bottom))
     )
@@
   (symbol (lib_id "mixduino-mk2:WS2812B") (at 74.295 132.715 0) (unit 1)
     (in_bom yes) (on_board yes)
-    (property "Reference" "NP20" (id 0) (at 79.375 127 0)
+    (property "Reference" "NP5" (id 0) (at 79.375 127 0)
       (effects (font (size 1.27 1.27)) (justify right bottom))
     )
@@
   (symbol (lib_id "mixduino-mk2:WS2812B") (at 74.93 99.695 180) (unit 1)
     (in_bom yes) (on_board yes)
-    (property "Reference" "NP12" (id 0) (at 69.85 105.41 0)
+    (property "Reference" "NP6" (id 0) (at 69.85 105.41 0)
       (effects (font (size 1.27 1.27)) (justify right bottom))
     )
@@
   (symbol (lib_id "mixduino-mk2:WS2812B") (at 86.36 64.135 0) (unit 1)
     (in_bom yes) (on_board yes)
-    (property "Reference" "NP3" (id 0) (at 91.44 58.42 0)
+    (property "Reference" "NP7" (id 0) (at 91.44 58.42 0)
       (effects (font (size 1.27 1.27)) (justify right bottom))
     )
@@
   (symbol (lib_id "mixduino-mk2:WS2812B") (at 100.33 132.715 0) (unit 1)
     (in_bom yes) (on_board yes)
-    (property "Reference" "NP21" (id 0) (at 105.41 127 0)
+    (property "Reference" "NP8" (id 0) (at 105.41 127 0)
       (effects (font (size 1.27 1.27)) (justify right bottom))
     )
@@
   (symbol (lib_id "mixduino-mk2:WS2812B") (at 100.965 99.695 180) (unit 1)
     (in_bom yes) (on_board yes)
-    (property "Reference" "NP13" (id 0) (at 95.885 105.41 0)
+    (property "Reference" "NP9" (id 0) (at 95.885 105.41 0)
       (effects (font (size 1.27 1.27)) (justify right bottom))
     )
@@
   (symbol (lib_id "mixduino-mk2:WS2812B") (at 107.315 64.135 0) (unit 1)
     (in_bom yes) (on_board yes)
-    (property "Reference" "NP4" (id 0) (at 112.395 58.42 0)
+    (property "Reference" "NP10" (id 0) (at 112.395 58.42 0)
       (effects (font (size 1.27 1.27)) (justify right bottom))
     )
@@
   (symbol (lib_id "mixduino-mk2:WS2812B") (at 126.365 99.695 180) (unit 1)
     (in_bom yes) (on_board yes)
-    (property "Reference" "NP14" (id 0) (at 121.285 105.41 0)
+    (property "Reference" "NP11" (id 0) (at 121.285 105.41 0)
       (effects (font (size 1.27 1.27)) (justify right bottom))
     )
@@
   (symbol (lib_id "mixduino-mk2:WS2812B") (at 127.635 64.135 0) (unit 1)
     (in_bom yes) (on_board yes)
-    (property "Reference" "NP5" (id 0) (at 132.715 58.42 0)
+    (property "Reference" "NP12" (id 0) (at 132.715 58.42 0)
       (effects (font (size 1.27 1.27)) (justify right bottom))
     )
@@
   (symbol (lib_id "mixduino-mk2:WS2812B") (at 148.59 64.135 0) (unit 1)
     (in_bom yes) (on_board yes)
-    (property "Reference" "NP6" (id 0) (at 153.67 58.42 0)
+    (property "Reference" "NP13" (id 0) (at 153.67 58.42 0)
       (effects (font (size 1.27 1.27)) (justify right bottom))
     )
@@
   (symbol (lib_id "mixduino-mk2:WS2812B") (at 150.495 99.695 180) (unit 1)
     (in_bom yes) (on_board yes)
-    (property "Reference" "NP15" (id 0) (at 145.415 105.41 0)
+    (property "Reference" "NP14" (id 0) (at 145.415 105.41 0)
       (effects (font (size 1.27 1.27)) (justify right bottom))
     )
@@
   (symbol (lib_id "mixduino-mk2:WS2812B") (at 169.545 64.135 0) (unit 1)
     (in_bom yes) (on_board yes)
-    (property "Reference" "NP7" (id 0) (at 174.625 58.42 0)
+    (property "Reference" "NP15" (id 0) (at 174.625 58.42 0)
       (effects (font (size 1.27 1.27)) (justify right bottom))
     )
@@
   (symbol (lib_id "mixduino-mk2:WS2812B") (at 189.23 64.135 0) (unit 1)
     (in_bom yes) (on_board yes)
-    (property "Reference" "NP8" (id 0) (at 194.31 58.42 0)
+    (property "Reference" "NP17" (id 0) (at 194.31 58.42 0)
       (effects (font (size 1.27 1.27)) (justify right bottom))
     )
@@
   (symbol (lib_id "mixduino-mk2:WS2812B") (at 201.93 99.695 180) (unit 1)
     (in_bom yes) (on_board yes)
-    (property "Reference" "NP17" (id 0) (at 196.85 105.41 0)
+    (property "Reference" "NP18" (id 0) (at 196.85 105.41 0)
       (effects (font (size 1.27 1.27)) (justify right bottom))
     )
@@
   (symbol (lib_id "mixduino-mk2:WS2812B") (at 207.645 64.135 0) (unit 1)
     (in_bom yes) (on_board yes)
-    (property "Reference" "NP9" (id 0) (at 212.725 58.42 0)
+    (property "Reference" "NP19" (id 0) (at 212.725 58.42 0)
       (effects (font (size 1.27 1.27)) (justify right bottom))
     )
@@
   (symbol (lib_id "mixduino-mk2:WS2812B") (at 227.33 64.135 0) (unit 1)
     (in_bom yes) (on_board yes)
-    (property "Reference" "NP10" (id 0) (at 232.41 58.42 0)
+    (property "Reference" "NP20" (id 0) (at 232.41 58.42 0)
       (effects (font (size 1.27 1.27)) (justify right bottom))
     )
@@
   (symbol (lib_id "mixduino-mk2:WS2812B") (at 227.33 99.695 180) (unit 1)
     (in_bom yes) (on_board yes)
-    (property "Reference" "NP18" (id 0) (at 222.25 105.41 0)
-      (effects (font (size 1.27 1.27)) (justify right bottom))
-    )
+    (property "Reference" "NP21" (id 0) (at 222.25 105.41 0)
+      (effects (font (size 1.27 1.27)) (justify right bottom))
+    )
