File: PCB/Kicad/neopixels.kicad_sch (KiCad schematic)
At the start: 22 parts

Commit message: routing WIP
Parts:
- renumbered NP20 to NP10, NP3 to NP11, NP6 to NP12, NP9 to NP13, NP11 to NP14, NP14 to NP15, NP18 to NP17, NP21 to NP18, NP2 to NP19, NP4 to NP2, NP5 to NP20, NP8 to NP21, NP7 to NP3, NP10 to NP4, NP12 to NP5, NP13 to NP6, NP15 to NP7, NP17 to NP8, NP19 to NP9
Changed lines of the file:
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@@
   (symbol (lib_id "mixduino-mk2:WS2812B") (at 48.895 132.715 0) (unit 1)
     (in_bom yes) (on_board yes)
-    (property "Reference" "NP2" (id 0) (at 53.975 127 0)
+    (property "Reference" "NP19" (id 0) (at 53.975 127 0)
       (effects (font (size 1.27 1.27)) (justify right bottom))
     )
@@
   (symbol (lib_id "mixduino-mk2:WS2812B") (at 49.53 99.695 180) (unit 1)
     (in_bom yes) (on_board yes)
-    (property "Reference" "NP3" (id 0) (at 44.45 105.41 0)
+    (property "Reference" "NP11" (id 0) (at 44.45 105.41 0)
       (effects (font (size 1.27 1.27)) (justify right bottom))
     )
@@
   (symbol (lib_id "mixduino-mk2:WS2812B") (at 65.405 64.135 0) (unit 1)
     (in_bom yes) (on_board yes)
-    (property "Reference" "NP4" (id 0) (at 70.485 58.42 0)
+    (property "Reference" "NP2" (id 0) (at 70.485 58.42 0)
       (effects (font (size 1.27 1.27)) (justify right bottom))
     )
@@
   (symbol (lib_id "mixduino-mk2:WS2812B") (at 74.295 132.715 0) (unit 1)
     (in_bom yes) (on_board yes)
-    (property "Reference" "NP5" (id 0) (at 79.375 127 0)
+    (property "Reference" "NP20" (id 0) (at 79.375 127 0)
       (effects (font (size 1.27 1.27)) (justify right bottom))
     )
@@
   (symbol (lib_id "mixduino-mk2:WS2812B") (at 74.93 99.695 180) (unit 1)
     (in_bom yes) (on_board yes)
-    (property "Reference" "NP6" (id 0) (at 69.85 105.41 0)
+    (property "Reference" "NP12" (id 0) (at 69.85 105.41 0)
       (effects (font (size 1.27 1.27)) (justify right bottom))
     )
@@
   (symbol (lib_id "mixduino-mk2:WS2812B") (at 86.36 64.135 0) (unit 1)
     (in_bom yes) (on_board yes)
-    (property "Reference" "NP7" (id 0) (at 91.44 58.42 0)
+    (property "Reference" "NP3" (id 0) (at 91.44 58.42 0)
       (effects (font (size 1.27 1.27)) (justify right bottom))
     )
@@
   (symbol (lib_id "mixduino-mk2:WS2812B") (at 100.33 132.715 0) (unit 1)
     (in_bom yes) (on_board yes)
-    (property "Reference" "NP8" (id 0) (at 105.41 127 0)
+    (property "Reference" "NP21" (id 0) (at 105.41 127 0)
       (effects (font (size 1.27 1.27)) (justify right bottom))
     )
@@
   (symbol (lib_id "mixduino-mk2:WS2812B") (at 100.965 99.695 180) (unit 1)
     (in_bom yes) (on_board yes)
-    (property "Reference" "NP9" (id 0) (at 95.885 105.41 0)
+    (property "Reference" "NP13" (id 0) (at 95.885 105.41 0)
       (effects (font (size 1.27 1.27)) (justify right bottom))
     )
@@
   (symbol (lib_id "mixduino-mk2:WS2812B") (at 107.315 64.135 0) (unit 1)
     (in_bom yes) (on_board yes)
-    (property "Reference" "NP10" (id 0) (at 112.395 58.42 0)
+    (property "Reference" "NP4" (id 0) (at 112.395 58.42 0)
       (effects (font (size 1.27 1.27)) (justify right bottom))
     )
@@
   (symbol (lib_id "mixduino-mk2:WS2812B") (at 126.365 99.695 180) (unit 1)
     (in_bom yes) (on_board yes)
-    (property "Reference" "NP11" (id 0) (at 121.285 105.41 0)
+    (property "Reference" "NP14" (id 0) (at 121.285 105.41 0)
       (effects (font (size 1.27 1.27)) (justify right bottom))
     )
@@
   (symbol (lib_id "mixduino-mk2:WS2812B") (at 127.635 64.135 0) (unit 1)
     (in_bom yes) (on_board yes)
-    (property "Reference" "NP12" (id 0) (at 132.715 58.42 0)
+    (property "Reference" "NP5" (id 0) (at 132.715 58.42 0)
       (effects (font (size 1.27 1.27)) (justify right bottom))
     )
@@
   (symbol (lib_id "mixduino-mk2:WS2812B") (at 148.59 64.135 0) (unit 1)
     (in_bom yes) (on_board yes)
-    (property "Reference" "NP13" (id 0) (at 153.67 58.42 0)
+    (property "Reference" "NP6" (id 0) (at 153.67 58.42 0)
       (effects (font (size 1.27 1.27)) (justify right bottom))
     )
@@
   (symbol (lib_id "mixduino-mk2:WS2812B") (at 150.495 99.695 180) (unit 1)
     (in_bom yes) (on_board yes)
-    (property "Reference" "NP14" (id 0) (at 145.415 105.41 0)
+    (property "Reference" "NP15" (id 0) (at 145.415 105.41 0)
       (effects (font (size 1.27 1.27)) (justify right bottom))
     )
@@
   (symbol (lib_id "mixduino-mk2:WS2812B") (at 169.545 64.135 0) (unit 1)
     (in_bom yes) (on_board yes)
-    (property "Reference" "NP15" (id 0) (at 174.625 58.42 0)
+    (property "Reference" "NP7" (id 0) (at 174.625 58.42 0)
       (effects (font (size 1.27 1.27)) (justify right bottom))
     )
@@
   (symbol (lib_id "mixduino-mk2:WS2812B") (at 189.23 64.135 0) (unit 1)
     (in_bom yes) (on_board yes)
-    (property "Reference" "NP17" (id 0) (at 194.31 58.42 0)
+    (property "Reference" "NP8" (id 0) (at 194.31 58.42 0)
       (effects (font (size 1.27 1.27)) (justify right bottom))
     )
@@
   (symbol (lib_id "mixduino-mk2:WS2812B") (at 201.93 99.695 180) (unit 1)
     (in_bom yes) (on_board yes)
-    (property "Reference" "NP18" (id 0) (at 196.85 105.41 0)
+    (property "Reference" "NP17" (id 0) (at 196.85 105.41 0)
       (effects (font (size 1.27 1.27)) (justify right bottom))
     )
@@
   (symbol (lib_id "mixduino-mk2:WS2812B") (at 207.645 64.135 0) (unit 1)
     (in_bom yes) (on_board yes)
-    (property "Reference" "NP19" (id 0) (at 212.725 58.42 0)
+    (property "Reference" "NP9" (id 0) (at 212.725 58.42 0)
       (effects (font (size 1.27 1.27)) (justify right bottom))
     )
@@
   (symbol (lib_id "mixduino-mk2:WS2812B") (at 227.33 64.135 0) (unit 1)
     (in_bom yes) (on_board yes)
-    (property "Reference" "NP20" (id 0) (at 232.41 58.42 0)
+    (property "Reference" "NP10" (id 0) (at 232.41 58.42 0)
       (effects (font (size 1.27 1.27)) (justify right bottom))
     )
@@
   (symbol (lib_id "mixduino-mk2:WS2812B") (at 227.33 99.695 180) (unit 1)
     (in_bom yes) (on_board yes)
-    (property "Reference" "NP21" (id 0) (at 222.25 105.41 0)
-      (effects (font (size 1.27 1.27)) (justify right bottom))
-    )
+    (property "Reference" "NP18" (id 0) (at 222.25 105.41 0)
+      (effects (font (size 1.27 1.27)) (justify right bottom))
+    )

Commit message: update schematic
Parts:
- NP1, NP10, NP11, NP12, NP13, NP14, NP15, NP16, NP17, NP18, NP19, NP2, NP20, NP21, NP3, NP4, NP5, NP6, NP7, NP8, NP9: footprint Library:LED_WS2812B_PLCC4_5.0x5.0mm_P3.2mm -> LED_SMD:LED_WS2812B_PLCC4_5.0x5.0mm_P3.2mm
- NPR1: footprint Library:R_1206_3216Metric_Pad1.30x1.75mm_HandSolder -> Resistor_SMD:R_1206_3216Metric_Pad1.30x1.75mm_HandSolder
Changed lines of the file:
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@@
     (property "Reference" "NPR1" (id 0) (at 31.115 61.595 90))
     (property "Value" "L-NP-PADS_R" (id 1) (at 31.115 66.675 90))
-    (property "Footprint" "Library:R_1206_3216Metric_Pad1.30x1.75mm_HandSolder" (id 2) (at 31.115 64.135 0)
+    (property "Footprint" "Resistor_SMD:R_1206_3216Metric_Pad1.30x1.75mm_HandSolder" (id 2) (at 31.115 64.135 0)
       (effects (font (size 1.27 1.27)) hide)
     )
@@
       (effects (font (size 1.27 1.27)) (justify left))
     )
-    (property "Footprint" "Library:LED_WS2812B_PLCC4_5.0x5.0mm_P3.2mm" (id 2) (at 45.085 71.755 0)
+    (property "Footprint" "LED_SMD:LED_WS2812B_PLCC4_5.0x5.0mm_P3.2mm" (id 2) (at 45.085 71.755 0)
       (effects (font (size 1.27 1.27)) (justify left top) hide)
     )
@@
       (effects (font (size 1.27 1.27)) (justify left))
     )
-    (property "Footprint" "Library:LED_WS2812B_PLCC4_5.0x5.0mm_P3.2mm" (id 2) (at 50.165 140.335 0)
+    (property "Footprint" "LED_SMD:LED_WS2812B_PLCC4_5.0x5.0mm_P3.2mm" (id 2) (at 50.165 140.335 0)
       (effects (font (size 1.27 1.27)) (justify left top) hide)
     )
@@
       (effects (font (size 1.27 1.27)) (justify left))
     )
-    (property "Footprint" "Library:LED_WS2812B_PLCC4_5.0x5.0mm_P3.2mm" (id 2) (at 48.26 92.075 0)
+    (property "Footprint" "LED_SMD:LED_WS2812B_PLCC4_5.0x5.0mm_P3.2mm" (id 2) (at 48.26 92.075 0)
       (effects (font (size 1.27 1.27)) (justify left top) hide)
     )
@@
       (effects (font (size 1.27 1.27)) (justify left))
     )
-    (property "Footprint" "Library:LED_WS2812B_PLCC4_5.0x5.0mm_P3.2mm" (id 2) (at 66.675 71.755 0)
+    (property "Footprint" "LED_SMD:LED_WS2812B_PLCC4_5.0x5.0mm_P3.2mm" (id 2) (at 66.675 71.755 0)
       (effects (font (size 1.27 1.27)) (justify left top) hide)
     )
@@
       (effects (font (size 1.27 1.27)) (justify left))
     )
-    (property "Footprint" "Library:LED_WS2812B_PLCC4_5.0x5.0mm_P3.2mm" (id 2) (at 75.565 140.335 0)
+    (property "Footprint" "LED_SMD:LED_WS2812B_PLCC4_5.0x5.0mm_P3.2mm" (id 2) (at 75.565 140.335 0)
       (effects (font (size 1.27 1.27)) (justify left top) hide)
     )
@@
       (effects (font (size 1.27 1.27)) (justify left))
     )
-    (property "Footprint" "Library:LED_WS2812B_PLCC4_5.0x5.0mm_P3.2mm" (id 2) (at 73.66 92.075 0)
+    (property "Footprint" "LED_SMD:LED_WS2812B_PLCC4_5.0x5.0mm_P3.2mm" (id 2) (at 73.66 92.075 0)
       (effects (font (size 1.27 1.27)) (justify left top) hide)
     )
@@
       (effects (font (size 1.27 1.27)) (justify left))
     )
-    (property "Footprint" "Library:LED_WS2812B_PLCC4_5.0x5.0mm_P3.2mm" (id 2) (at 87.63 71.755 0)
+    (property "Footprint" "LED_SMD:LED_WS2812B_PLCC4_5.0x5.0mm_P3.2mm" (id 2) (at 87.63 71.755 0)
       (effects (font (size 1.27 1.27)) (justify left top) hide)
     )
@@
       (effects (font (size 1.27 1.27)) (justify left))
     )
-    (property "Footprint" "Library:LED_WS2812B_PLCC4_5.0x5.0mm_P3.2mm" (id 2) (at 101.6 140.335 0)
+    (property "Footprint" "LED_SMD:LED_WS2812B_PLCC4_5.0x5.0mm_P3.2mm" (id 2) (at 101.6 140.335 0)
       (effects (font (size 1.27 1.27)) (justify left top) hide)
     )
@@
       (effects (font (size 1.27 1.27)) (justify left))
     )
-    (property "Footprint" "Library:LED_WS2812B_PLCC4_5.0x5.0mm_P3.2mm" (id 2) (at 99.695 92.075 0)
+    (property "Footprint" "LED_SMD:LED_WS2812B_PLCC4_5.0x5.0mm_P3.2mm" (id 2) (at 99.695 92.075 0)
       (effects (font (size 1.27 1.27)) (justify left top) hide)
     )
@@
       (effects (font (size 1.27 1.27)) (justify left))
     )
-    (property "Footprint" "Library:LED_WS2812B_PLCC4_5.0x5.0mm_P3.2mm" (id 2) (at 108.585 71.755 0)
+    (property "Footprint" "LED_SMD:LED_WS2812B_PLCC4_5.0x5.0mm_P3.2mm" (id 2) (at 108.585 71.755 0)
       (effects (font (size 1.27 1.27)) (justify left top) hide)
     )
@@
       (effects (font (size 1.27 1.27)) (justify left))
     )
-    (property "Footprint" "Library:LED_WS2812B_PLCC4_5.0x5.0mm_P3.2mm" (id 2) (at 125.095 92.075 0)
+    (property "Footprint" "LED_SMD:LED_WS2812B_PLCC4_5.0x5.0mm_P3.2mm" (id 2) (at 125.095 92.075 0)
       (effects (font (size 1.27 1.27)) (justify left top) hide)
     )
@@
       (effects (font (size 1.27 1.27)) (justify left))
     )
-    (property "Footprint" "Library:LED_WS2812B_PLCC4_5.0x5.0mm_P3.2mm" (id 2) (at 128.905 71.755 0)
+    (property "Footprint" "LED_SMD:LED_WS2812B_PLCC4_5.0x5.0mm_P3.2mm" (id 2) (at 128.905 71.755 0)
       (effects (font (size 1.27 1.27)) (justify left top) hide)
     )
@@
       (effects (font (size 1.27 1.27)) (justify left))
     )
-    (property "Footprint" "Library:LED_WS2812B_PLCC4_5.0x5.0mm_P3.2mm" (id 2) (at 149.86 71.755 0)
+    (property "Footprint" "LED_SMD:LED_WS2812B_PLCC4_5.0x5.0mm_P3.2mm" (id 2) (at 149.86 71.755 0)
       (effects (font (size 1.27 1.27)) (justify left top) hide)
     )
@@
       (effects (font (size 1.27 1.27)) (justify left))
     )
-    (property "Footprint" "Library:LED_WS2812B_PLCC4_5.0x5.0mm_P3.2mm" (id 2) (at 149.225 92.075 0)
+    (property "Footprint" "LED_SMD:LED_WS2812B_PLCC4_5.0x5.0mm_P3.2mm" (id 2) (at 149.225 92.075 0)
       (effects (font (size 1.27 1.27)) (justify left top) hide)
     )
@@
       (effects (font (size 1.27 1.27)) (justify left))
     )
-    (property "Footprint" "Library:LED_WS2812B_PLCC4_5.0x5.0mm_P3.2mm" (id 2) (at 170.815 71.755 0)
+    (property "Footprint" "LED_SMD:LED_WS2812B_PLCC4_5.0x5.0mm_P3.2mm" (id 2) (at 170.815 71.755 0)
       (effects (font (size 1.27 1.27)) (justify left top) hide)
     )
@@
       (effects (font (size 1.27 1.27)) (justify left))
     )
-    (property "Footprint" "Library:LED_WS2812B_PLCC4_5.0x5.0mm_P3.2mm" (id 2) (at 174.625 92.075 0)
+    (property "Footprint" "LED_SMD:LED_WS2812B_PLCC4_5.0x5.0mm_P3.2mm" (id 2) (at 174.625 92.075 0)
       (effects (font (size 1.27 1.27)) (justify left top) hide)
     )
@@
       (effects (font (size 1.27 1.27)) (justify left))
     )
-    (property "Footprint" "Library:LED_WS2812B_PLCC4_5.0x5.0mm_P3.2mm" (id 2) (at 190.5 71.755 0)
+    (property "Footprint" "LED_SMD:LED_WS2812B_PLCC4_5.0x5.0mm_P3.2mm" (id 2) (at 190.5 71.755 0)
       (effects (font (size 1.27 1.27)) (justify left top) hide)
     )
@@
       (effects (font (size 1.27 1.27)) (justify left))
     )
-    (property "Footprint" "Library:LED_WS2812B_PLCC4_5.0x5.0mm_P3.2mm" (id 2) (at 200.66 92.075 0)
+    (property "Footprint" "LED_SMD:LED_WS2812B_PLCC4_5.0x5.0mm_P3.2mm" (id 2) (at 200.66 92.075 0)
       (effects (font (size 1.27 1.27)) (justify left top) hide)
     )
@@
       (effects (font (size 1.27 1.27)) (justify left))
     )
-    (property "Footprint" "Library:LED_WS2812B_PLCC4_5.0x5.0mm_P3.2mm" (id 2) (at 208.915 71.755 0)
+    (property "Footprint" "LED_SMD:LED_WS2812B_PLCC4_5.0x5.0mm_P3.2mm" (id 2) (at 208.915 71.755 0)
       (effects (font (size 1.27 1.27)) (justify left top) hide)
     )
@@
       (effects (font (size 1.27 1.27)) (justify left))
     )
-    (property "Footprint" "Library:LED_WS2812B_PLCC4_5.0x5.0mm_P3.2mm" (id 2) (at 228.6 71.755 0)
+    (property "Footprint" "LED_SMD:LED_WS2812B_PLCC4_5.0x5.0mm_P3.2mm" (id 2) (at 228.6 71.755 0)
       (effects (font (size 1.27 1.27)) (justify left top) hide)
     )
@@
       (effects (font (size 1.27 1.27)) (justify left))
     )
-    (property "Footprint" "Library:LED_WS2812B_PLCC4_5.0x5.0mm_P3.2mm" (id 2) (at 226.06 92.075 0)
-      (effects (font (size 1.27 1.27)) (justify left top) hide)
-    )
+    (property "Footprint" "LED_SMD:LED_WS2812B_PLCC4_5.0x5.0mm_P3.2mm" (id 2) (at 226.06 92.075 0)
+      (effects (font (size 1.27 1.27)) (justify left top) hide)
+    )
