File: PCB/Kicad/potenciometers.kicad_sch (KiCad schematic)
At the start: 29 parts

Commit message: update elements WIP
Parts:
- gave numbers to parts that had none: 29

Commit message: progress
Parts:
- RV1, RV10, RV11, RV12, RV13, RV14, RV15, RV16, RV17, RV18, RV19, RV2, RV20, RV21, RV22, RV23, RV24, RV25, RV26, RV27, RV28, RV29, RV3, RV4, RV5, RV6, RV7, RV8, RV9: footprint (none) -> Potentiometer_THT:Potentiometer_Bourns_PTV09A-1_Single_Vertical
Changed lines of the file:
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@@
       (effects (font (size 1.27 1.27)) (justify right))
     )
-    (property "Footprint" "" (id 2) (at 27.94 25.4 0)
+    (property "Footprint" "Potentiometer_THT:Potentiometer_Bourns_PTV09A-1_Single_Vertical" (id 2) (at 27.94 25.4 0)
       (effects (font (size 1.27 1.27)) hide)
     )
@@
       (effects (font (size 1.27 1.27)) (justify right))
     )
-    (property "Footprint" "" (id 2) (at 27.94 57.15 0)
+    (property "Footprint" "Potentiometer_THT:Potentiometer_Bourns_PTV09A-1_Single_Vertical" (id 2) (at 27.94 57.15 0)
       (effects (font (size 1.27 1.27)) hide)
     )
@@
       (effects (font (size 1.27 1.27)) (justify right))
     )
-    (property "Footprint" "" (id 2) (at 27.94 88.9 0)
+    (property "Footprint" "Potentiometer_THT:Potentiometer_Bourns_PTV09A-1_Single_Vertical" (id 2) (at 27.94 88.9 0)
       (effects (font (size 1.27 1.27)) hide)
     )
@@
       (effects (font (size 1.27 1.27)) (justify right))
     )
-    (property "Footprint" "" (id 2) (at 27.94 120.65 0)
+    (property "Footprint" "Potentiometer_THT:Potentiometer_Bourns_PTV09A-1_Single_Vertical" (id 2) (at 27.94 120.65 0)
       (effects (font (size 1.27 1.27)) hide)
     )
@@
       (effects (font (size 1.27 1.27)) (justify right))
     )
-    (property "Footprint" "" (id 2) (at 29.21 151.13 0)
+    (property "Footprint" "Potentiometer_THT:Potentiometer_Bourns_PTV09A-1_Single_Vertical" (id 2) (at 29.21 151.13 0)
       (effects (font (size 1.27 1.27)) hide)
     )
@@
       (effects (font (size 1.27 1.27)) (justify right))
     )
-    (property "Footprint" "" (id 2) (at 29.21 180.34 0)
+    (property "Footprint" "Potentiometer_THT:Potentiometer_Bourns_PTV09A-1_Single_Vertical" (id 2) (at 29.21 180.34 0)
       (effects (font (size 1.27 1.27)) hide)
     )
@@
       (effects (font (size 1.27 1.27)) (justify right))
     )
-    (property "Footprint" "" (id 2) (at 63.5 25.4 0)
+    (property "Footprint" "Potentiometer_THT:Potentiometer_Bourns_PTV09A-1_Single_Vertical" (id 2) (at 63.5 25.4 0)
       (effects (font (size 1.27 1.27)) hide)
     )
@@
       (effects (font (size 1.27 1.27)) (justify right))
     )
-    (property "Footprint" "" (id 2) (at 63.5 57.15 0)
+    (property "Footprint" "Potentiometer_THT:Potentiometer_Bourns_PTV09A-1_Single_Vertical" (id 2) (at 63.5 57.15 0)
       (effects (font (size 1.27 1.27)) hide)
     )
@@
       (effects (font (size 1.27 1.27)) (justify right))
     )
-    (property "Footprint" "" (id 2) (at 63.5 88.9 0)
+    (property "Footprint" "Potentiometer_THT:Potentiometer_Bourns_PTV09A-1_Single_Vertical" (id 2) (at 63.5 88.9 0)
       (effects (font (size 1.27 1.27)) hide)
     )
@@
       (effects (font (size 1.27 1.27)) (justify right))
     )
-    (property "Footprint" "" (id 2) (at 63.5 120.65 0)
+    (property "Footprint" "Potentiometer_THT:Potentiometer_Bourns_PTV09A-1_Single_Vertical" (id 2) (at 63.5 120.65 0)
       (effects (font (size 1.27 1.27)) hide)
     )
@@
       (effects (font (size 1.27 1.27)) (justify right))
     )
-    (property "Footprint" "" (id 2) (at 64.77 151.13 0)
+    (property "Footprint" "Potentiometer_THT:Potentiometer_Bourns_PTV09A-1_Single_Vertical" (id 2) (at 64.77 151.13 0)
       (effects (font (size 1.27 1.27)) hide)
     )
@@
       (effects (font (size 1.27 1.27)) (justify right))
     )
-    (property "Footprint" "" (id 2) (at 64.77 180.34 0)
+    (property "Footprint" "Potentiometer_THT:Potentiometer_Bourns_PTV09A-1_Single_Vertical" (id 2) (at 64.77 180.34 0)
       (effects (font (size 1.27 1.27)) hide)
     )
@@
       (effects (font (size 1.27 1.27)) (justify right))
     )
-    (property "Footprint" "" (id 2) (at 100.33 25.4 0)
+    (property "Footprint" "Potentiometer_THT:Potentiometer_Bourns_PTV09A-1_Single_Vertical" (id 2) (at 100.33 25.4 0)
       (effects (font (size 1.27 1.27)) hide)
     )
@@
       (effects (font (size 1.27 1.27)) (justify right))
     )
-    (property "Footprint" "" (id 2) (at 100.33 57.15 0)
+    (property "Footprint" "Potentiometer_THT:Potentiometer_Bourns_PTV09A-1_Single_Vertical" (id 2) (at 100.33 57.15 0)
       (effects (font (size 1.27 1.27)) hide)
     )
@@
       (effects (font (size 1.27 1.27)) (justify right))
     )
-    (property "Footprint" "" (id 2) (at 100.33 88.9 0)
+    (property "Footprint" "Potentiometer_THT:Potentiometer_Bourns_PTV09A-1_Single_Vertical" (id 2) (at 100.33 88.9 0)
       (effects (font (size 1.27 1.27)) hide)
     )
@@
       (effects (font (size 1.27 1.27)) (justify right))
     )
-    (property "Footprint" "" (id 2) (at 100.33 120.65 0)
+    (property "Footprint" "Potentiometer_THT:Potentiometer_Bourns_PTV09A-1_Single_Vertical" (id 2) (at 100.33 120.65 0)
       (effects (font (size 1.27 1.27)) hide)
     )
@@
       (effects (font (size 1.27 1.27)) (justify right))
     )
-    (property "Footprint" "" (id 2) (at 101.6 151.13 0)
+    (property "Footprint" "Potentiometer_THT:Potentiometer_Bourns_PTV09A-1_Single_Vertical" (id 2) (at 101.6 151.13 0)
       (effects (font (size 1.27 1.27)) hide)
     )
@@
       (effects (font (size 1.27 1.27)) (justify right))
     )
-    (property "Footprint" "" (id 2) (at 101.6 180.34 0)
+    (property "Footprint" "Potentiometer_THT:Potentiometer_Bourns_PTV09A-1_Single_Vertical" (id 2) (at 101.6 180.34 0)
       (effects (font (size 1.27 1.27)) hide)
     )
@@
       (effects (font (size 1.27 1.27)) (justify right))
     )
-    (property "Footprint" "" (id 2) (at 137.16 25.4 0)
+    (property "Footprint" "Potentiometer_THT:Potentiometer_Bourns_PTV09A-1_Single_Vertical" (id 2) (at 137.16 25.4 0)
       (effects (font (size 1.27 1.27)) hide)
     )
@@
       (effects (font (size 1.27 1.27)) (justify right))
     )
-    (property "Footprint" "" (id 2) (at 137.16 57.15 0)
+    (property "Footprint" "Potentiometer_THT:Potentiometer_Bourns_PTV09A-1_Single_Vertical" (id 2) (at 137.16 57.15 0)
       (effects (font (size 1.27 1.27)) hide)
     )
@@
       (effects (font (size 1.27 1.27)) (justify right))
     )
-    (property "Footprint" "" (id 2) (at 137.16 88.9 0)
+    (property "Footprint" "Potentiometer_THT:Potentiometer_Bourns_PTV09A-1_Single_Vertical" (id 2) (at 137.16 88.9 0)
       (effects (font (size 1.27 1.27)) hide)
     )
@@
       (effects (font (size 1.27 1.27)) (justify right))
     )
-    (property "Footprint" "" (id 2) (at 137.16 120.65 0)
+    (property "Footprint" "Potentiometer_THT:Potentiometer_Bourns_PTV09A-1_Single_Vertical" (id 2) (at 137.16 120.65 0)
       (effects (font (size 1.27 1.27)) hide)
     )
@@
       (effects (font (size 1.27 1.27)) (justify right))
     )
-    (property "Footprint" "" (id 2) (at 138.43 151.13 0)
+    (property "Footprint" "Potentiometer_THT:Potentiometer_Bourns_PTV09A-1_Single_Vertical" (id 2) (at 138.43 151.13 0)
       (effects (font (size 1.27 1.27)) hide)
     )
@@
       (effects (font (size 1.27 1.27)) (justify right))
     )
-    (property "Footprint" "" (id 2) (at 176.53 25.4 0)
+    (property "Footprint" "Potentiometer_THT:Potentiometer_Bourns_PTV09A-1_Single_Vertical" (id 2) (at 176.53 25.4 0)
       (effects (font (size 1.27 1.27)) hide)
     )
@@
       (effects (font (size 1.27 1.27)) (justify right))
     )
-    (property "Footprint" "" (id 2) (at 176.53 57.15 0)
+    (property "Footprint" "Potentiometer_THT:Potentiometer_Bourns_PTV09A-1_Single_Vertical" (id 2) (at 176.53 57.15 0)
       (effects (font (size 1.27 1.27)) hide)
     )
@@
       (effects (font (size 1.27 1.27)) (justify right))
     )
-    (property "Footprint" "" (id 2) (at 176.53 88.9 0)
+    (property "Footprint" "Potentiometer_THT:Potentiometer_Bourns_PTV09A-1_Single_Vertical" (id 2) (at 176.53 88.9 0)
       (effects (font (size 1.27 1.27)) hide)
     )
@@
       (effects (font (size 1.27 1.27)) (justify right))
     )
-    (property "Footprint" "" (id 2) (at 213.36 25.4 0)
+    (property "Footprint" "Potentiometer_THT:Potentiometer_Bourns_PTV09A-1_Single_Vertical" (id 2) (at 213.36 25.4 0)
       (effects (font (size 1.27 1.27)) hide)
     )
@@
       (effects (font (size 1.27 1.27)) (justify right))
     )
-    (property "Footprint" "" (id 2) (at 213.36 57.15 0)
+    (property "Footprint" "Potentiometer_THT:Potentiometer_Bourns_PTV09A-1_Single_Vertical" (id 2) (at 213.36 57.15 0)
       (effects (font (size 1.27 1.27)) hide)
     )
@@
       (effects (font (size 1.27 1.27)) (justify right))
     )
-    (property "Footprint" "" (id 2) (at 213.36 88.9 0)
-      (effects (font (size 1.27 1.27)) hide)
-    )
+    (property "Footprint" "Potentiometer_THT:Potentiometer_Bourns_PTV09A-1_Single_Vertical" (id 2) (at 213.36 88.9 0)
+      (effects (font (size 1.27 1.27)) hide)
+    )

Commit message: mod layout
Parts:
- RV1: value R_POT -> FADERL1; footprint Potentiometer_THT:Potentiometer_Bourns_PTV09A-1_Single_Vertical -> Library:fader-L60
- RV10: renamed from RV20; value R_POT -> PFX1L
- RV11: renamed from RV24; value R_POT -> PFX1R
- RV12: renamed from RV28; value R_POT -> PVOL-HP
- RV13: renamed from RV3; value R_POT -> BASL1
- RV14: renamed from RV9; value R_POT -> BASL2
- RV15: value R_POT -> BASL3
- RV16: renamed from RV21; value R_POT -> PFX2L
- RV17: renamed from RV25; value R_POT -> PFX2R
- RV18: renamed from RV29; value R_POT -> PMASTER
- RV19: renamed from RV4; value R_POT -> MIDL1
- RV2: renamed from RV7; value R_POT -> FADERL2; footprint Potentiometer_THT:Potentiometer_Bourns_PTV09A-1_Single_Vertical -> Library:fader-L60
- RV20: renamed from RV10; value R_POT -> MIDL2
- RV21: renamed from RV16; value R_POT -> MIDL3
- RV22: value R_POT -> PFX3L
- RV23: renamed from RV26; value R_POT -> PFX3R
- RV24: renamed from RV5; value R_POT -> TREL1
- RV25: renamed from RV11; value R_POT -> TREL2
- RV26: renamed from RV17; value R_POT -> TREL3
- RV27: renamed from RV6; value R_POT -> GAINL1
- RV28: renamed from RV12; value R_POT -> GAINL2
- RV29: renamed from RV18; value R_POT -> GAINL3
- RV3: renamed from RV13; value R_POT -> FADERL3; footprint Potentiometer_THT:Potentiometer_Bourns_PTV09A-1_Single_Vertical -> Library:fader-L60
- RV4: renamed from RV19; value R_POT -> PITCH-L; footprint Potentiometer_THT:Potentiometer_Bourns_PTV09A-1_Single_Vertical -> Library:fader-L60
- RV5: renamed from RV23; value R_POT -> PITH-R; footprint Potentiometer_THT:Potentiometer_Bourns_PTV09A-1_Single_Vertical -> Library:fader-L60
- RV6: renamed from RV27; value R_POT -> PMIX-HP
- RV7: renamed from RV2; value R_POT -> FILTERL1
- RV8: value R_POT -> FILTERL2
- RV9: renamed from RV14; value R_POT -> FILTERL3

Commit message: trillbar added
Parts:
- RV4, RV5: footprint Library:fader-L60 -> Library:fader-L75
Changed lines of the file:
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@@
       (effects (font (size 1.27 1.27)) (justify right))
     )
-    (property "Footprint" "Library:fader-L60" (id 2) (at 27.94 120.65 0)
+    (property "Footprint" "Library:fader-L75" (id 2) (at 27.94 120.65 0)
       (effects (font (size 1.27 1.27)) hide)
     )
@@
       (effects (font (size 1.27 1.27)) (justify right))
     )
-    (property "Footprint" "Library:fader-L60" (id 2) (at 29.21 151.13 0)
+    (property "Footprint" "Library:fader-L75" (id 2) (at 29.21 151.13 0)
       (effects (font (size 1.27 1.27)) hide)
     )

Commit message: fixing 3dmodels
Parts:
- RV10, RV11, RV12, RV13, RV14, RV15, RV16, RV17, RV18, RV19, RV20, RV21, RV22, RV23, RV24, RV25, RV26, RV27, RV28, RV29, RV6, RV7, RV8, RV9: footprint Potentiometer_THT:Potentiometer_Bourns_PTV09A-1_Single_Vertical -> Library:Potentiometer_Bourns_PTV09A-1_Single_Vertical
Changed lines of the file:
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@@
       (effects (font (size 1.27 1.27)) (justify right))
     )
-    (property "Footprint" "Potentiometer_THT:Potentiometer_Bourns_PTV09A-1_Single_Vertical" (id 2) (at 29.21 180.34 0)
+    (property "Footprint" "Library:Potentiometer_Bourns_PTV09A-1_Single_Vertical" (id 2) (at 29.21 180.34 0)
       (effects (font (size 1.27 1.27)) hide)
     )
@@
       (effects (font (size 1.27 1.27)) (justify right))
     )
-    (property "Footprint" "Potentiometer_THT:Potentiometer_Bourns_PTV09A-1_Single_Vertical" (id 2) (at 63.5 25.4 0)
+    (property "Footprint" "Library:Potentiometer_Bourns_PTV09A-1_Single_Vertical" (id 2) (at 63.5 25.4 0)
       (effects (font (size 1.27 1.27)) hide)
     )
@@
       (effects (font (size 1.27 1.27)) (justify right))
     )
-    (property "Footprint" "Potentiometer_THT:Potentiometer_Bourns_PTV09A-1_Single_Vertical" (id 2) (at 63.5 57.15 0)
+    (property "Footprint" "Library:Potentiometer_Bourns_PTV09A-1_Single_Vertical" (id 2) (at 63.5 57.15 0)
       (effects (font (size 1.27 1.27)) hide)
     )
@@
       (effects (font (size 1.27 1.27)) (justify right))
     )
-    (property "Footprint" "Potentiometer_THT:Potentiometer_Bourns_PTV09A-1_Single_Vertical" (id 2) (at 63.5 88.9 0)
+    (property "Footprint" "Library:Potentiometer_Bourns_PTV09A-1_Single_Vertical" (id 2) (at 63.5 88.9 0)
       (effects (font (size 1.27 1.27)) hide)
     )
@@
       (effects (font (size 1.27 1.27)) (justify right))
     )
-    (property "Footprint" "Potentiometer_THT:Potentiometer_Bourns_PTV09A-1_Single_Vertical" (id 2) (at 63.5 120.65 0)
+    (property "Footprint" "Library:Potentiometer_Bourns_PTV09A-1_Single_Vertical" (id 2) (at 63.5 120.65 0)
       (effects (font (size 1.27 1.27)) hide)
     )
@@
       (effects (font (size 1.27 1.27)) (justify right))
     )
-    (property "Footprint" "Potentiometer_THT:Potentiometer_Bourns_PTV09A-1_Single_Vertical" (id 2) (at 64.77 151.13 0)
+    (property "Footprint" "Library:Potentiometer_Bourns_PTV09A-1_Single_Vertical" (id 2) (at 64.77 151.13 0)
       (effects (font (size 1.27 1.27)) hide)
     )
@@
       (effects (font (size 1.27 1.27)) (justify right))
     )
-    (property "Footprint" "Potentiometer_THT:Potentiometer_Bourns_PTV09A-1_Single_Vertical" (id 2) (at 64.77 180.34 0)
+    (property "Footprint" "Library:Potentiometer_Bourns_PTV09A-1_Single_Vertical" (id 2) (at 64.77 180.34 0)
       (effects (font (size 1.27 1.27)) hide)
     )
@@
       (effects (font (size 1.27 1.27)) (justify right))
     )
-    (property "Footprint" "Potentiometer_THT:Potentiometer_Bourns_PTV09A-1_Single_Vertical" (id 2) (at 100.33 25.4 0)
+    (property "Footprint" "Library:Potentiometer_Bourns_PTV09A-1_Single_Vertical" (id 2) (at 100.33 25.4 0)
       (effects (font (size 1.27 1.27)) hide)
     )
@@
       (effects (font (size 1.27 1.27)) (justify right))
     )
-    (property "Footprint" "Potentiometer_THT:Potentiometer_Bourns_PTV09A-1_Single_Vertical" (id 2) (at 100.33 57.15 0)
+    (property "Footprint" "Library:Potentiometer_Bourns_PTV09A-1_Single_Vertical" (id 2) (at 100.33 57.15 0)
       (effects (font (size 1.27 1.27)) hide)
     )
@@
       (effects (font (size 1.27 1.27)) (justify right))
     )
-    (property "Footprint" "Potentiometer_THT:Potentiometer_Bourns_PTV09A-1_Single_Vertical" (id 2) (at 100.33 88.9 0)
+    (property "Footprint" "Library:Potentiometer_Bourns_PTV09A-1_Single_Vertical" (id 2) (at 100.33 88.9 0)
       (effects (font (size 1.27 1.27)) hide)
     )
@@
       (effects (font (size 1.27 1.27)) (justify right))
     )
-    (property "Footprint" "Potentiometer_THT:Potentiometer_Bourns_PTV09A-1_Single_Vertical" (id 2) (at 100.33 120.65 0)
+    (property "Footprint" "Library:Potentiometer_Bourns_PTV09A-1_Single_Vertical" (id 2) (at 100.33 120.65 0)
       (effects (font (size 1.27 1.27)) hide)
     )
@@
       (effects (font (size 1.27 1.27)) (justify right))
     )
-    (property "Footprint" "Potentiometer_THT:Potentiometer_Bourns_PTV09A-1_Single_Vertical" (id 2) (at 101.6 151.13 0)
+    (property "Footprint" "Library:Potentiometer_Bourns_PTV09A-1_Single_Vertical" (id 2) (at 101.6 151.13 0)
       (effects (font (size 1.27 1.27)) hide)
     )
@@
       (effects (font (size 1.27 1.27)) (justify right))
     )
-    (property "Footprint" "Potentiometer_THT:Potentiometer_Bourns_PTV09A-1_Single_Vertical" (id 2) (at 101.6 180.34 0)
+    (property "Footprint" "Library:Potentiometer_Bourns_PTV09A-1_Single_Vertical" (id 2) (at 101.6 180.34 0)
       (effects (font (size 1.27 1.27)) hide)
     )
@@
       (effects (font (size 1.27 1.27)) (justify right))
     )
-    (property "Footprint" "Potentiometer_THT:Potentiometer_Bourns_PTV09A-1_Single_Vertical" (id 2) (at 137.16 25.4 0)
+    (property "Footprint" "Library:Potentiometer_Bourns_PTV09A-1_Single_Vertical" (id 2) (at 137.16 25.4 0)
       (effects (font (size 1.27 1.27)) hide)
     )
@@
       (effects (font (size 1.27 1.27)) (justify right))
     )
-    (property "Footprint" "Potentiometer_THT:Potentiometer_Bourns_PTV09A-1_Single_Vertical" (id 2) (at 137.16 57.15 0)
+    (property "Footprint" "Library:Potentiometer_Bourns_PTV09A-1_Single_Vertical" (id 2) (at 137.16 57.15 0)
       (effects (font (size 1.27 1.27)) hide)
     )
@@
       (effects (font (size 1.27 1.27)) (justify right))
     )
-    (property "Footprint" "Potentiometer_THT:Potentiometer_Bourns_PTV09A-1_Single_Vertical" (id 2) (at 137.16 88.9 0)
+    (property "Footprint" "Library:Potentiometer_Bourns_PTV09A-1_Single_Vertical" (id 2) (at 137.16 88.9 0)
       (effects (font (size 1.27 1.27)) hide)
     )
@@
       (effects (font (size 1.27 1.27)) (justify right))
     )
-    (property "Footprint" "Potentiometer_THT:Potentiometer_Bourns_PTV09A-1_Single_Vertical" (id 2) (at 137.16 120.65 0)
+    (property "Footprint" "Library:Potentiometer_Bourns_PTV09A-1_Single_Vertical" (id 2) (at 137.16 120.65 0)
       (effects (font (size 1.27 1.27)) hide)
     )
@@
       (effects (font (size 1.27 1.27)) (justify right))
     )
-    (property "Footprint" "Potentiometer_THT:Potentiometer_Bourns_PTV09A-1_Single_Vertical" (id 2) (at 138.43 151.13 0)
+    (property "Footprint" "Library:Potentiometer_Bourns_PTV09A-1_Single_Vertical" (id 2) (at 138.43 151.13 0)
       (effects (font (size 1.27 1.27)) hide)
     )
@@
       (effects (font (size 1.27 1.27)) (justify right))
     )
-    (property "Footprint" "Potentiometer_THT:Potentiometer_Bourns_PTV09A-1_Single_Vertical" (id 2) (at 176.53 25.4 0)
+    (property "Footprint" "Library:Potentiometer_Bourns_PTV09A-1_Single_Vertical" (id 2) (at 176.53 25.4 0)
       (effects (font (size 1.27 1.27)) hide)
     )
@@
       (effects (font (size 1.27 1.27)) (justify right))
     )
-    (property "Footprint" "Potentiometer_THT:Potentiometer_Bourns_PTV09A-1_Single_Vertical" (id 2) (at 176.53 57.15 0)
+    (property "Footprint" "Library:Potentiometer_Bourns_PTV09A-1_Single_Vertical" (id 2) (at 176.53 57.15 0)
       (effects (font (size 1.27 1.27)) hide)
     )
@@
       (effects (font (size 1.27 1.27)) (justify right))
     )
-    (property "Footprint" "Potentiometer_THT:Potentiometer_Bourns_PTV09A-1_Single_Vertical" (id 2) (at 176.53 88.9 0)
+    (property "Footprint" "Library:Potentiometer_Bourns_PTV09A-1_Single_Vertical" (id 2) (at 176.53 88.9 0)
       (effects (font (size 1.27 1.27)) hide)
     )
@@
       (effects (font (size 1.27 1.27)) (justify right))
     )
-    (property "Footprint" "Potentiometer_THT:Potentiometer_Bourns_PTV09A-1_Single_Vertical" (id 2) (at 213.36 25.4 0)
+    (property "Footprint" "Library:Potentiometer_Bourns_PTV09A-1_Single_Vertical" (id 2) (at 213.36 25.4 0)
       (effects (font (size 1.27 1.27)) hide)
     )
@@
       (effects (font (size 1.27 1.27)) (justify right))
     )
-    (property "Footprint" "Potentiometer_THT:Potentiometer_Bourns_PTV09A-1_Single_Vertical" (id 2) (at 213.36 57.15 0)
+    (property "Footprint" "Library:Potentiometer_Bourns_PTV09A-1_Single_Vertical" (id 2) (at 213.36 57.15 0)
       (effects (font (size 1.27 1.27)) hide)
     )
@@
       (effects (font (size 1.27 1.27)) (justify right))
     )
-    (property "Footprint" "Potentiometer_THT:Potentiometer_Bourns_PTV09A-1_Single_Vertical" (id 2) (at 213.36 88.9 0)
-      (effects (font (size 1.27 1.27)) hide)
-    )
+    (property "Footprint" "Library:Potentiometer_Bourns_PTV09A-1_Single_Vertical" (id 2) (at 213.36 88.9 0)
+      (effects (font (size 1.27 1.27)) hide)
+    )

Commit message: routing
Parts:
- renumbered RV20 to RV10, RV25 to RV11, RV28 to RV12, RV3 to RV13, RV9 to RV14, RV21 to RV16, RV26 to RV17, RV29 to RV18, RV4 to RV19, RV7 to RV2, RV10 to RV20, RV16 to RV21, RV5 to RV23, RV11 to RV24, RV17 to RV25, RV23 to RV26, RV6 to RV27, RV12 to RV28, RV18 to RV29, RV13 to RV3, RV19 to RV4, RV24 to RV5, RV27 to RV6, RV2 to RV7, RV14 to RV9
