File: PCB/Kicad/potenciometers.kicad_sch (KiCad schematic)
At the start: 29 parts

Commit message: SCHEMATIC FINISHED
Parts:
- removed RV1: FADERL1, Library:fader-L60, symbol Device:R_Potentiometer
- removed RV10: MIDL2, Library:Potentiometer_Bourns_PTV09A-1_Single_Vertical, symbol Device:R_Potentiometer
- removed RV12: GAINL2, Library:Potentiometer_Bourns_PTV09A-1_Single_Vertical, symbol Device:R_Potentiometer
- removed RV13: FADERL3, Library:fader-L60, symbol Device:R_Potentiometer
- removed RV14: FILTERL3, Library:Potentiometer_Bourns_PTV09A-1_Single_Vertical, symbol Device:R_Potentiometer
- removed RV15: BASL3, Library:Potentiometer_Bourns_PTV09A-1_Single_Vertical, symbol Device:R_Potentiometer
- removed RV16: MIDL3, Library:Potentiometer_Bourns_PTV09A-1_Single_Vertical, symbol Device:R_Potentiometer
- removed RV18: GAINL3, Library:Potentiometer_Bourns_PTV09A-1_Single_Vertical, symbol Device:R_Potentiometer
- removed RV19: PITCH-L, Library:fader-L75, symbol Device:R_Potentiometer
- removed RV2: FILTERL1, Library:Potentiometer_Bourns_PTV09A-1_Single_Vertical, symbol Device:R_Potentiometer
- removed RV20: PFX1L, Library:Potentiometer_Bourns_PTV09A-1_Single_Vertical, symbol Device:R_Potentiometer
- removed RV21: PFX2L, Library:Potentiometer_Bourns_PTV09A-1_Single_Vertical, symbol Device:R_Potentiometer
- removed RV22: PFX3L, Library:Potentiometer_Bourns_PTV09A-1_Single_Vertical, symbol Device:R_Potentiometer
- removed RV23: PITH-R, Library:fader-L75, symbol Device:R_Potentiometer
- removed RV24: PFX1R, Library:Potentiometer_Bourns_PTV09A-1_Single_Vertical, symbol Device:R_Potentiometer
- removed RV26: PFX3R, Library:Potentiometer_Bourns_PTV09A-1_Single_Vertical, symbol Device:R_Potentiometer
- removed RV27: PMIX-HP, Library:Potentiometer_Bourns_PTV09A-1_Single_Vertical, symbol Device:R_Potentiometer
- removed RV28: PVOL-HP, Library:Potentiometer_Bourns_PTV09A-1_Single_Vertical, symbol Device:R_Potentiometer
- removed RV29: PMASTER, Library:Potentiometer_Bourns_PTV09A-1_Single_Vertical, symbol Device:R_Potentiometer
- removed RV3: BASL1, Library:Potentiometer_Bourns_PTV09A-1_Single_Vertical, symbol Device:R_Potentiometer
- removed RV4: MIDL1, Library:Potentiometer_Bourns_PTV09A-1_Single_Vertical, symbol Device:R_Potentiometer
- removed RV6: GAINL1, Library:Potentiometer_Bourns_PTV09A-1_Single_Vertical, symbol Device:R_Potentiometer
- removed RV7: FADERL2, Library:fader-L60, symbol Device:R_Potentiometer
- removed RV8: FILTERL2, Library:Potentiometer_Bourns_PTV09A-1_Single_Vertical, symbol Device:R_Potentiometer
- removed RV9: BASL2, Library:Potentiometer_Bourns_PTV09A-1_Single_Vertical, symbol Device:R_Potentiometer
- added IC-MPLEX-?: MP-TOP-POTS, Library:SOIC-24W_7.5x15.4mm_P1.27mm, symbol mixduino-mk2:74HC4067D,653
- added RV?: PGAINL3, Library:Potentiometer_Bourns_PTV09A-1_Single_Vertical, symbol Device:R_Potentiometer
- added RV?: PFX2L, Library:Potentiometer_Bourns_PTV09A-1_Single_Vertical, symbol Device:R_Potentiometer
- added RV?: PGAINL1, Library:Potentiometer_Bourns_PTV09A-1_Single_Vertical, symbol Device:R_Potentiometer
- added RV?: PFX3R, Library:Potentiometer_Bourns_PTV09A-1_Single_Vertical, symbol Device:R_Potentiometer
- added RV?: PFX1L, Library:Potentiometer_Bourns_PTV09A-1_Single_Vertical, symbol Device:R_Potentiometer
- added RV?: PGAINL2, Library:Potentiometer_Bourns_PTV09A-1_Single_Vertical, symbol Device:R_Potentiometer
- added RV?: PFX3L, Library:Potentiometer_Bourns_PTV09A-1_Single_Vertical, symbol Device:R_Potentiometer
- renumbered RV25 to RV17, RV5 to RV24, RV11 to RV25, RV17 to RV26
Connections:
- net +5V: now also IC-MPLEX-?.24 (VCC), RV?.1, RV?.1, RV?.1, RV?.1, RV?.1, RV?.1, RV?.1
- net GND: now also IC-MPLEX-?.12 (GND), IC-MPLEX-?.15 (~E), RV?.3, RV?.3, RV?.3, RV?.3, RV?.3, RV?.3, RV?.3
- net PFX-2R: no longer names the net of RV17.2
- net PFX-2R: now also IC-MPLEX-?.2 (Y7)
- net TRE-L1: no longer names the net of RV24.2
- net TRE-L1: now also IC-MPLEX-?.23 (Y8)
- net TRE-L2: no longer names the net of RV25.2
- net TRE-L2: now also IC-MPLEX-?.22 (Y9)
- net TRE-L3: no longer names the net of RV26.2
- net TRE-L3: now also IC-MPLEX-?.21 (Y10)
- new net: IC-MPLEX-?.4 (Y5), RV?.2
- new net: IC-MPLEX-?.3 (Y6), RV?.2
- new net: IC-MPLEX-?.5 (Y4), RV?.2
- new net: IC-MPLEX-?.6 (Y3), RV?.2
- new net: IC-MPLEX-?.7 (Y2), RV?.2
- new net: IC-MPLEX-?.8 (Y1), RV?.2
- new net: IC-MPLEX-?.9 (Y0), RV?.2
- new net MPLEX-A1: IC-MPLEX-?.1 (Z)
- new net MPLEX-S0: IC-MPLEX-?.10 (S0)
- new net MPLEX-S1: IC-MPLEX-?.11 (S1)
- new net MPLEX-S2: IC-MPLEX-?.14 (S2)
- new net MPLEX-S3: IC-MPLEX-?.13 (S3)
- no-connect marks 0 -> 5
Other:
- moved on the sheet: RV17, RV24, RV25, RV26
