File: PCB/Kicad/MPX-SW-BTNS.kicad_sch (KiCad schematic)
At the start: 34 parts, among them SW13 SWCUEL, SW14 SWPLAYL, SW15 SWRANGEL, SW16 SWSYNCL, SW17 SWLOOPL, SW18 SWSHIFTL, SW19 SWSHIFTR, SW20 SWPCUEL1, SW21 SWPCUEL2, SW22 SWCUER, SW23 SWPLAYR, SW24 SWRANGER, SW25 SWLOOPR, SW26 SWPCUEL3, SW27 SWSYNCR, SW28 SWDECKSEL, SW29 SWPADL5, SW30 SWPADL1, SW31 SWPADL6, SW32 SWPADL2, SW33 SWPADL7, SW34 SWPADL3, SW35 SWPADL4, SW36 SWPADL8, SW37 SWPADR5, SW38 SWPADR1, SW39 SWPADR6, SW40 SWPADR2, SW41 SWPADR7, SW42 SWPADR3, SW43 SWPADR4, SW44 SWPADR8

Commit message: PDF
Other:
- note added: "MULTIPLEXER SWITCH BUTTONS"
- moved on the sheet: IC-MPLEX-2, IC-MPLEX-3, SW13, SW14, SW15, SW16, SW17, SW18, SW19, SW20, SW21, SW22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

Commit message: routing WIP
Parts:
- SW13, SW14, SW15, SW16, SW17, SW18, SW19, SW20, SW21, SW22, SW23, SW24, SW25, SW26, SW27, SW28: footprint Library:SW_PUSH_6mm_H8mm -> Library:SW_Push_1P1T_NO_6x6mm_H8mm
Connections:
- net at SW41.1: now also IC-MPLEX-2.20 (Y11); no longer IC-MPLEX-2.19 (Y12)
- net at SW27.2: now also IC-MPLEX-2.3 (Y6); no longer IC-MPLEX-2.8 (Y1)
- net at IC-MPLEX-3.16 (Y15): now also SW29.1; no longer SW36.1
- net at IC-MPLEX-3.17 (Y14): now also SW30.1; no longer SW35.1
- net at IC-MPLEX-3.18 (Y13): now also SW31.1; no longer SW34.1
- net at IC-MPLEX-3.19 (Y12): now also SW32.1; no longer SW33.1
- net at IC-MPLEX-3.20 (Y11): now also SW33.1; no longer SW32.1
- net at IC-MPLEX-3.21 (Y10): now also SW34.1; no longer SW31.1
- net at IC-MPLEX-3.22 (Y9): now also SW35.1; no longer SW30.1
- net at IC-MPLEX-3.23 (Y8): now also SW36.1; no longer SW29.1
- net at SW40.1: now also IC-MPLEX-2.19 (Y12); no longer IC-MPLEX-2.20 (Y11)
- net at SW44.1: now also IC-MPLEX-2.23 (Y8); no longer IC-MPLEX-2.16 (Y15)
- net at SW38.1: now also IC-MPLEX-2.17 (Y14); no longer IC-MPLEX-2.22 (Y9)
- net at SW26.2: now also IC-MPLEX-2.4 (Y5); no longer IC-MPLEX-2.7 (Y2)
- net at SW42.1: now also IC-MPLEX-2.21 (Y10); no longer IC-MPLEX-2.18 (Y13)
- net at SW43.1: now also IC-MPLEX-2.22 (Y9); no longer IC-MPLEX-2.17 (Y14)
- net at IC-MPLEX-2.2 (Y7): now also SW28.2; no longer SW22.2
- net at SW39.1: now also IC-MPLEX-2.18 (Y13); no longer IC-MPLEX-2.21 (Y10)
- net at SW37.1: now also IC-MPLEX-2.16 (Y15); no longer IC-MPLEX-2.23 (Y8)
- net at SW23.2: now also IC-MPLEX-2.8 (Y1); no longer IC-MPLEX-2.3 (Y6)
- net at SW24.2: now also IC-MPLEX-2.7 (Y2); no longer IC-MPLEX-2.4 (Y5)
- net at IC-MPLEX-2.9 (Y0): now also SW22.2; no longer SW28.2
Other:
- moved on the sheet: SW22, SW23, SW24, SW26, SW27, SW28, SW29, SW30, SW31, SW32, SW33, SW34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

Commit message: routes done
Connections:
- net at IC-MPLEX-3.20 (Y11): now also SW34.1; no longer SW33.1
- net at IC-MPLEX-3.21 (Y10): now also SW33.1; no longer SW34.1
Other:
- moved on the sheet: SW33, SW34
Changed lines of the file:
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@@
   (symbol (lib_id "mixduino-mk2:SW_Push") (at 169.545 55.245 0) (unit 1)
     (in_bom yes) (on_board yes)
-    (property "Reference" "SW34" (id 0) (at 164.465 52.705 0)
+    (property "Reference" "SW33" (id 0) (at 164.465 52.705 0)
       (effects (font (size 1.27 1.27)) (justify left))
     )
-    (property "Value" "SWPADL3" (id 1) (at 174.625 52.705 0))
+    (property "Value" "SWPADL7" (id 1) (at 174.625 52.705 0))
     (property "Footprint" "Library:sw-pad" (id 2) (at 169.545 50.165 0)
       (effects (font (size 1.27 1.27)) hide)
@@
   (symbol (lib_id "mixduino-mk2:SW_Push") (at 169.545 60.325 0) (unit 1)
     (in_bom yes) (on_board yes)
-    (property "Reference" "SW33" (id 0) (at 164.465 57.785 0)
+    (property "Reference" "SW34" (id 0) (at 164.465 57.785 0)
       (effects (font (size 1.27 1.27)) (justify left))
     )
-    (property "Value" "SWPADL7" (id 1) (at 174.625 57.785 0))
+    (property "Value" "SWPADL3" (id 1) (at 174.625 57.785 0))
     (property "Footprint" "Library:sw-pad" (id 2) (at 169.545 55.245 0)
       (effects (font (size 1.27 1.27)) hide)

Commit message: routing WIP
Connections:
- net at SW41.1: now also IC-MPLEX-2.21 (Y10); no longer IC-MPLEX-2.20 (Y11)
- net at SW42.1: now also IC-MPLEX-2.20 (Y11); no longer IC-MPLEX-2.21 (Y10)
Other:
- moved on the sheet: SW41, SW42
Changed lines of the file:
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@@
   (symbol (lib_id "mixduino-mk2:SW_Push") (at 169.545 125.095 0) (unit 1)
     (in_bom yes) (on_board yes)
-    (property "Reference" "SW42" (id 0) (at 164.465 122.555 0)
+    (property "Reference" "SW41" (id 0) (at 164.465 122.555 0)
       (effects (font (size 1.27 1.27)) (justify left))
     )
-    (property "Value" "SWPADR3" (id 1) (at 174.625 122.555 0))
+    (property "Value" "SWPADR7" (id 1) (at 174.625 122.555 0))
     (property "Footprint" "Library:sw-pad" (id 2) (at 169.545 120.015 0)
       (effects (font (size 1.27 1.27)) hide)
@@
   (symbol (lib_id "mixduino-mk2:SW_Push") (at 169.545 130.175 0) (unit 1)
     (in_bom yes) (on_board yes)
-    (property "Reference" "SW41" (id 0) (at 164.465 127.635 0)
+    (property "Reference" "SW42" (id 0) (at 164.465 127.635 0)
       (effects (font (size 1.27 1.27)) (justify left))
     )
-    (property "Value" "SWPADR7" (id 1) (at 174.625 127.635 0))
+    (property "Value" "SWPADR3" (id 1) (at 174.625 127.635 0))
     (property "Footprint" "Library:sw-pad" (id 2) (at 169.545 125.095 0)
       (effects (font (size 1.27 1.27)) hide)

Commit message: update schematic
Parts:
- IC-MPLEX-2, IC-MPLEX-3: footprint Library:SOIC-24W_7.5x15.4mm_P1.27mm -> Package_SO:SOIC-24W_7.5x15.4mm_P1.27mm
Changed lines of the file:
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@@
     (property "Reference" "IC-MPLEX-2" (id 0) (at 129.54 114.3 0))
     (property "Value" "MP-RIGHT-BTNS" (id 1) (at 129.54 116.84 0))
-    (property "Footprint" "Library:SOIC-24W_7.5x15.4mm_P1.27mm" (id 2) (at 138.43 118.11 0)
+    (property "Footprint" "Package_SO:SOIC-24W_7.5x15.4mm_P1.27mm" (id 2) (at 138.43 118.11 0)
       (effects (font (size 1.27 1.27)) (justify left) hide)
     )
@@
     (property "Reference" "IC-MPLEX-3" (id 0) (at 132.08 44.45 0))
     (property "Value" "MP-LEFT-BTNS" (id 1) (at 132.08 46.99 0))
-    (property "Footprint" "Library:SOIC-24W_7.5x15.4mm_P1.27mm" (id 2) (at 140.97 48.26 0)
+    (property "Footprint" "Package_SO:SOIC-24W_7.5x15.4mm_P1.27mm" (id 2) (at 140.97 48.26 0)
       (effects (font (size 1.27 1.27)) (justify left) hide)
     )
