File: PCB/Kicad/TOP-POTS.kicad_sch (KiCad schematic)
At the start: 12 parts

Commit message: PDF
Other:
- note added: "TOP POTS"
- moved on the sheet: IC-MPLEX-1, RV10, RV11, RV12, RV13, RV3, RV4, RV5, RV6, RV7, RV8, RV9

Commit message: routing WIP
Connections:
- net at RV9.2: now also IC-MPLEX-1.3 (Y6); no longer IC-MPLEX-1.2 (Y7)
- net at RV5.2: now also IC-MPLEX-1.2 (Y7); no longer IC-MPLEX-1.3 (Y6)
Other:
- moved on the sheet: RV5, RV9
Changed lines of the file:
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@@
   (symbol (lib_id "Device:R_Potentiometer") (at 69.85 66.04 0) (unit 1)
     (in_bom yes) (on_board yes)
-    (property "Reference" "RV5" (id 0) (at 68.0974 64.8716 0)
+    (property "Reference" "RV9" (id 0) (at 68.0974 64.8716 0)
       (effects (font (size 1.27 1.27)) (justify right))
     )
-    (property "Value" "PFX3R" (id 1) (at 68.0974 67.183 0)
+    (property "Value" "PFX2R" (id 1) (at 68.0974 67.183 0)
       (effects (font (size 1.27 1.27)) (justify right))
     )
@@
   (symbol (lib_id "Device:R_Potentiometer") (at 93.345 66.04 0) (unit 1)
     (in_bom yes) (on_board yes)
-    (property "Reference" "RV9" (id 0) (at 91.5924 64.8716 0)
+    (property "Reference" "RV5" (id 0) (at 91.5924 64.8716 0)
       (effects (font (size 1.27 1.27)) (justify right))
     )
-    (property "Value" "PFX2R" (id 1) (at 91.5924 67.183 0)
+    (property "Value" "PFX3R" (id 1) (at 91.5924 67.183 0)
       (effects (font (size 1.27 1.27)) (justify right))
     )

Commit message: update schematic
Parts:
- IC-MPLEX-1: footprint Library:SOIC-24W_7.5x15.4mm_P1.27mm -> Package_SO:SOIC-24W_7.5x15.4mm_P1.27mm
Changed lines of the file:
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@@
     (property "Reference" "IC-MPLEX-1" (id 0) (at 148.59 80.645 0))
     (property "Value" "MP-TOP-POTS" (id 1) (at 148.59 83.185 0))
-    (property "Footprint" "Library:SOIC-24W_7.5x15.4mm_P1.27mm" (id 2) (at 157.48 84.455 0)
+    (property "Footprint" "Package_SO:SOIC-24W_7.5x15.4mm_P1.27mm" (id 2) (at 157.48 84.455 0)
       (effects (font (size 1.27 1.27)) (justify left) hide)
     )
