File: PCB/Kicad/fb-leds.kicad_sch (KiCad schematic)
At the start: 52 parts, among them Q1 MMBTA05L, Q2 MMBTA05L, Q3 MMBTA05L, Q4 MMBTA05L

Commit message: update schematic
Parts:
- R1, R10, R11, R12, R13, R14, R15, R16, R17, R18, R19, R2, R20, R21, R22, R23, R3, R4, R5, R6, R7, R8, R9: footprint Library:R_1206_3216Metric_Pad1.30x1.75mm_HandSolder -> Resistor_SMD:R_1206_3216Metric_Pad1.30x1.75mm_HandSolder
Changed lines of the file:
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@@
     (property "Reference" "R1" (id 0) (at 124.46 50.8 90))
     (property "Value" "R-PCUEL3" (id 1) (at 124.46 55.88 90))
-    (property "Footprint" "Library:R_1206_3216Metric_Pad1.30x1.75mm_HandSolder" (id 2) (at 124.46 53.34 0)
+    (property "Footprint" "Resistor_SMD:R_1206_3216Metric_Pad1.30x1.75mm_HandSolder" (id 2) (at 124.46 53.34 0)
       (effects (font (size 1.27 1.27)) hide)
     )
@@
     (property "Reference" "R2" (id 0) (at 124.46 71.755 90))
     (property "Value" "R-LOOP-R" (id 1) (at 124.46 76.835 90))
-    (property "Footprint" "Library:R_1206_3216Metric_Pad1.30x1.75mm_HandSolder" (id 2) (at 124.46 74.295 0)
+    (property "Footprint" "Resistor_SMD:R_1206_3216Metric_Pad1.30x1.75mm_HandSolder" (id 2) (at 124.46 74.295 0)
       (effects (font (size 1.27 1.27)) hide)
     )
@@
     (property "Reference" "R3" (id 0) (at 124.46 78.74 90))
     (property "Value" "R-FX3-R" (id 1) (at 124.46 83.82 90))
-    (property "Footprint" "Library:R_1206_3216Metric_Pad1.30x1.75mm_HandSolder" (id 2) (at 124.46 81.28 0)
+    (property "Footprint" "Resistor_SMD:R_1206_3216Metric_Pad1.30x1.75mm_HandSolder" (id 2) (at 124.46 81.28 0)
       (effects (font (size 1.27 1.27)) hide)
     )
@@
     (property "Reference" "R4" (id 0) (at 124.46 85.725 90))
     (property "Value" "R-FX2-R" (id 1) (at 124.46 90.805 90))
-    (property "Footprint" "Library:R_1206_3216Metric_Pad1.30x1.75mm_HandSolder" (id 2) (at 124.46 88.265 0)
+    (property "Footprint" "Resistor_SMD:R_1206_3216Metric_Pad1.30x1.75mm_HandSolder" (id 2) (at 124.46 88.265 0)
       (effects (font (size 1.27 1.27)) hide)
     )
@@
     (property "Reference" "R5" (id 0) (at 124.46 92.71 90))
     (property "Value" "R-FX1-R" (id 1) (at 124.46 97.79 90))
-    (property "Footprint" "Library:R_1206_3216Metric_Pad1.30x1.75mm_HandSolder" (id 2) (at 124.46 95.25 0)
+    (property "Footprint" "Resistor_SMD:R_1206_3216Metric_Pad1.30x1.75mm_HandSolder" (id 2) (at 124.46 95.25 0)
       (effects (font (size 1.27 1.27)) hide)
     )
@@
     (property "Reference" "R6" (id 0) (at 124.46 117.475 90))
     (property "Value" "R-FX3-L" (id 1) (at 124.46 122.555 90))
-    (property "Footprint" "Library:R_1206_3216Metric_Pad1.30x1.75mm_HandSolder" (id 2) (at 124.46 120.015 0)
+    (property "Footprint" "Resistor_SMD:R_1206_3216Metric_Pad1.30x1.75mm_HandSolder" (id 2) (at 124.46 120.015 0)
       (effects (font (size 1.27 1.27)) hide)
     )
@@
     (property "Reference" "R7" (id 0) (at 124.46 124.46 90))
     (property "Value" "R-FX2-L" (id 1) (at 124.46 129.54 90))
-    (property "Footprint" "Library:R_1206_3216Metric_Pad1.30x1.75mm_HandSolder" (id 2) (at 124.46 127 0)
+    (property "Footprint" "Resistor_SMD:R_1206_3216Metric_Pad1.30x1.75mm_HandSolder" (id 2) (at 124.46 127 0)
       (effects (font (size 1.27 1.27)) hide)
     )
@@
     (property "Reference" "R8" (id 0) (at 124.46 131.445 90))
     (property "Value" "R-FX1-L" (id 1) (at 124.46 136.525 90))
-    (property "Footprint" "Library:R_1206_3216Metric_Pad1.30x1.75mm_HandSolder" (id 2) (at 124.46 133.985 0)
+    (property "Footprint" "Resistor_SMD:R_1206_3216Metric_Pad1.30x1.75mm_HandSolder" (id 2) (at 124.46 133.985 0)
       (effects (font (size 1.27 1.27)) hide)
     )
@@
     (property "Reference" "R9" (id 0) (at 124.46 152.4 90))
     (property "Value" "R-LOOP-L" (id 1) (at 124.46 157.48 90))
-    (property "Footprint" "Library:R_1206_3216Metric_Pad1.30x1.75mm_HandSolder" (id 2) (at 124.46 154.94 0)
+    (property "Footprint" "Resistor_SMD:R_1206_3216Metric_Pad1.30x1.75mm_HandSolder" (id 2) (at 124.46 154.94 0)
       (effects (font (size 1.27 1.27)) hide)
     )
@@
     (property "Reference" "R11" (id 0) (at 124.46 164.465 90))
     (property "Value" "R-PCUE2" (id 1) (at 124.46 159.385 90))
-    (property "Footprint" "Library:R_1206_3216Metric_Pad1.30x1.75mm_HandSolder" (id 2) (at 124.46 161.925 0)
+    (property "Footprint" "Resistor_SMD:R_1206_3216Metric_Pad1.30x1.75mm_HandSolder" (id 2) (at 124.46 161.925 0)
       (effects (font (size 1.27 1.27)) hide)
     )
@@
     (property "Reference" "R10" (id 0) (at 124.46 171.45 90))
     (property "Value" "R-PCUE1" (id 1) (at 124.46 166.37 90))
-    (property "Footprint" "Library:R_1206_3216Metric_Pad1.30x1.75mm_HandSolder" (id 2) (at 124.46 168.91 0)
+    (property "Footprint" "Resistor_SMD:R_1206_3216Metric_Pad1.30x1.75mm_HandSolder" (id 2) (at 124.46 168.91 0)
       (effects (font (size 1.27 1.27)) hide)
     )
@@
       (effects (font (size 1.27 1.27)) (justify left))
     )
-    (property "Footprint" "Library:R_1206_3216Metric_Pad1.30x1.75mm_HandSolder" (id 2) (at 163.83 57.785 0)
+    (property "Footprint" "Resistor_SMD:R_1206_3216Metric_Pad1.30x1.75mm_HandSolder" (id 2) (at 163.83 57.785 0)
       (effects (font (size 1.27 1.27)) hide)
     )
@@
       (effects (font (size 1.27 1.27)) (justify left))
     )
-    (property "Footprint" "Library:R_1206_3216Metric_Pad1.30x1.75mm_HandSolder" (id 2) (at 163.83 145.415 0)
+    (property "Footprint" "Resistor_SMD:R_1206_3216Metric_Pad1.30x1.75mm_HandSolder" (id 2) (at 163.83 145.415 0)
       (effects (font (size 1.27 1.27)) hide)
     )
@@
     (property "Reference" "R14" (id 0) (at 169.545 50.8 90))
     (property "Value" "7.5K" (id 1) (at 169.545 55.88 90))
-    (property "Footprint" "Library:R_1206_3216Metric_Pad1.30x1.75mm_HandSolder" (id 2) (at 169.545 53.34 0)
+    (property "Footprint" "Resistor_SMD:R_1206_3216Metric_Pad1.30x1.75mm_HandSolder" (id 2) (at 169.545 53.34 0)
       (effects (font (size 1.27 1.27)) hide)
     )
@@
     (property "Reference" "R15" (id 0) (at 169.545 138.43 90))
     (property "Value" "7.5K" (id 1) (at 169.545 143.51 90))
-    (property "Footprint" "Library:R_1206_3216Metric_Pad1.30x1.75mm_HandSolder" (id 2) (at 169.545 140.97 0)
+    (property "Footprint" "Resistor_SMD:R_1206_3216Metric_Pad1.30x1.75mm_HandSolder" (id 2) (at 169.545 140.97 0)
       (effects (font (size 1.27 1.27)) hide)
     )
@@
       (effects (font (size 1.27 1.27)) (justify left))
     )
-    (property "Footprint" "Library:R_1206_3216Metric_Pad1.30x1.75mm_HandSolder" (id 2) (at 181.61 29.21 0)
+    (property "Footprint" "Resistor_SMD:R_1206_3216Metric_Pad1.30x1.75mm_HandSolder" (id 2) (at 181.61 29.21 0)
       (effects (font (size 1.27 1.27)) hide)
     )
@@
       (effects (font (size 1.27 1.27)) (justify left))
     )
-    (property "Footprint" "Library:R_1206_3216Metric_Pad1.30x1.75mm_HandSolder" (id 2) (at 181.61 116.84 0)
+    (property "Footprint" "Resistor_SMD:R_1206_3216Metric_Pad1.30x1.75mm_HandSolder" (id 2) (at 181.61 116.84 0)
       (effects (font (size 1.27 1.27)) hide)
     )
@@
       (effects (font (size 1.27 1.27)) (justify left))
     )
-    (property "Footprint" "Library:R_1206_3216Metric_Pad1.30x1.75mm_HandSolder" (id 2) (at 208.28 57.785 0)
+    (property "Footprint" "Resistor_SMD:R_1206_3216Metric_Pad1.30x1.75mm_HandSolder" (id 2) (at 208.28 57.785 0)
       (effects (font (size 1.27 1.27)) hide)
     )
@@
       (effects (font (size 1.27 1.27)) (justify left))
     )
-    (property "Footprint" "Library:R_1206_3216Metric_Pad1.30x1.75mm_HandSolder" (id 2) (at 208.28 145.415 0)
+    (property "Footprint" "Resistor_SMD:R_1206_3216Metric_Pad1.30x1.75mm_HandSolder" (id 2) (at 208.28 145.415 0)
       (effects (font (size 1.27 1.27)) hide)
     )
@@
     (property "Reference" "R20" (id 0) (at 213.995 50.8 90))
     (property "Value" "7.5K" (id 1) (at 213.995 55.88 90))
-    (property "Footprint" "Library:R_1206_3216Metric_Pad1.30x1.75mm_HandSolder" (id 2) (at 213.995 53.34 0)
+    (property "Footprint" "Resistor_SMD:R_1206_3216Metric_Pad1.30x1.75mm_HandSolder" (id 2) (at 213.995 53.34 0)
       (effects (font (size 1.27 1.27)) hide)
     )
@@
     (property "Reference" "R21" (id 0) (at 213.995 138.43 90))
     (property "Value" "7.5K" (id 1) (at 213.995 143.51 90))
-    (property "Footprint" "Library:R_1206_3216Metric_Pad1.30x1.75mm_HandSolder" (id 2) (at 213.995 140.97 0)
+    (property "Footprint" "Resistor_SMD:R_1206_3216Metric_Pad1.30x1.75mm_HandSolder" (id 2) (at 213.995 140.97 0)
       (effects (font (size 1.27 1.27)) hide)
     )
@@
       (effects (font (size 1.27 1.27)) (justify left))
     )
-    (property "Footprint" "Library:R_1206_3216Metric_Pad1.30x1.75mm_HandSolder" (id 2) (at 226.06 29.21 0)
+    (property "Footprint" "Resistor_SMD:R_1206_3216Metric_Pad1.30x1.75mm_HandSolder" (id 2) (at 226.06 29.21 0)
       (effects (font (size 1.27 1.27)) hide)
     )
@@
       (effects (font (size 1.27 1.27)) (justify left))
     )
-    (property "Footprint" "Library:R_1206_3216Metric_Pad1.30x1.75mm_HandSolder" (id 2) (at 226.06 116.84 0)
-      (effects (font (size 1.27 1.27)) hide)
-    )
+    (property "Footprint" "Resistor_SMD:R_1206_3216Metric_Pad1.30x1.75mm_HandSolder" (id 2) (at 226.06 116.84 0)
+      (effects (font (size 1.27 1.27)) hide)
+    )
